File: Bird_detector_V1/Audio.kicad_sch (KiCad schematic)
At the start: 0 parts

Commit message: r
Parts:
- added C10, C11, C12, C14, C16: 100n, symbol Device:C_Small
- added C13, C15, C17, CA1, CA2, CA3, CA4: 1u, symbol Device:C_Small
- added C9: 10u, symbol Device:C_Small
- added JP1: ADR1, Jumper:SolderJumper-3_P1.3mm_Bridged12_RoundedPad1.0x1.5mm_NumberLabels, symbol Jumper:SolderJumper_3_Bridged12
- added JP2: ADR0, Jumper:SolderJumper-3_P1.3mm_Bridged12_RoundedPad1.0x1.5mm_NumberLabels, symbol Jumper:SolderJumper_3_Bridged12
- added R? (x2): 2k, symbol Device:R_Small
- added TP4: TestPoint, TestPoint:TestPoint_Pad_1.5x1.5mm, symbol Connector:TestPoint
- added U4: TLV320ADC3100, Package_DFN_QFN:VQFN-24-1EP_4x4mm_P0.5mm_EP2.45x2.45mm_ThermalVias, symbol My_custom_lib:TLV320ADC3100
Connections:
- new net: CA3.2, R?.2, U4.12 (IN2R(P))
- new net: JP2.2 (C), U4.15 (I2C_ADR0)
- new net: JP1.2 (C), U4.16 (I2C_ADR1)
- new net: R?.1, R?.2, U4.5 (MICBIAS1)
- new net: CA2.2, R?.1, U4.7 (IN2L(P))
- new net +3.3VA: C14.1, C15.1, C16.1, C17.1, JP1.1 (A), JP2.1 (A), U4.10 (AVDD), U4.21 (IOVDD)
- new net 12MHz: U4.24 (MCLK)
- new net 1V8A: C12.1, C13.1, U4.22 (DVDD)
- new net GND: C11.2, C12.2, C13.2, C14.2, C15.2, C16.2, C17.2, CA1.2, CA4.2, JP1.3 (B), JP2.3 (B), U4.13 (IN3R(M)), U4.23 (DVSS), U4.6 (IN3L(M)), U4.9 (AVSS)
- new net RESET: C11.1, U4.4 (RESET)
- new net SCK: U4.1 (BCLK(SCK))
- new net SCL: U4.17 (SCL)
- new net SD: U4.3 (DOUT(SD))
- new net SDA: U4.18 (SDA)
- new net WS: U4.2 (WCLK(WS))
- no-connect marks 0 -> 4
Other:
- note added: "10mA max expected consumption"
- note added: "I2C Adress: 00110[ADR0][ADR1] @400KHz max"
- note added: "maybe instead of RESET add a lond delay like 50-100ms"

Commit message: g
Parts:
- added C11, C12, C13, CA2, CA5: 1u, Capacitor_SMD:C_0603_1608Metric_Pad1.08x0.95mm_HandSolder, symbol Device:C_Small
- added FB1: MZ1608-102Y, Resistor_SMD:R_0603_1608Metric_Pad0.98x0.95mm_HandSolder, symbol Device:FerriteBead_Small
- added U5, U6: MIC5317, Package_TO_SOT_SMD:SOT-23-5_HandSoldering, symbol My_custom_lib:MIC5317
- C10: renamed from C11; footprint (none) -> Capacitor_SMD:C_0603_1608Metric_Pad1.08x0.95mm_HandSolder
- C14: renamed from C12; footprint (none) -> Capacitor_SMD:C_0603_1608Metric_Pad1.08x0.95mm_HandSolder
- C15: renamed from C13; footprint (none) -> Capacitor_SMD:C_0603_1608Metric_Pad1.08x0.95mm_HandSolder
- C16: renamed from C14; footprint (none) -> Capacitor_SMD:C_0603_1608Metric_Pad1.08x0.95mm_HandSolder
- C17: renamed from C15; footprint (none) -> Capacitor_SMD:C_0603_1608Metric_Pad1.08x0.95mm_HandSolder
- C18: renamed from C16; footprint (none) -> Capacitor_SMD:C_0603_1608Metric_Pad1.08x0.95mm_HandSolder
- C19: renamed from C17; footprint (none) -> Capacitor_SMD:C_0603_1608Metric_Pad1.08x0.95mm_HandSolder
- C8: renamed from C9; footprint (none) -> Capacitor_SMD:C_0603_1608Metric_Pad1.08x0.95mm_HandSolder
- C9: renamed from C10; footprint (none) -> Capacitor_SMD:C_0603_1608Metric_Pad1.08x0.95mm_HandSolder
- CA1: footprint (none) -> Capacitor_SMD:C_0603_1608Metric_Pad1.08x0.95mm_HandSolder
- CA3: renamed from CA2; footprint (none) -> Capacitor_SMD:C_0603_1608Metric_Pad1.08x0.95mm_HandSolder
- CA4: renamed from CA3; footprint (none) -> Capacitor_SMD:C_0603_1608Metric_Pad1.08x0.95mm_HandSolder
- CA6: renamed from CA4; footprint (none) -> Capacitor_SMD:C_0603_1608Metric_Pad1.08x0.95mm_HandSolder
- R2, R3: renamed from R?; footprint (none) -> Resistor_SMD:R_0603_1608Metric_Pad0.98x0.95mm_HandSolder
Connections:
- net +3.3VA: now also C13.1, U5.5 (OUT), U6.1 (IN), U6.3 (EN)
- net 1V8A: now also U6.5 (OUT)
- net GND: now also C11.2, C12.2, C13.2, U5.2 (GND), U6.2 (GND)
- net at CA6.1: now also CA5.1
- net at CA4.1: now also CA5.2
- net at CA3.1: now also CA2.1
- net at CA1.1: now also CA2.2
- net RESET renamed RESET_AUDIO
- new net: C12.1, FB1.2, U5.1 (IN), U5.3 (EN)
- new net +3V8: C11.1, FB1.1
- no-connect marks 4 -> 5
Other:
- note added: "20mA max expected consumption"
- note removed: "10mA max expected consumption"
- moved on the sheet: C14, C15, C16, C17, C18, C19

Commit message: g
Parts:
- JP1, JP2: now left out of the parts list
- renumbered C8 to C15, C9 to C16, C10 to C17, C11 to C18, C12 to C19, C13 to C20, C14 to C21, C15 to C22, C16 to C23, C17 to C24, C18 to C25, C19 to C26, R2 to R5, R3 to R6

Commit message: f
Parts:
- removed C15: 10u, Capacitor_SMD:C_0603_1608Metric_Pad1.08x0.95mm_HandSolder, symbol Device:C_Small
- removed C16: 100n, Capacitor_SMD:C_0603_1608Metric_Pad1.08x0.95mm_HandSolder, symbol Device:C_Small
- removed TP4: TestPoint, TestPoint:TestPoint_Pad_1.5x1.5mm, symbol Connector:TestPoint
- renumbered R5 to R23, R6 to R24

Commit message: j
Parts:
- added J? (x2): 292132-3, SHDR3W65P0X200_1X3_780X580X710P, symbol SamacSys_Parts:292132-3
- added R?: 1k, Resistor_SMD:R_0603_1608Metric_Pad0.98x0.95mm_HandSolder, symbol Device:R_Small
- added Y?: SiT1602BI-13-33E-12.000000G, Crystal:Crystal_SMD_2520-4Pin_2.5x2.0mm, symbol Device:Crystal_GND23
- renumbered C17 to C15, C18 to C16, C19 to C17, C20 to C18, C21 to C19, C22 to C20, C23 to C21, C24 to C22, C25 to C23, C26 to C24
Connections:
- net +3.3VA: now also R?.2, Y?.4
- net 12MHz: now also Y?.3
- net GND: now also Y?.2
- new net: R?.1, Y?.1
Other:
- note added: "direct connection is 90db so 12db loss vs preamp"
- moved on the sheet: C15, C16, C17, C18, C19, C20, C21, C22, C23, C24, CA1, CA2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

Commit message: f
Parts:
- J6, J7: renamed from J?; footprint SHDR3W65P0X200_1X3_780X580X710P -> SamacSys_Parts:SHDR3W65P0X200_1X3_780X580X710P
- gave numbers to parts that had none: 2
- renumbered R23 to R27, R24 to R28, U4 to U3, U5 to U4, U6 to U5

Commit message: R
Parts:
- removed J7: 292132-3, SamacSys_Parts:SHDR3W65P0X200_1X3_780X580X710P, symbol SamacSys_Parts:292132-3
- added C? (x2): 220p, Capacitor_SMD:C_0603_1608Metric_Pad1.08x0.95mm_HandSolder, symbol Device:C_Small
- added C? (x2): 4p7-10p, Capacitor_SMD:C_0603_1608Metric_Pad1.08x0.95mm_HandSolder, symbol Device:C_Small
- added CA?: 10n?, Capacitor_SMD:C_0603_1608Metric_Pad1.08x0.95mm_HandSolder, symbol Device:C_Small
- added CA?: 10u?, Capacitor_SMD:C_0603_1608Metric_Pad1.08x0.95mm_HandSolder, symbol Device:C_Small
- added J?: 292132-3, SamacSys_Parts:SHDR3W65P0X200_1X3_780X580X710P, symbol SamacSys_Parts:292132-3
- added R?: supresor, Resistor_SMD:R_0603_1608Metric_Pad0.98x0.95mm_HandSolder, symbol Device:R_Small
- added R? (x4): 1Meg, Resistor_SMD:R_0603_1608Metric_Pad0.98x0.95mm_HandSolder, symbol Device:R_Small
- added R?: 1k, Resistor_SMD:R_0603_1608Metric_Pad0.98x0.95mm_HandSolder, symbol Device:R_Small
- added R?: 100, Resistor_SMD:R_0603_1608Metric_Pad0.98x0.95mm_HandSolder, symbol Device:R_Small
- added U?: OP179GS, Package_SO:SOIC-8_3.9x4.9mm_P1.27mm, symbol Amplifier_Operational:OP179GS
Connections:
- net GND: now also C?.2, C?.2, C?.2, C?.2, R?.2, R?.2, R?.2
- net Shield1: now reaches J6.2
- net Shield1: now also C?.1, R?.1
- new net: CA?.2, R?.2, U?.2 (-)
- new net: R?.1, U?.3 (+), U?.6
- new net: R?.1, R?.1
- new net: C?.1, CA?.1, R?.2
- new net: CA?.1, R?.2
- new net Shield2: C?.1, J?.2, R?.1
- new net bias: R?.1
Other:
- note added: "16mm^2 = 5.77pF with this stack up"
- note added: "Power"
- note added: "Shield terminations"
- note added: "low pass filter 16khz"
- moved on the sheet: C16, C17, C18, C19, C20, C21, C22, C23, C24, FB1, U4, U5

Commit message: b
Parts:
- removed CA?: 10u?, Capacitor_SMD:C_0603_1608Metric_Pad1.08x0.95mm_HandSolder, symbol Device:C_Small
- added R?: 10k, Resistor_SMD:R_0603_1608Metric_Pad0.98x0.95mm_HandSolder, symbol Device:R_Small
- added R?: 33k, Resistor_SMD:R_0603_1608Metric_Pad0.98x0.95mm_HandSolder, symbol Device:R_Small
- R?: value supresor -> ESD supresor
Connections:
- net GND: now also CA5.1, CA6.1, J?.1, R?.2, U?.4 (V-), R?.1
- net at CA?.2, R?.2: now also U?.3 (+); no longer U?.2 (-)
- net at R?.1, U?.6: now also R?.2; no longer U?.3 (+)
- net at R26.1: no longer Y1.1
- net at R?.1, R?.1: now also J?.3
- net at C?.1, R?.2: now also CA4.1, CA5.2
- net at R?.1: now also C?.1, CA?.1, R?.2
- new net: R?.1, R?.2, U?.2 (-)
Other:
- note added: "low pass filter not even sure why since cut off si so high"
- note added: "or 36k"
- note added: "since i have only one power rail"
- note removed: "low pass filter 16khz"
- moved on the sheet: C16, C17, C18, C19, C20, C21, C22, C23, C24, C?, CA2, CA5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
