File: Bird_detector_V1/Audio.kicad_sch (KiCad schematic)
At the start: 43 parts, among them J6 292132-3, U3 TLV320ADC3100, U4 MIC5317, U5 MIC5317, Y1 SiT1602BI-13-33E-12.000000G

Commit message: v
Parts:
- gave numbers to parts that had none: 16
- renumbered C15 to C24, C16 to C27, C17 to C28, C18 to C29, C19 to C30, C20 to C31, C21 to C32, C22 to C33, C23 to C34, C24 to C35, CA4 to CA5, CA5 to CA6, CA6 to CA7, JP1 to JP3, JP2 to JP4, R26 to R38, R27 to R40, R28 to R42, U3 to U4, U4 to U6, U5 to U7

Commit message: f
Parts:
- C24: renamed from C25; value 220p -> 15n
- C26: value 220p -> 15n
- R44: renamed from R43; value 1k -> 100
- U5: value OP179GS -> TLV9161IDBVR
- renumbered C22 to C23, C23 to C25, C24 to C27, C27 to C28, C28 to C29, C29 to C30, C32 to C31, C33 to C32, C34 to C33, C35 to C34, C30 to C35, C31 to C36, CA4 to CA1, CA6 to CA3, CA1 to CA4, CA3 to CA5, CA5 to CA6, J7 to J6, J6 to J7, JP3 to JP4, JP4 to JP5, R44 to R36, R41 to R37, R36 to R38, R45 to R39, R37 to R40, R39 to R41, R46 to R42, R47 to R43, R40 to R45, R42 to R46, R38 to R47, U4 to U6, U6 to U7, U7 to U8
Other:
- note added: "gain of about x4"
- note removed: "low pass filter not even sure why since cut off si so high"
- moved on the sheet: C25, R40

Commit message: v
Parts:
- removed CA4, CA7: 1u, Capacitor_SMD:C_0603_1608Metric_Pad1.08x0.95mm_HandSolder, symbol Device:C_Small
- removed J7: 292132-3, SamacSys_Parts:SHDR3W65P0X200_1X3_780X580X710P, symbol SamacSys_Parts:292132-3
- removed R41: 1Meg, Resistor_SMD:R_0603_1608Metric_Pad0.98x0.95mm_HandSolder, symbol Device:R_Small
- removed R45: 2k, Resistor_SMD:R_0603_1608Metric_Pad0.98x0.95mm_HandSolder, symbol Device:R_Small
- added C30, C33: 15n, Capacitor_SMD:C_0603_1608Metric_Pad1.08x0.95mm_HandSolder, symbol Device:C_Small
- added CA6: 10n?, Capacitor_SMD:C_0603_1608Metric_Pad1.08x0.95mm_HandSolder, symbol Device:C_Small
- added J9: 292132-3, SamacSys_Parts:SHDR3W65P0X200_1X3_780X580X710P, symbol SamacSys_Parts:292132-3
- added R49, R53, R54: 100, Resistor_SMD:R_0603_1608Metric_Pad0.98x0.95mm_HandSolder, symbol Device:R_Small
- added R51: 2k, Resistor_SMD:R_0603_1608Metric_Pad0.98x0.95mm_HandSolder, symbol Device:R_Small
- added R52: 1Meg, Resistor_SMD:R_0603_1608Metric_Pad0.98x0.95mm_HandSolder, symbol Device:R_Small
- added R57: ESD supresor, Resistor_SMD:R_0603_1608Metric_Pad0.98x0.95mm_HandSolder, symbol Device:R_Small
- added R58: 33k, Resistor_SMD:R_0603_1608Metric_Pad0.98x0.95mm_HandSolder, symbol Device:R_Small
- added R59: 10k, Resistor_SMD:R_0603_1608Metric_Pad0.98x0.95mm_HandSolder, symbol Device:R_Small
- added U9: TLV9161IDBVR, Package_SO:SOIC-8_3.9x4.9mm_P1.27mm, symbol Amplifier_Operational:OP179GS
- renumbered C24 to C27, C26 to C28, C27 to C29, C23 to C31, C25 to C32, C28 to C34, C29 to C35, C30 to C36, C35 to C37, C36 to C38, C31 to C39, C32 to C40, C33 to C41, C34 to C42, CA6 to CA4, J6 to J8, JP4 to JP3, JP5 to JP4, R46 to R42, R39 to R43, R37 to R44, R44 to R45, R47 to R46, R36 to R47, R42 to R48, R43 to R50, R38 to R55, R40 to R56, U7 to U10, U8 to U11, U5 to U7, U6 to U8
Connections:
- net +3.3VA: now also U7.7 (V+), U9.7 (V+)
- net 12MHz: now also R49.2; no longer Y1.3
- net 1V8A: now also R43.1, R52.1
- net GND: now also CA2.2, CA5.2, C30.2, C33.2, J9.1, R57.2, R59.1, U9.4 (V-); no longer CA3.1, R43.2, U8.13 (IN3R(M)), U8.6 (IN3L(M))
- net Shield1: now also J8.2
- net Shield2: now also J9.2; no longer J8.2
- net FB_L: now reaches R48.1, R50.2, U7.2 (-)
- net at U7.3 (+): now also CA1.1, R43.2; no longer CA1.2
- net OUT_L: now reaches R45.1, R48.2, U7.6
- net at R46.1: now also Y1.1
- net RAW_AUDIO_L: now reaches J8.3, R44.1, R47.1
- net RAW_AUDIO_L: now also R42.2
- net filtered_3v8: now reaches C35.1, FB1.2, U10.1 (IN), U10.3 (EN)
- net at C28.1, R45.2: now also CA3.1; no longer CA3.2, CA4.1
- net at CA4.2, U8.12 (IN2R(P)): no longer R42.2
- net MIC_BIASS: now reaches R42.1, U8.5 (MICBIAS1)
- net MIC_BIASS: now also R51.1
- net at U8.7 (IN2L(P)): now also CA3.2; no longer CA5.2
- net at C27.1, R44.2: now also CA1.2; no longer CA1.1, R43.1
- net at CA5.1: now also U8.13 (IN3R(M)); no longer CA2.1
- new net: C33.1, CA4.1, R54.2
- new net: R49.1, Y1.3
- new net: CA6.1, R52.2, U9.3 (+)
- new net: C30.1, CA6.2, R53.2
- new net: CA2.1, U8.6 (IN3L(M))
- new net FB_R: R58.1, R59.2, U9.2 (-)
- new net OUT_R: R54.1, R58.2, U9.6
- new net RAW_AUDIO_P: J9.3, R51.2, R53.1, R57.1
Other:
- note removed: "since i have only one power rail"
- moved on the sheet: C27, C28, C29, C31, C32, C34, C35, C36, C37, C38, C39, C40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

Commit message: v
Parts:
- removed C31, C32: 4p7-10p, Capacitor_SMD:C_0603_1608Metric_Pad1.08x0.95mm_HandSolder, symbol Device:C_Small
- added J12, J16: PCB CAP, Z_mycustom_footprint_lib:PCB cap start, symbol Connector_Generic:Conn_01x01
Connections:
- net Shield1: now also J12.1 (Pin_1)
- net Shield2: now also J16.1 (Pin_1)
- net RIGHT_IN_AMP: now reaches C33.1, CA4.1, R54.2
- net 12MHz_enable: now reaches R46.1, Y1.1
- net 12MHz_raw: now reaches R49.1, Y1.3
- net LEFT_IN_AMP: now reaches C28.1, CA3.1, R45.2
Changed lines of the file:
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@@
-    (stroke (width 0) (type default) (color 0 0 0 0))
-  )
-  (wire (pts (xy 341.63 99.06) (xy 341.63 101.6))
     (stroke (width 0) (type default) (color 0 0 0 0))
   )
@@
   )
   (wire (pts (xy 241.3 46.99) (xy 241.3 49.53))
-    (stroke (width 0) (type default) (color 0 0 0 0))
-  )
-  (wire (pts (xy 370.84 99.06) (xy 370.84 101.6))
     (stroke (width 0) (type default) (color 0 0 0 0))
   )
@@
     (effects (font (size 0.5 0.5)) (justify left bottom))
   )
+  (label "RIGHT_IN_AMP" (at 177.8 77.47 0)
+    (effects (font (size 1.27 1.27)) (justify left bottom))
+  )
+  (label "12MHz_raw" (at 265.43 31.75 0)
+    (effects (font (size 0.5 0.5)) (justify left bottom))
+  )
   (label "RAW_AUDIO_P" (at 44.45 90.17 0)
     (effects (font (size 1.27 1.27)) (justify left bottom))
@@
     (effects (font (size 0.5 0.5)) (justify left bottom))
   )
+  (label "LEFT_IN_AMP" (at 177.8 62.23 0)
+    (effects (font (size 1.27 1.27)) (justify left bottom))
+  )
   (label "OUT_L" (at 139.7 38.1 0)
+    (effects (font (size 0.5 0.5)) (justify left bottom))
+  )
+  (label "12MHz_enable" (at 283.21 38.1 0)
     (effects (font (size 0.5 0.5)) (justify left bottom))
   )
@@
     )
     (property "Datasheet" "~" (id 3) (at 148.59 38.1 0)
-      (effects (font (size 1.27 1.27)) hide)
-    )
-    (pin "1")
-    (pin "2")
-  )
-  (symbol (lib_id "Device:C_Small") (at 341.63 96.52 0) (unit 1)
-    (in_bom yes) (on_board yes) (fields_autoplaced)
-    (property "Reference" "C31" (id 0) (at 344.17 95.2562 0)
-      (effects (font (size 1.27 1.27)) (justify left))
-    )
-    (property "Value" "4p7-10p" (id 1) (at 344.17 97.7962 0)
-      (effects (font (size 1.27 1.27)) (justify left))
-    )
-    (property "Footprint" "Capacitor_SMD:C_0603_1608Metric_Pad1.08x0.95mm_HandSolder" (id 2) (at 341.63 96.52 0)
-      (effects (font (size 1.27 1.27)) hide)
-    )
-    (property "Datasheet" "~" (id 3) (at 341.63 96.52 0)
       (effects (font (size 1.27 1.27)) hide)
     )
@@
     (pin "2")
   )
-  (symbol (lib_id "Device:C_Small") (at 370.84 96.52 0) (unit 1)
-    (in_bom yes) (on_board yes) (fields_autoplaced)
-    (property "Reference" "C32" (id 0) (at 373.38 95.2562 0)
-      (effects (font (size 1.27 1.27)) (justify left))
-    )
-    (property "Value" "4p7-10p" (id 1) (at 373.38 97.7962 0)
-      (effects (font (size 1.27 1.27)) (justify left))
-    )
-    (property "Footprint" "Capacitor_SMD:C_0603_1608Metric_Pad1.08x0.95mm_HandSolder" (id 2) (at 370.84 96.52 0)
-      (effects (font (size 1.27 1.27)) hide)
-    )
-    (property "Datasheet" "~" (id 3) (at 370.84 96.52 0)
-      (effects (font (size 1.27 1.27)) hide)
-    )
-    (pin "1")
-    (pin "2")
-  )
-  (symbol (lib_id "power:GND") (at 370.84 101.6 0) (unit 1)
-    (in_bom yes) (on_board yes) (fields_autoplaced)
-    (property "Reference" "#PWR0105" (id 0) (at 370.84 107.95 0)
-      (effects (font (size 1.27 1.27)) hide)
-    )
-    (property "Value" "GND" (id 1) (at 370.84 106.68 0)
-      (effects (font (size 1.27 1.27)) hide)
-    )
-    (property "Footprint" "" (id 2) (at 370.84 101.6 0)
-      (effects (font (size 1.27 1.27)) hide)
-    )
-    (property "Datasheet" "" (id 3) (at 370.84 101.6 0)
-      (effects (font (size 1.27 1.27)) hide)
-    )
-    (pin "1")
-  )
   (symbol (lib_id "Device:C_Small") (at 381 139.7 0) (unit 1)
     (in_bom yes) (on_board yes) (fields_autoplaced)
@@
     )
     (property "Datasheet" "" (id 3) (at 204.47 57.15 0)
+      (effects (font (size 1.27 1.27)) hide)
+    )
+    (pin "1")
+  )
+  (symbol (lib_id "Connector_Generic:Conn_01x01") (at 370.84 99.06 270) (unit 1)
+    (in_bom no) (on_board yes)
+    (property "Reference" "J16" (id 0) (at 369.57 102.87 90)
+      (effects (font (size 1.27 1.27)) (justify left))
+    )
+    (property "Value" "PCB CAP" (id 1) (at 367.03 105.41 90)
+      (effects (font (size 1.27 1.27)) (justify left))
+    )
+    (property "Footprint" "Z_mycustom_footprint_lib:PCB cap start" (id 2) (at 370.84 99.06 0)
+      (effects (font (size 1.27 1.27)) hide)
+    )
+    (property "Datasheet" "~" (id 3) (at 370.84 99.06 0)
       (effects (font (size 1.27 1.27)) hide)
     )
@@
     )
     (property "Datasheet" "" (id 3) (at 284.48 144.78 0)
+      (effects (font (size 1.27 1.27)) hide)
+    )
+    (pin "1")
+  )
+  (symbol (lib_id "Connector_Generic:Conn_01x01") (at 341.63 99.06 270) (unit 1)
+    (in_bom no) (on_board yes)
+    (property "Reference" "J12" (id 0) (at 340.36 102.87 90)
+      (effects (font (size 1.27 1.27)) (justify left))
+    )
+    (property "Value" "PCB CAP" (id 1) (at 337.82 105.41 90)
+      (effects (font (size 1.27 1.27)) (justify left))
+    )
+    (property "Footprint" "Z_mycustom_footprint_lib:PCB cap start" (id 2) (at 341.63 99.06 0)
+      (effects (font (size 1.27 1.27)) hide)
+    )
+    (property "Datasheet" "~" (id 3) (at 341.63 99.06 0)
       (effects (font (size 1.27 1.27)) hide)
     )
@@
     (pin "2")
   )
-  (symbol (lib_id "power:GND") (at 341.63 101.6 0) (unit 1)
-    (in_bom yes) (on_board yes) (fields_autoplaced)
-    (property "Reference" "#PWR0103" (id 0) (at 341.63 107.95 0)
-      (effects (font (size 1.27 1.27)) hide)
-    )
-    (property "Value" "GND" (id 1) (at 341.63 106.68 0)
-      (effects (font (size 1.27 1.27)) hide)
-    )
-    (property "Footprint" "" (id 2) (at 341.63 101.6 0)
-      (effects (font (size 1.27 1.27)) hide)
-    )
-    (property "Datasheet" "" (id 3) (at 341.63 101.6 0)
-      (effects (font (size 1.27 1.27)) hide)
-    )
-    (pin "1")
-  )
   (symbol (lib_id "power:GND") (at 76.2 45.72 0) (unit 1)

Commit message: f
Parts:
- C27, C28, C30, C33: value 15n -> 100n
- C68: renamed from CA1; value 10n? -> 15n
- C73: renamed from CA6; value 10n? -> 15n
- J8, J9: footprint SamacSys_Parts:SHDR3W65P0X200_1X3_780X580X710P -> SHDR3W65P0X200_1X3_780X580X710P
- R44, R45, R49, R53, R54: value 100 -> 60
- renumbered CA2 to C69, CA3 to C70, CA4 to C71, CA5 to C72
Connections:
- net +3.3VA: now also JP3.3 (B), JP4.3 (B); no longer JP3.1 (A), JP4.1 (A)
- net GND: now also JP3.1 (A), JP4.1 (A), U8.25 (GND); no longer JP3.3 (B), JP4.3 (B)
- no-connect marks 5 -> 1
Other:
- moved on the sheet: JP3, JP4

Commit message: h
Parts:
- removed FB1: MZ1608-102Y, Resistor_SMD:R_0603_1608Metric_Pad0.98x0.95mm_HandSolder, symbol Device:FerriteBead_Small
- removed U7, U9: TLV9161IDBVR, Package_SO:SOIC-8_3.9x4.9mm_P1.27mm, symbol Amplifier_Operational:OP179GS
- added C19, C6: 22u, Capacitor_SMD:C_0805_2012Metric_Pad1.18x1.45mm_HandSolder, symbol Device:C_Small
- added C79: 100n, Capacitor_SMD:C_0603_1608Metric_Pad1.08x0.95mm_HandSolder, symbol Device:C_Small
- added L4, L5: 47u, Inductor_SMD:L_0603_1608Metric, symbol Device:L_Small
- added R102, R103: 64k, Resistor_SMD:R_0603_1608Metric_Pad0.98x0.95mm_HandSolder, symbol Device:R_Small
- added U7: TLV9062xD, Package_SO:SOIC-8_3.9x4.9mm_P1.27mm, symbol Amplifier_Operational:TLV9062xD
- C34, C35: value 1u -> 22u; footprint Capacitor_SMD:C_0603_1608Metric_Pad1.08x0.95mm_HandSolder -> Capacitor_SMD:C_0805_2012Metric_Pad1.18x1.45mm_HandSolder
- J8, J9: footprint SHDR3W65P0X200_1X3_780X580X710P -> SamacSys_Parts:SHDR3W65P0X200_1X3_780X580X710P
- R42, R51: value 2k -> 2k2
- R47, R57: value ESD supresor -> ESD
- R48, R58: value 33k -> 64k
Connections:
- net +3.3VA: now also C19.1, C79.1, L4.2, U7.8 (V+); no longer U8.10 (AVDD)
- net +3V8: now also L5.1
- net FB_L: now also R58.2, U7.2 (-)
- net FB_R: now also R102.1, R103.2, U7.6 (-); no longer R58.1
- net GND: now also C19.2, C6.2, C79.2, U7.4 (V-)
- net OUT_L: now also R58.1, U7.1
- net OUT_R: now also R102.2, R103.1, U7.7; no longer R58.2
- net filtered_3v8: now also L5.2
- net at C68.1, R43.2: now also U7.3 (+)
- net at C73.1, R52.2: now also U7.5 (+)
- new net: C6.1, L4.1, U8.10 (AVDD)
Other:
- note removed: "or 36k"
- moved on the sheet: C29, C34, C35, R43, R52

Commit message: b
Other:
- title: (none) -> Bird Detection and Recognition System
Changed lines of the file:
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@@
 (kicad_sch (version 20211123) (generator eeschema)
   (paper "A3")
+  (title_block
+    (title "Bird Detection and Recognition System")
+    (rev "V0.1")
+  )
   (junction (at 58.42 35.56) (diameter 0) (color 0 0 0 0)
   )
