File: Bird_detector_V1/Audio.kicad_sch (KiCad schematic)
At the start: 56 parts, among them J12 PCB CAP, J16 PCB CAP, J8 292132-3, J9 292132-3, U10 MIC5317, U11 MIC5317, U7 TLV9062xD, U8 TLV320ADC3100, Y1 SiT1602BI-13-33E-12.000000G

Commit message: y
Parts:
- removed J12, J16: PCB CAP, Z_mycustom_footprint_lib:PCB cap start, symbol Connector_Generic:Conn_01x01
- added C83, C84: 6p8, Capacitor_SMD:C_0603_1608Metric, symbol Device:C_Small
Connections:
- net GND: now also C83.2, C84.2
- net Shield1: now also C83.1
- net Shield2: now also C84.1
Changed lines of the file:
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@@
+    (stroke (width 0) (type default) (color 0 0 0 0))
+  )
+  (wire (pts (xy 375.92 99.06) (xy 375.92 101.6))
     (stroke (width 0) (type default) (color 0 0 0 0))
   )
@@
     (stroke (width 0) (type default) (color 0 0 0 0))
   )
-  (wire (pts (xy 341.63 91.44) (xy 356.87 91.44))
+  (wire (pts (xy 349.25 91.44) (xy 356.87 91.44))
     (stroke (width 0) (type default) (color 0 0 0 0))
   )
@@
     (stroke (width 0) (type default) (color 0 0 0 0))
   )
-  (wire (pts (xy 370.84 91.44) (xy 383.54 91.44))
+  (wire (pts (xy 375.92 91.44) (xy 383.54 91.44))
     (stroke (width 0) (type default) (color 0 0 0 0))
   )
@@
     (stroke (width 0) (type default) (color 0 0 0 0))
   )
-  (wire (pts (xy 370.84 93.98) (xy 370.84 91.44))
+  (wire (pts (xy 375.92 93.98) (xy 375.92 91.44))
     (stroke (width 0) (type default) (color 0 0 0 0))
   )
@@
     (stroke (width 0) (type default) (color 0 0 0 0))
   )
-  (wire (pts (xy 341.63 93.98) (xy 341.63 91.44))
+  (wire (pts (xy 349.25 93.98) (xy 349.25 91.44))
+    (stroke (width 0) (type default) (color 0 0 0 0))
+  )
+  (wire (pts (xy 349.25 99.06) (xy 349.25 101.6))
     (stroke (width 0) (type default) (color 0 0 0 0))
   )
@@
     (stroke (width 0) (type default) (color 0 0 0 0))
   )
-  (text "16mm^2 = 5.77pF\n with this stack up" (at 320.04 96.52 0)
+  (text "16mm^2 = 5.77pF\n with this stack up" (at 330.2 87.63 0)
     (effects (font (size 1.27 1.27)) (justify left bottom))
   )
@@
     )
     (property "Datasheet" "" (id 3) (at 337.82 144.78 0)
+      (effects (font (size 1.27 1.27)) hide)
+    )
+    (pin "1")
+  )
+  (symbol (lib_id "power:GND") (at 349.25 101.6 0) (unit 1)
+    (in_bom yes) (on_board yes) (fields_autoplaced)
+    (property "Reference" "#PWR0225" (id 0) (at 349.25 107.95 0)
+      (effects (font (size 1.27 1.27)) hide)
+    )
+    (property "Value" "GND" (id 1) (at 349.25 106.68 0)
+      (effects (font (size 1.27 1.27)) hide)
+    )
+    (property "Footprint" "" (id 2) (at 349.25 101.6 0)
+      (effects (font (size 1.27 1.27)) hide)
+    )
+    (property "Datasheet" "" (id 3) (at 349.25 101.6 0)
       (effects (font (size 1.27 1.27)) hide)
     )
@@
     (pin "9")
   )
+  (symbol (lib_id "power:GND") (at 375.92 101.6 0) (unit 1)
+    (in_bom yes) (on_board yes) (fields_autoplaced)
+    (property "Reference" "#PWR0223" (id 0) (at 375.92 107.95 0)
+      (effects (font (size 1.27 1.27)) hide)
+    )
+    (property "Value" "GND" (id 1) (at 375.92 106.68 0)
+      (effects (font (size 1.27 1.27)) hide)
+    )
+    (property "Footprint" "" (id 2) (at 375.92 101.6 0)
+      (effects (font (size 1.27 1.27)) hide)
+    )
+    (property "Datasheet" "" (id 3) (at 375.92 101.6 0)
+      (effects (font (size 1.27 1.27)) hide)
+    )
+    (pin "1")
+  )
   (symbol (lib_id "power:+3V8") (at 276.86 132.08 0) (unit 1)
     (in_bom yes) (on_board yes) (fields_autoplaced)
@@
     (pin "1")
   )
-  (symbol (lib_id "Connector_Generic:Conn_01x01") (at 370.84 99.06 270) (unit 1)
-    (in_bom no) (on_board yes)
-    (property "Reference" "J16" (id 0) (at 369.57 102.87 90)
-      (effects (font (size 1.27 1.27)) (justify left))
-    )
-    (property "Value" "PCB CAP" (id 1) (at 367.03 105.41 90)
-      (effects (font (size 1.27 1.27)) (justify left))
-    )
-    (property "Footprint" "Z_mycustom_footprint_lib:PCB cap start" (id 2) (at 370.84 99.06 0)
-      (effects (font (size 1.27 1.27)) hide)
-    )
-    (property "Datasheet" "~" (id 3) (at 370.84 99.06 0)
-      (effects (font (size 1.27 1.27)) hide)
-    )
-    (pin "1")
-  )
   (symbol (lib_id "Device:R_Small") (at 71.12 90.17 90) (unit 1)
     (in_bom yes) (on_board yes) (fields_autoplaced)
@@
     (pin "1")
   )
-  (symbol (lib_id "Connector_Generic:Conn_01x01") (at 341.63 99.06 270) (unit 1)
-    (in_bom no) (on_board yes)
-    (property "Reference" "J12" (id 0) (at 340.36 102.87 90)
-      (effects (font (size 1.27 1.27)) (justify left))
-    )
-    (property "Value" "PCB CAP" (id 1) (at 337.82 105.41 90)
-      (effects (font (size 1.27 1.27)) (justify left))
-    )
-    (property "Footprint" "Z_mycustom_footprint_lib:PCB cap start" (id 2) (at 341.63 99.06 0)
-      (effects (font (size 1.27 1.27)) hide)
-    )
-    (property "Datasheet" "~" (id 3) (at 341.63 99.06 0)
-      (effects (font (size 1.27 1.27)) hide)
-    )
-    (pin "1")
+  (symbol (lib_id "Device:C_Small") (at 349.25 96.52 0) (unit 1)
+    (in_bom yes) (on_board yes)
+    (property "Reference" "C83" (id 0) (at 351.79 95.25 0)
+      (effects (font (size 1.27 1.27)) (justify left))
+    )
+    (property "Value" "6p8" (id 1) (at 351.79 97.79 0)
+      (effects (font (size 1.27 1.27)) (justify left))
+    )
+    (property "Footprint" "Capacitor_SMD:C_0603_1608Metric" (id 2) (at 349.25 96.52 0)
+      (effects (font (size 1.27 1.27)) hide)
+    )
+    (property "Datasheet" "~" (id 3) (at 349.25 96.52 0)
+      (effects (font (size 1.27 1.27)) hide)
+    )
+    (pin "1")
+    (pin "2")
   )
   (symbol (lib_id "Device:C_Small") (at 360.68 170.18 0) (unit 1)
@@
       (effects (font (size 1.27 1.27)) hide)
     )
+    (pin "1")
+    (pin "2")
+  )
+  (symbol (lib_id "Device:C_Small") (at 375.92 96.52 0) (unit 1)
+    (in_bom yes) (on_board yes)
+    (property "Reference" "C84" (id 0) (at 378.46 95.25 0)
+      (effects (font (size 1.27 1.27)) (justify left))
+    )
+    (property "Value" "6p8" (id 1) (at 378.46 97.79 0)
+      (effects (font (size 1.27 1.27)) (justify left))
+    )
+    (property "Footprint" "Capacitor_SMD:C_0603_1608Metric" (id 2) (at 375.92 96.52 0)
+      (effects (font (size 1.27 1.27)) hide)
+    )
+    (property "Datasheet" "~" (id 3) (at 375.92 96.52 0)
+      (effects (font (size 1.27 1.27)) hide)
+    )

Commit message: g
Other:
- note added: "AUDIO ADC + MIC PREAMPLIFIER"
- note removed: "16mm^2 = 5.77pF with this stack up"
- moved on the sheet: C19, C27, C28, C29, C30, C33, C34, C35, C36, C37, C38, C39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
