File: Bird_detector_V1/Bird_detector_V1.kicad_sch (KiCad schematic)
At the start: 0 parts

Commit message: r
Other:
- sheet GSM+GPS ports: added CTS, DCD, DTR, ENABLE, RI, RTS, RX, STAT, TX; removed none

Commit message: g
Other:
- sheet Audio capture ports: added RESET_AUDIO, SCK, SCL, SD, SDA, WS; removed none
- sheet GSM+GPS ports: added RESET_GSM, SCL, SDA; removed none
- sheet MCU+WIFI+BT ports: added CTS, DCD, DTR, ENABLE, RESET_AUDIO, RESET_GSM, RI, RTS, RX, SCK, SCL, SD, SDA, STAT, TX, WS; removed none
- sheet Power Management +BMS ports: added SCL, SDA; removed none
- note added: "All SMD caps ceramic are 0603 16V X7R or better unless other notes are made All SMD resistors are 0603 Stack up: 4 layer FR4 sig gnd gnd+sig sig All non power traces should aim to be 50 ohm single ended impedance unless other requirements are in place Delata(T) aimed for is 20C or less"

Commit message: f
Other:
- sheet GSM+GPS ports: added RF_SYNC; removed none
- sheet MCU+WIFI+BT ports: added CARD_DET, CMD, DATA0, DATA1, DATA2, DATA3/CS, SCLK; removed none
- sheet Other data+storage ports: added CARD_DET, CMD, DATA0, DATA1, DATA2, DATA3/CS, SCLK; removed none
- sheet Power Management +BMS ports: added RF_SYNC; removed none

Commit message: R
Parts:
- added FID1: Fiducial, Fiducial:Fiducial_0.5mm_Mask1.5mm, symbol Mechanical:Fiducial
- added FID10: scale, Calibration_Scale:Gauge_10mm_Type2_SilkScreenTop, symbol Mechanical:Fiducial
- added FID2: kicad, Symbol:KiCad-Logo2_5mm_SilkScreen, symbol Mechanical:Fiducial
- added FID3: Case, symbol Mechanical:Fiducial
- added FID4, FID5, FID8, FID9: Cell, symbol Mechanical:Fiducial
- added FID6: garbage, Symbol:WEEE-Logo_4.2x6mm_SilkScreen, symbol Mechanical:Fiducial
- added FID7: Lid, symbol Mechanical:Fiducial
- added H1, H2, H3, H4: M3, MountingHole:MountingHole_3.2mm_M3_ISO7380_Pad_TopBottom, symbol Mechanical:MountingHole_Pad
Connections:
- new net GND: H1.1, H2.1, H3.1, H4.1
Other:
- note added: "CASE+ GRAPHICS + MECHANICAL"
