File: Bird_detector_V1/Bird_detector_V1.kicad_sch (KiCad schematic)
At the start: 14 parts

Commit message: v
Parts:
- removed FID8: Cell, symbol Mechanical:Fiducial
- added FID10: Cell, Z_mycustom_footprint_lib:18650 cell 3d model, symbol Mechanical:Fiducial
- added H1, H2: M3, MountingHole:MountingHole_3.2mm_M3_ISO7380_Pad_TopBottom, symbol Mechanical:MountingHole_Pad
- FID4, FID5, FID9: footprint (none) -> Z_mycustom_footprint_lib:18650 cell 3d model
- renumbered FID10 to FID8, H1 to H3, H2 to H4, H3 to H5, H4 to H6
Connections:
- net GND: now also H1.1, H2.1
Other:
- moved on the sheet: FID4, H3, H4, H5, H6

Commit message: f
Parts:
- renumbered FID8 to FID2, FID2 to FID3, FID6 to FID4, FID3 to FID5, FID7 to FID6, FID4 to FID7, FID9 to FID8, FID5 to FID9
Other:
- sheet Power Management +BMS ports: added PG_3V3, PG_3V8; removed none

Commit message: v
Parts:
- renumbered FID3 to FID2, FID5 to FID3, FID7 to FID4, FID9 to FID5, FID4 to FID6, FID6 to FID7, FID2 to FID8, FID8 to FID9
Other:
- sheet MCU+WIFI+BT ports: added HEAT, PG_3V3, PG_3V8; removed none
- sheet Power Management +BMS ports: added HEAT; removed none

Commit message: v
Parts:
- FID2: value kicad -> KiCAD
- FID8: value scale -> Scale
Other:
- sheet MCU+WIFI+BT ports: added INT_EXTENDER, USB_OTG_D+, USB_OTG_D-; removed none
- sheet Other data+storage ports: added INT_EXTENDER, SCL, SDA, USB_OTG_D+, USB_OTG_D-; removed none
- note added: "All SMD caps ceramic are 0603 16V X7R or better unless other notes are made All SMD resistors are 0603 Stack up: 4 layer FR4 sig gnd gnd+sig sig Delata(T) aimed for is 20C or less"
- note removed: "All SMD caps ceramic are 0603 16V X7R or better unless other notes are made All SMD resistors are 0603 Stack up: 4 layer FR4 sig gnd gnd+sig sig All non power traces should aim to be 50 ohm single ended impedance unless other requirements are in place Delata(T) aimed for is 20C or less"

Commit message: f
Other:
- note added: "------------------- |I2C ADRESSES | ------------------- |BME280 0x76 | ------------------- |TLV320ADC3100 0x30 | ------------------- |TCA9554A 0x21 | ------------------- |INA3221 0x40 | ------------------- |TCA9545APWR 0x20 | -------------------"

Commit message: h
Parts:
- removed H6: M3, MountingHole:MountingHole_3.2mm_M3_ISO7380_Pad_TopBottom, symbol Mechanical:MountingHole_Pad
Other:
- sheet MCU+WIFI+BT ports: added CHG_EN; removed none
- sheet Power Management +BMS ports: added CHG_EN; removed none
