File: Bird_detector_V1/Bird_detector_V1.kicad_sch (KiCad schematic)
At the start: 15 parts

Commit message: b
Other:
- title: (none) -> Bird Detection and Recognition System
Changed lines of the file:
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@@
 (kicad_sch (version 20211123) (generator eeschema)
   (paper "A3")
+  (title_block
+    (title "Bird Detection and Recognition System")
+    (rev "V0.1")
+  )
   (junction (at 379.73 171.45) (diameter 0) (color 0 0 0 0)
   )
@@
       (reference "#PWR0219") (unit 1) (value "GND") (footprint "")
     )
-    (path "/94b5dc3a-5793-40ef-bc39-7863e8733196/d3ba6849-323c-47dd-8776-a0c87bca3b0c/7294281e-976a-4aeb-9034-756fb3c8fcb8"
-      (reference "#PWR0220") (unit 1) (value "+3V3") (footprint "")
-    )
-    (path "/94b5dc3a-5793-40ef-bc39-7863e8733196/d3ba6849-323c-47dd-8776-a0c87bca3b0c/9ad98729-5d44-4d9b-bb3b-863273e099b5"
-      (reference "#PWR0221") (unit 1) (value "+3V3") (footprint "")
-    )
     (path "/94b5dc3a-5793-40ef-bc39-7863e8733196/d3ba6849-323c-47dd-8776-a0c87bca3b0c/a4b049ce-1f56-488c-9ffa-b2ff362e1177"
       (reference "#PWR0222") (unit 1) (value "GND") (footprint "")
     )
-    (path "/94b5dc3a-5793-40ef-bc39-7863e8733196/d3ba6849-323c-47dd-8776-a0c87bca3b0c/448360a9-d77e-40fa-8c06-e6112ed173b7"
-      (reference "#PWR0223") (unit 1) (value "+3V3") (footprint "")
-    )
-    (path "/94b5dc3a-5793-40ef-bc39-7863e8733196/d3ba6849-323c-47dd-8776-a0c87bca3b0c/8836b1d8-ae97-4ec7-9ac1-0443d2ace691"
-      (reference "#PWR0225") (unit 1) (value "+3V3") (footprint "")
+    (path "/94b5dc3a-5793-40ef-bc39-7863e8733196/41f92477-07aa-4f31-92b2-b9a504643ddc"
+      (reference "#PWR0224") (unit 1) (value "GND") (footprint "")
     )
     (path "/94b5dc3a-5793-40ef-bc39-7863e8733196/d3ba6849-323c-47dd-8776-a0c87bca3b0c/2402a4e2-c33c-4741-83b5-542a448dda7c"
       (reference "#PWR0226") (unit 1) (value "GND") (footprint "")
     )
+    (path "/94b5dc3a-5793-40ef-bc39-7863e8733196/49cd66d3-b152-4450-89dc-fc6dc26c224a"
+      (reference "#PWR0227") (unit 1) (value "+3V3") (footprint "")
+    )
     (path "/94b5dc3a-5793-40ef-bc39-7863e8733196/d3ba6849-323c-47dd-8776-a0c87bca3b0c/2a44c078-f688-4ebd-aa93-473aeaf965d2"
       (reference "#PWR0228") (unit 1) (value "GND") (footprint "")
@@
       (reference "J17") (unit 1) (value "PCB CAP") (footprint "Z_mycustom_footprint_lib:PCB cap start")
     )
+    (path "/94b5dc3a-5793-40ef-bc39-7863e8733196/558a3f68-0ce3-41c3-bab1-ffdc35d1492e"
+      (reference "J18") (unit 1) (value "Conn_02x02_Odd_Even") (footprint "Connector_PinHeader_2.54mm:PinHeader_2x02_P2.54mm_Vertical_SMD")
+    )
     (path "/94b5dc3a-5793-40ef-bc39-7863e8733196/d3ba6849-323c-47dd-8776-a0c87bca3b0c/1f6e798f-90d9-4c46-b40c-241219b7f92f"

Commit message: f
Parts:
- added FID11, FID12: mouse bites, Z_mycustom_panelization:mouse bites 2mm wide 6mm long 0.6mm holes 0.3mm apart round edges, symbol Mechanical:Fiducial
Changed lines of the file:
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@@
+    )
+  )
+  (symbol (lib_id "Mechanical:Fiducial") (at 295.91 185.42 0) (unit 1)
+    (in_bom no) (on_board yes) (fields_autoplaced)
+    (property "Reference" "FID12" (id 0) (at 299.085 184.1499 0)
+      (effects (font (size 1.27 1.27)) (justify left))
+    )
+    (property "Value" "mouse bites" (id 1) (at 299.085 186.6899 0)
+      (effects (font (size 1.27 1.27)) (justify left))
+    )
+    (property "Footprint" "Z_mycustom_panelization:mouse bites 2mm wide   6mm long     0.6mm holes  0.3mm apart round edges" (id 2) (at 295.91 185.42 0)
+      (effects (font (size 1.27 1.27)) hide)
+    )
+    (property "Datasheet" "~" (id 3) (at 295.91 185.42 0)
+      (effects (font (size 1.27 1.27)) hide)
     )
   )
@@
     )
     (property "Datasheet" "~" (id 3) (at 316.23 166.37 0)
+      (effects (font (size 1.27 1.27)) hide)
+    )
+  )
+  (symbol (lib_id "Mechanical:Fiducial") (at 275.59 185.42 0) (unit 1)
+    (in_bom no) (on_board yes) (fields_autoplaced)
+    (property "Reference" "FID11" (id 0) (at 278.765 184.1499 0)
+      (effects (font (size 1.27 1.27)) (justify left))
+    )
+    (property "Value" "mouse bites" (id 1) (at 278.765 186.6899 0)
+      (effects (font (size 1.27 1.27)) (justify left))
+    )
+    (property "Footprint" "Z_mycustom_panelization:mouse bites 2mm wide   6mm long     0.6mm holes  0.3mm apart round edges" (id 2) (at 275.59 185.42 0)
+      (effects (font (size 1.27 1.27)) hide)
+    )
+    (property "Datasheet" "~" (id 3) (at 275.59 185.42 0)
       (effects (font (size 1.27 1.27)) hide)
     )
@@
       (reference "FID10") (unit 1) (value "Cell") (footprint "Z_mycustom_footprint_lib:18650 cell 3d model")
     )
+    (path "/a1a05b46-143d-41fc-bdff-1eea7cac84dd"
+      (reference "FID11") (unit 1) (value "mouse bites") (footprint "Z_mycustom_panelization:mouse bites 2mm wide   6mm long     0.6mm holes  0.3mm apart round edges")
+    )
+    (path "/14198894-f1d8-4279-8616-7868eeb7e852"
+      (reference "FID12") (unit 1) (value "mouse bites") (footprint "Z_mycustom_panelization:mouse bites 2mm wide   6mm long     0.6mm holes  0.3mm apart round edges")
+    )
     (path "/18ed1543-e14e-447a-872b-bcd85b6c55d3"
