File: Bird_detector_V1/Power.kicad_sch (KiCad schematic)
At the start: 0 parts

Commit message: g
Parts:
- added FB2: MH2029-401Y, Resistor_SMD:R_0805_2012Metric_Pad1.20x1.40mm_HandSolder, symbol Device:FerriteBead_Small
Changed lines of the file:
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@@
 (kicad_sch (version 20211123) (generator eeschema)
   (paper "A3")
+  (wire (pts (xy 48.26 38.1) (xy 48.26 40.64))
+    (stroke (width 0) (type default) (color 0 0 0 0))
+  )
+  (wire (pts (xy 45.72 38.1) (xy 45.72 40.64))
+    (stroke (width 0) (type default) (color 0 0 0 0))
+  )
+  (hierarchical_label "SCL" (shape input) (at 48.26 40.64 270)
+    (effects (font (size 1.27 1.27)) (justify right))
+  )
+  (hierarchical_label "SDA" (shape input) (at 45.72 40.64 270)
+    (effects (font (size 1.27 1.27)) (justify right))
+  )
+  (symbol (lib_id "Device:FerriteBead_Small") (at 74.93 68.58 90) (unit 1)
+    (in_bom yes) (on_board yes) (fields_autoplaced)
+    (property "Reference" "FB2" (id 0) (at 74.8919 62.23 90))
+    (property "Value" "MH2029-401Y" (id 1) (at 74.8919 64.77 90))
+    (property "Footprint" "Resistor_SMD:R_0805_2012Metric_Pad1.20x1.40mm_HandSolder" (id 2) (at 74.93 70.358 90)
+      (effects (font (size 1.27 1.27)) hide)
+    )
+    (property "Datasheet" "~" (id 3) (at 74.93 68.58 0)
+      (effects (font (size 1.27 1.27)) hide)
+    )
+    (pin "1")
+    (pin "2")
+  )
 )

Commit message: f
Parts:
- added C28, C29, C30, C31: 22u, Capacitor_SMD:C_0603_1608Metric_Pad1.08x0.95mm_HandSolder, symbol Device:C_Small
- added D8: D5V0P4UR6SO-7, SOT95P285X140-6N, symbol SamacSys_Parts:D5V0P4UR6SO-7
- added F1, F2, F3: Polyfuse_Small, symbol Device:Polyfuse_Small
- added J7: Conn_01x02, symbol Connector_Generic:Conn_01x02
- added J8: USB_A, Connector_USB:USB_A_Molex_105057_Vertical, symbol Connector:USB_A
- added L1: 1-1.5u, symbol Device:L
- added Q5, Q6: DMP2040USD, Package_SO:SO-8_3.9x4.9mm_P1.27mm, symbol My_custom_lib:DMP2040USD
- added R26, R27, R31, R36: 100k, symbol Device:R_Small
- added R28, R33: 1Meg, symbol Device:R_Small
- added R29, R37: 180k, symbol Device:R_Small
- added R30: 1k, symbol Device:R_Small
- added R32: 1.32Meg, symbol Device:R_Small
- added R34: 200k, symbol Device:R_Small
- added R35: 1.18Meg, symbol Device:R_Small
- added U7: APX810S05, Package_TO_SOT_SMD:SOT-23, symbol My_custom_lib:APX810S05
- added U8: TPS63020DSJR, Z_mycustom_footprint_lib:TPS63020, symbol My_custom_lib:TPS63020DSJR
Connections:
- net VBUS: now reaches FB2.1
- net VBUS: now also D8.5 (VCC), J8.1 (VBUS)
- net at FB2.2: now also F3.1
- new net: Q5.2 (G), R27.1
- new net: F2.1, J7.2 (Pin_2)
- new net: F2.2, Q6.3 (S)
- new net: Q5.4 (G), R26.1, U7.1 (RESET)
- new net: F1.2, Q5.3 (S), U7.3 (Vcc)
- new net: Q5.5 (D), Q5.6 (D), Q5.7 (D), Q5.8 (D)
- new net: R33.2, U8.14 (PG)
- new net: L1.2, U8.6 (L2), U8.7 (L2)
- new net: L1.1, U8.8 (L1), U8.9 (L1)
- new net: Q6.2 (G), R31.1
- new net: Q6.4 (G), R30.1
- new net: Q6.5 (D), Q6.6 (D), Q6.7 (D), Q6.8 (D)
- new net +3V8: R33.1, U8.4 (VOUT), U8.5 (VOUT)
- new net +5V: F3.2
- new net +BATT: F1.1
- new net +VDC: U8.1 (VINA), U8.10 (VIN), U8.11 (VIN), U8.12 (EN)
- new net D+: D8.6 (I/O4), J8.3 (D+)
- new net D-: D8.4 (I/O3), J8.2 (D-)
- new net GND: D8.2 (VSS), J7.1 (Pin_1), J8.4 (GND), R26.2, R27.2, R30.2, R31.2, R36.2, U7.2 (GND), U8.2 (GND)
- new net RF_SYNC: R36.1, U8.13 (PS/SYNC)
- no-connect marks 0 -> 3
Other:
- note added: "0.5v FB pin"
- note added: "3V8-4V"
- note added: "3v3"
- note added: "3v3 TVS goes here"
- moved on the sheet: FB2

Commit message: j
Parts:
- removed C30, C31: 22u, Capacitor_SMD:C_0603_1608Metric_Pad1.08x0.95mm_HandSolder, symbol Device:C_Small
- removed R32: 1.32Meg, symbol Device:R_Small
- removed R33: 1Meg, symbol Device:R_Small
- removed R34: 200k, symbol Device:R_Small
- removed R35: 1.18Meg, symbol Device:R_Small
- removed R36: 100k, symbol Device:R_Small
- removed R37: 180k, symbol Device:R_Small
- removed U8: TPS63020DSJR, Z_mycustom_footprint_lib:TPS63020, symbol My_custom_lib:TPS63020DSJR
- added C26, C? (x4): 100n, Capacitor_SMD:C_0603_1608Metric_Pad1.08x0.95mm_HandSolder, symbol Device:C_Small
- added C27: 10u+, Capacitor_SMD:C_0603_1608Metric_Pad1.08x0.95mm_HandSolder, symbol Device:C_Small
- added C?: 22u+, Capacitor_SMD:C_0603_1608Metric_Pad1.08x0.95mm_HandSolder, symbol Device:C_Small
- added D8, D9: LED_Small, LED_SMD:LED_0603_1608Metric_Pad1.05x0.95mm_HandSolder, symbol Device:LED_Small
- added J?: 140-502-415-000, 140502415000, symbol SamacSys_Parts:140-502-415-000
- added JP3: leds, Connector_PinHeader_2.54mm:PinHeader_1x03_P2.54mm_Vertical, symbol Jumper:Jumper_3_Bridged12
- added JP?: ADR1, Jumper:SolderJumper-3_P1.3mm_Bridged12_RoundedPad1.0x1.5mm_NumberLabels, symbol Jumper:SolderJumper_3_Bridged12
- added R26, R? (x3): 50m, Resistor_SMD:R_0805_2012Metric, symbol Device:R_Small
- added R27: 100K, Resistor_SMD:R_0603_1608Metric_Pad0.98x0.95mm_HandSolder, symbol Device:R_Small
- added R30: 10k, Resistor_SMD:R_0603_1608Metric_Pad0.98x0.95mm_HandSolder, symbol Device:R_Small
- added R?: 100k, Resistor_SMD:R_0603_1608Metric_Pad0.98x0.95mm_HandSolder, symbol Device:R_Small
- added SW?: BMS_RESET, SamacSys_Parts:PTS526SK15SMTR2LFS, symbol Switch:SW_SPST
- added U7: MP2615, SamacSys_Parts:MP2615GQZ, symbol My_custom_lib:MP2615
- added U?: INA3221, Package_DFN_QFN:Texas_RGV_S-PVQFN-N16_EP2.1x2.1mm, symbol Power_Management:INA3221
- C28, C29: value 22u -> 1u
- D10: renamed from D8; footprint SOT95P285X140-6N -> SamacSys_Parts:SOT95P285X140-6N
- F2: value Polyfuse_Small -> 2A
- J7: value Conn_01x02 -> ntc 10k
- L1: value 1-1.5u -> x
- R28: value 1Meg -> 1k; footprint (none) -> Resistor_SMD:R_0603_1608Metric_Pad0.98x0.95mm_HandSolder
- R29: value 180k -> 1k; footprint (none) -> Resistor_SMD:R_0603_1608Metric_Pad0.98x0.95mm_HandSolder
- R31: renamed from R26; footprint (none) -> Resistor_SMD:R_0603_1608Metric_Pad0.98x0.95mm_HandSolder
- R32: renamed from R27; footprint (none) -> Resistor_SMD:R_0603_1608Metric_Pad0.98x0.95mm_HandSolder
- R33: renamed from R30; footprint (none) -> Resistor_SMD:R_0603_1608Metric_Pad0.98x0.95mm_HandSolder
- R34: renamed from R31; footprint (none) -> Resistor_SMD:R_0603_1608Metric_Pad0.98x0.95mm_HandSolder
- renumbered J8 to J9, U7 to U8
Connections:
- net +5V: now also C?.2, R?.2, U?.11 (IN-1); no longer F3.2
- net +BATT: now also Q6.3 (S), C27.1, C?.2, R26.2, R?.2, U7.9 (BATT), U?.14 (IN-2)
- net GND: now also C28.2, C29.2, J7.2 (Pin_2), C27.2, C?.2, C?.2, J?.1, JP?.3 (B), R27.2, U7.16 (PGND), U7.8 (AGND), U?.17 (EP), U?.3 (GND); no longer J7.1 (Pin_1)
- net SCL: now also U?.6 (SCL)
- net SDA: now also U?.7 (SDA)
- net VCC: now reaches C28.1
- net VCC: now also R30.2, R?.1, SW?.2 (B), U7.3 (VCC), U7.4 (CELL)
- net at F2.1: now also J?.2; no longer J7.2 (Pin_2)
- net IN_SOLAR+: now reaches F2.2
- net IN_SOLAR+: now also C?.1, R?.1, U?.15 (IN+2); no longer Q6.3 (S)
- net at L1.2: now also R26.1, U7.10 (CSP)
- net at L1.1: now also C26.1, U7.1 (SW)
- net at C29.1: now also U7.14 (TMR)
- net at R29.1: now also U7.12 (~{ACOK})
- net at R29.2: now also D9.1 (K)
- net at R28.1: now also U7.11 (~{CHGOK})
- net at R28.2: now also D8.1 (K)
- new net: JP?.2 (C), U?.5 (A0)
- new net: R?.2, U7.5 (SEL)
- new net: D8.2 (A), D9.2 (A), JP3.2 (C)
- new net: C26.2, U7.15 (BST)
- new net: J7.1 (Pin_1), R30.1, U7.13 (NTC)
- new net +3V3: C?.1, JP?.1 (A), U?.4 (VS)
- new net IN_SYSTEM+: C?.2, R?.1, U?.2 (IN+3)
- new net IN_SYSTEM-: C?.1, C?.1, JP3.1 (A), R?.2, U7.2 (VIN), U?.1 (IN-3)
- new net IN_USB_+: C?.1, F3.2, R?.1, U?.12 (IN+1)
- new net ~{EN}: R27.1, SW?.1 (A), U7.6 (~{EN})
- no-connect marks 3 -> 9
Other:
- added sheet SMPSs (SMPSs.kicad_sch)
- note added: "0.2W max"
- note added: "4.5-18V absolute max input Buck only"
- note added: "Adress: 100000[A0]"
- note added: "CELL: 1 short to VCC for single cell OR 2 connect to GND for 2 cell SEL: 1 pull up for 4.1V (longer cell live) 2 pull down or float for 4.2V (more storage)"
- note added: "CHGOK: Charging completion indicator. When this pin goes logic low, the device is charging. The pin becomes an open drain once the charge is completed or suspended. ACOK: Valid input supply indicator. A logic low on this pin indicates the presence of a valid input power supply."
- note added: "MAX 150mV on shunt"
- note added: "Solar input"
- note added: "T_p (seconds) = 0.46 X C (uF) t_trickle (minutes) = 62.8 X C (uF)"
- note added: "switching frequency 760KHz Inductor: DC resistance less than 50mΩ"
- note removed: "0.5v FB pin"
- note removed: "3V8-4V"
- note removed: "3v3"
- moved on the sheet: D10, F1, F2, F3, FB2, J9, Q5A, Q5B, Q6A, Q6B, R31, R32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

Commit message: f
Parts:
- removed F1: Polyfuse_Small, symbol Device:Polyfuse_Small
- removed F2: 2A, symbol Device:Polyfuse_Small
- added F? (x2): PPTC 2A 16V, Fuse:Fuse_1812_4532Metric_Pad1.30x3.40mm_HandSolder, symbol Device:Polyfuse_Small
- F3: value Polyfuse_Small -> PPTC 2A 16V; footprint (none) -> Fuse:Fuse_1812_4532Metric_Pad1.30x3.40mm_HandSolder
- J10: renamed from J?; footprint 140502415000 -> SamacSys_Parts:140502415000
- J9: renamed from J7; footprint (none) -> Connector_PinSocket_2.54mm:PinSocket_1x02_P2.54mm_Vertical
- gave numbers to parts that had none: 12
- renumbered C26 to C27, C27 to C29, C28 to C30, C29 to C31, J9 to J11, Q5 to Q6, Q6 to Q7, R26 to R31, R27 to R32, R28 to R33, R29 to R34, R31 to R36, R32 to R37, R30 to R38, R33 to R40, R34 to R41, U7 to U6, U8 to U7
Connections:
- net +BATT: now also F?.1
- net IN_SOLAR+: now also F?.2
- net at J10.2: now also F?.1
- net at Q6.3 (S), U7.3 (Vcc): now also F?.2
Other:
- sheet SMPSs ports: added RF_SYNC; removed none

Commit message: R
Parts:
- added D10, D11: MMSZ5245B, Diode_SMD:D_SOD-123, symbol Device:D_Zener
- added D12: LED_Small, LED_SMD:LED_0603_1608Metric_Pad1.05x0.95mm_HandSolder, symbol Device:LED_Small
- added J10: backup, TerminalBlock:TerminalBlock_Altech_AK300-2_P5.00mm, symbol Connector:Screw_Terminal_01x02
- added R40: 1k, Resistor_SMD:R_0603_1608Metric_Pad0.98x0.95mm_HandSolder, symbol Device:R_Small
- L1: value x -> 6u8
- gave numbers to parts that had none: 2
- renumbered D10 to D13, J10 to J11, J11 to J12, R40 to R41, R41 to R42, R42 to R43
Connections:
- net +BATT: no longer C32.2, Q7.3 (S), R39.2, U8.14 (IN-2)
- net GND: now also D10.2 (A), D11.2 (A), D12.2 (A), J10.1 (Pin_1)
- net at F2.1, J11.2: now also J10.2 (Pin_2), R40.1
- new net: D12.1 (K), R40.2
- new net IN_SOLAR-: C32.2, D10.1 (K), D11.1 (K), Q7.3 (S), R39.2, U8.14 (IN-2)
Other:
- note added: "************************************** * Model Generated by MODPEX * *Copyright(c) Symmetry Design Systems* * All Rights Reserved * * UNPUBLISHED LICENSED SOFTWARE * * Contains Proprietary Information * * Which is The Property of * * SYMMETRY OR ITS LICENSORS * *Commercial Use or Resale Restricted * * by Symmetry License Agreement * ************************************** * Model generated on Jul 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"
- note added: "15V 1W total"
- note added: "Reverse Voltage Protection +Indicator(0.17W R at 15V) &Over Voltage Protection &Overcurrent Protection (Short Circuit too)"
- moved on the sheet: C32, C33, F2, J11, JP4, Q7A, Q7B, R39, R41, R42, U8

Commit message: v
Parts:
- L1: footprint (none) -> Z_mycustom_footprint_lib:inductor 6x6mm
- renumbered C26 to C37, C27 to C38, C28 to C39, C29 to C40, C30 to C41, C31 to C42, C32 to C43, C33 to C44, C34 to C45, D8 to D10, D9 to D11, D10 to D12, D11 to D13, D12 to D14, D13 to D15, JP3 to JP5, JP4 to JP6, Q6 to Q7, Q7 to Q8, R30 to R49, R31 to R50, R32 to R51, R33 to R52, R34 to R53, R35 to R54, R36 to R55, R37 to R56, R38 to R57, R39 to R58, R40 to R59, R41 to R60, R42 to R61, R43 to R62, SW2 to SW3, U8 to U10, U6 to U8, U7 to U9
Connections:
- net CSP: now reaches L1.2, R50.1, U8.10 (CSP)
- net SEL: now reaches R54.2, U8.5 (SEL)
- net BMS_LED: now reaches D10.2 (A), D11.2 (A), JP5.2 (C)
- net SW: now reaches C38.1, L1.1, U8.1 (SW)
- net BST: now reaches C38.2, U8.15 (BST)
- net NTC: now reaches J9.1 (Pin_1), R57.1, U8.13 (NTC)
- net TMR: now reaches C42.1, U8.14 (TMR)
