File: Bird_detector_V1/Power.kicad_sch (KiCad schematic)
At the start: 47 parts, among them J10 backup, J11 140-502-415-000, J12 USB_A, J9 ntc 10k, Q7 DMP2040USD, Q8 DMP2040USD, SW3 BMS_RESET, U10 INA3221, U8 MP2615, U9 APX810S05

Commit message: f
Parts:
- removed C38: 100n, Capacitor_SMD:C_0603_1608Metric_Pad1.08x0.95mm_HandSolder, symbol Device:C_Small
- removed C39: 22u+, Capacitor_SMD:C_0603_1608Metric_Pad1.08x0.95mm_HandSolder, symbol Device:C_Small
- removed C40: 10u+, Capacitor_SMD:C_0603_1608Metric_Pad1.08x0.95mm_HandSolder, symbol Device:C_Small
- removed D10, D11: LED_Small, LED_SMD:LED_0603_1608Metric_Pad1.05x0.95mm_HandSolder, symbol Device:LED_Small
- removed J9: ntc 10k, Connector_PinSocket_2.54mm:PinSocket_1x02_P2.54mm_Vertical, symbol Connector_Generic:Conn_01x02
- removed JP5: leds, Connector_PinHeader_2.54mm:PinHeader_1x03_P2.54mm_Vertical, symbol Jumper:Jumper_3_Bridged12
- removed R50: 50m, Resistor_SMD:R_0805_2012Metric, symbol Device:R_Small
- removed R51: 100K, Resistor_SMD:R_0603_1608Metric_Pad0.98x0.95mm_HandSolder, symbol Device:R_Small
- removed R52, R53: 1k, Resistor_SMD:R_0603_1608Metric_Pad0.98x0.95mm_HandSolder, symbol Device:R_Small
- removed R54: 100k, Resistor_SMD:R_0603_1608Metric_Pad0.98x0.95mm_HandSolder, symbol Device:R_Small
- removed SW3: BMS_RESET, SamacSys_Parts:PTS526SK15SMTR2LFS, symbol Switch:SW_SPST
- removed U8: MP2615, SamacSys_Parts:MP2615GQZ, symbol My_custom_lib:MP2615
- added C43: 220n, Capacitor_SMD:C_0603_1608Metric_Pad1.08x0.95mm_HandSolder, symbol Device:C_Small
- added C45: 22u, Capacitor_SMD:C_0603_1608Metric_Pad1.08x0.95mm_HandSolder, symbol Device:C_Small
- added D14, D15: LED_Small, LED_SMD:LED_0603_1608Metric_Pad1.05x0.95mm_HandSolder, symbol Device:LED_Small
- added D16: D_Schottky, symbol Device:D_Schottky
- added Q9: Q_PMOS_DGS, symbol Device:Q_PMOS_DGS
- added R58: 100k, Resistor_SMD:R_0603_1608Metric_Pad0.98x0.95mm_HandSolder, symbol Device:R_Small
- added R59: X, Resistor_SMD:R_0603_1608Metric_Pad0.98x0.95mm_HandSolder, symbol Device:R_Small
- added R60: 120, Resistor_SMD:R_0603_1608Metric_Pad0.98x0.95mm_HandSolder, symbol Device:R_Small
- added R61: 50m, Resistor_SMD:R_0805_2012Metric, symbol Device:R_Small
- C41: value 1u -> 10u
- C42: value 1u -> 100n
- L1: value 6u8 -> 12u; footprint Z_mycustom_footprint_lib:inductor 6x6mm -> Inductor_SMD:L_Wuerth_MAPI-3012
- R57: value 10k -> 100k
- gave numbers to parts that had none: 1
- renumbered C45 to C38, C43 to C39, C37 to C40, D14 to D10, D12 to D11, D13 to D12, D15 to D13, F3 to F2, F2 to F3, J11 to J10, J10 to J11, J12 to J9, R59 to R49, R62 to R50, R58 to R51, R55 to R52, R56 to R53, R60 to R54, R61 to R55, R49 to R56, U10 to U11
Connections:
- net CSP is gone; now on an unnamed net: L1.2
- net NTC is gone; now on net IN_SYSTEM-: R57.1
- net TMR is gone; now on an unnamed net: C42.1
- net +BATT: now also U10.7 (BAT), C45.1, R61.2
- net GND: now also U10.2 (GND), C43.2, C45.2, D16.2 (A), R58.2; no longer C42.2
- net IN_SYSTEM+: now also Q8.1 (S)
- net IN_SYSTEM-: now also C41.1, C42.2, U10.9 (VCC), Q9.3 (S), R59.2
- net at U10.10 (DRV): now also Q9.2 (G)
- net at U10.3 (~{CHRG}): now also D14.1 (K)
- net at U10.4 (~{DONE}): now also D15.1 (K)
- net at U10.5 (COM): now also R60.2
- net at U10.6 (MPPT): now also R57.2, R58.1
- net at U10.8 (CSP): now also R61.1
- net SW: no longer names the net of L1.1
- net SW: now also D16.1 (K), Q9.1 (D)
- removed net VCC: C41.1, R57.2
- new net: D14.2 (A), D15.2 (A), R59.1
- new net: C43.1, R60.1
- no-connect marks 9 -> 8
Other:
- sheet SMPSs ports: added PG_3V3, PG_3V8; removed none
- note added: "1.205V at MPPT"
- note added: "4.5-28V input"
- note added: "5.5V MPPT for seed studio solar"
- note removed: "0.2W max"
- note removed: "4.5-18V absolute max input Buck only"
- note removed: "CELL: 1 short to VCC for single cell OR 2 connect to GND for 2 cell SEL: 1 pull up for 4.1V (longer cell live) 2 pull down or float for 4.2V (more storage)"
- note removed: "CHGOK: Charging completion indicator. When this pin goes logic low, the device is charging. The pin becomes an open drain once the charge is completed or suspended. ACOK: Valid input supply indicator. A logic low on this pin indicates the presence of a valid input power supply."
- note removed: "T_p (seconds) = 0.46 X C (uF) t_trickle (minutes) = 62.8 X C (uF)"
- note removed: "switching frequency 760KHz Inductor: DC resistance less than 50mΩ"
- moved on the sheet: C39, C40, D10, D11, D12, F1, F3, J10, J11, Q7A, Q7B, Q8A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

Commit message: v
Parts:
- removed J11: backup, TerminalBlock:TerminalBlock_Altech_AK300-2_P5.00mm, symbol Connector:Screw_Terminal_01x02
- removed Q9: Q_PMOS_DGS, symbol Device:Q_PMOS_DGS
- added C46: 10u, Capacitor_SMD:C_0603_1608Metric_Pad1.08x0.95mm_HandSolder, symbol Device:C_Small
- added C49: 22u, Capacitor_SMD:C_0603_1608Metric_Pad1.08x0.95mm_HandSolder, symbol Device:C_Small
- added C50: 1u, Capacitor_SMD:C_0603_1608Metric_Pad1.08x0.95mm_HandSolder, symbol Device:C_Small
- added C51: 3.5n, Capacitor_SMD:C_0603_1608Metric_Pad1.08x0.95mm_HandSolder, symbol Device:C_Small
- added C53: 100n, Capacitor_SMD:C_0603_1608Metric_Pad1.08x0.95mm_HandSolder, symbol Device:C_Small
- added D10, D18: SX33L_R1_00001, Diode_SMD:D_SMA_Handsoldering, symbol Device:D_Schottky
- added J11: Solar input, TerminalBlock:TerminalBlock_Altech_AK300-3_P5.00mm, symbol Connector:Screw_Terminal_01x03
- added J14: batt input, TerminalBlock:TerminalBlock_Altech_AK300-3_P5.00mm, symbol Connector:Screw_Terminal_01x03
- added Q10: SSM6N7002, Package_TO_SOT_SMD:SOT-363_SC-70-6_Handsoldering, symbol Device:Q_Dual_NMOS_S1G1D2S2G2D1
- added Q7, Q9: DMP3028LSD, Package_SO:SO-8_3.9x4.9mm_P1.27mm, symbol My_custom_lib:DMP2040USD
- added R63: 45, Resistor_SMD:R_0603_1608Metric_Pad0.98x0.95mm_HandSolder, symbol Device:R_Small
- added R65, R82: 1k, Resistor_SMD:R_0603_1608Metric_Pad0.98x0.95mm_HandSolder, symbol Device:R_Small
- added R71: 10k, Resistor_SMD:R_0603_1608Metric_Pad0.98x0.95mm_HandSolder, symbol Device:R_Small
- added R73: 64k, Resistor_SMD:R_0603_1608Metric_Pad0.98x0.95mm_HandSolder, symbol Device:R_Small
- added R74, R75: 100k, Resistor_SMD:R_0603_1608Metric_Pad0.98x0.95mm_HandSolder, symbol Device:R_Small
- added R76, R77, R79, R80: 50k+, Resistor_SMD:R_0603_1608Metric_Pad0.98x0.95mm_HandSolder, symbol Device:R_Small
- added TH1, TH2: 100k, Resistor_SMD:R_1812_4532Metric_Pad1.30x3.40mm_HandSolder, symbol Device:Thermistor_NTC
- added U13: MAX11601, Package_TO_SOT_SMD:SOT-23-8_Handsoldering, symbol My_custom_lib:MAX11601
- D11: renamed from D16; value D_Schottky -> SX33L_R1_00001; footprint (none) -> Diode_SMD:D_SMA_Handsoldering
- L1: value 12u -> 15u; footprint Inductor_SMD:L_Wuerth_MAPI-3012 -> Z_mycustom_footprint_lib:L_SMD_3131_(8080_metric)
- Q11: renamed from Q7; value DMP2040USD -> DMP3028LSD
- Q8: value DMP2040USD -> DMP3028LSD
- R69: renamed from R57; value 100k -> 1Meg
- R72: renamed from R58; value 100k -> 280.5587k
- renumbered C39 to C44, C42 to C45, C41 to C47, C45 to C48, C43 to C52, C44 to C54, C38 to C55, C40 to C56, D11 to D12, D12 to D13, D10 to D14, D14 to D15, D15 to D16, D13 to D17, F3 to F1, F1 to F3, J10 to J12, J9 to J13, JP6 to JP5, R51 to R61, R61 to R62, R49 to R64, R54 to R66, R55 to R67, R59 to R68, R60 to R70, R50 to R78, R56 to R81, R52 to R83, R53 to R84, U10 to U12, U11 to U14, U9 to U15
Connections:
- net +3V3: now also C53.1, R76.2, R77.2, U13.8 (Vdd)
- net +5V: now also Q11.2 (G), Q8.2 (G), R67.1, R84.1, D10.2 (A), D18.2 (A), Q10.2 (G), Q9.5 (D), Q9.6 (D), Q9.7 (D), Q9.8 (D), R74.2
- net +BATT: now also C49.1, C50.1, J14.2 (Pin_2)
- net +VDC: now also C56.2, R81.1, U14.2 (IN+3)
- net GND: now also C46.1, C49.2, C50.2, C51.2, C53.2, J11.1 (Pin_1), J14.1 (Pin_1), Q10.1 (S), Q10.4 (S), R65.2, R73.1, R74.1, R75.1, R79.1, R80.1, R82.2, U13.7 (GND); no longer R72.2
- net IN_SYSTEM-: now also Q11.1 (S), D18.1 (K), Q9.3 (S); no longer C45.2, C47.1, R68.2, R69.1, U12.9 (VCC)
- net SCL: now also U13.5 (SCL)
- net SDA: now also U13.6 (SDA)
- net at U12.10 (DRV): now also Q7.4 (G)
- net at F1.1, J12.2, R64.1: now also J11.2 (Pin_2)
- net at D11.1 (K), L1.1: now also Q7.5 (D), Q7.6 (D), R63.2
- removed net IN_SYSTEM+: C56.2, Q8.1 (S), R81.1, U14.2 (IN+3)
- new net: Q10.5 (G), Q10.6 (D), R71.1, R75.2
- new net: Q10.3 (D), R72.2, R73.2
- new net: Q9.4 (G), R82.1
- new net: R77.1, TH2.1
- new net: R76.1, TH1.1
- new net: Q9.2 (G), R65.1
- new net: C51.1, R63.1
- new net HEAT: Q7.2 (G)
- new net Heater_Input: J14.3 (Pin_3), Q7.7 (D), Q7.8 (D)
- new net Temp1: R79.2, TH1.2, U13.1 (AIN0)
- new net Temp2: R80.2, TH2.2, U13.2 (AIN1)
- new net VDC: C45.2, C46.2, C47.1, D10.1 (K), Q7.1 (S), Q7.3 (S), Q8.1 (S), Q9.1 (S), R68.2, R69.1, R71.2, U12.9 (VCC)
- no-connect marks 8 -> 11
Other:
- note added: "for the heater?"
- note added: "snubber"
- note removed: "************************************** * Model Generated by MODPEX * *Copyright(c) Symmetry Design Systems* * All Rights Reserved * * UNPUBLISHED LICENSED SOFTWARE * * Contains Proprietary Information * * Which is The Property of * * SYMMETRY OR ITS LICENSORS * *Commercial Use or Resale Restricted * * by Symmetry License Agreement * ************************************** * Model generated on Jul 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"
- moved on the sheet: C44, C45, C47, C48, C52, C54, C55, C56, D11, D12, D13, D14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

Commit message: v
Parts:
- removed J12: 140-502-415-000, SamacSys_Parts:140502415000, symbol SamacSys_Parts:140-502-415-000
- J13: footprint Connector_USB:USB_A_Molex_105057_Vertical -> SamacSys_Parts:USB1040GFLB
Connections:
- net BMS_SW_OUT: now reaches D11.1 (K), L1.1, Q7.5 (D), Q7.6 (D), R63.2
- net COM: now reaches R70.2, U12.5 (COM)
- net MPPT: now reaches R69.2, R72.1, U12.6 (MPPT)
- net CSP: now reaches L1.2, R62.1, U12.8 (CSP)
- net COM_CAP: now reaches C52.1, R70.1
Changed lines of the file:
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@@
   (junction (at 278.13 71.12) (diameter 0) (color 0 0 0 0)
   )
-  (junction (at 35.56 53.34) (diameter 0) (color 0 0 0 0)
-  )
   (junction (at 137.16 231.14) (diameter 0) (color 0 0 0 0)
   )
@@
   )
   (junction (at 170.18 48.26) (diameter 0) (color 0 0 0 0)
-  )
-  (junction (at 43.18 48.26) (diameter 0) (color 0 0 0 0)
   )
   (junction (at 53.34 104.14) (diameter 0) (color 0 0 0 0)
@@
     (stroke (width 0) (type default) (color 0 0 0 0))
   )
-  (wire (pts (xy 35.56 53.34) (xy 35.56 55.88))
+  (wire (pts (xy 40.64 41.91) (xy 40.64 44.45))
     (stroke (width 0) (type default) (color 0 0 0 0))
   )
@@
     (stroke (width 0) (type default) (color 0 0 0 0))
   )
-  (wire (pts (xy 370.84 199.39) (xy 373.38 199.39))
+  (wire (pts (xy 370.84 199.39) (xy 382.27 199.39))
     (stroke (width 0) (type default) (color 0 0 0 0))
   )
@@
     (stroke (width 0) (type default) (color 0 0 0 0))
   )
-  (wire (pts (xy 35.56 48.26) (xy 43.18 48.26))
-    (stroke (width 0) (type default) (color 0 0 0 0))
-  )
   (wire (pts (xy 45.72 170.18) (xy 53.34 170.18))
     (stroke (width 0) (type default) (color 0 0 0 0))
@@
     (stroke (width 0) (type default) (color 0 0 0 0))
   )
-  (wire (pts (xy 35.56 53.34) (xy 40.64 53.34))
-    (stroke (width 0) (type default) (color 0 0 0 0))
-  )
   (wire (pts (xy 374.65 48.26) (xy 378.46 48.26))
     (stroke (width 0) (type default) (color 0 0 0 0))
@@
     (stroke (width 0) (type default) (color 0 0 0 0))
   )
-  (wire (pts (xy 40.64 41.91) (xy 40.64 53.34))
-    (stroke (width 0) (type default) (color 0 0 0 0))
-  )
   (wire (pts (xy 209.55 123.19) (xy 207.01 123.19))
     (stroke (width 0) (type default) (color 0 0 0 0))
@@
     (stroke (width 0) (type default) (color 0 0 0 0))
   )
-  (wire (pts (xy 66.04 120.65) (xy 68.58 120.65))
+  (wire (pts (xy 66.04 120.65) (xy 81.28 120.65))
     (stroke (width 0) (type default) (color 0 0 0 0))
   )
@@
     (stroke (width 0) (type default) (color 0 0 0 0))
   )
-  (wire (pts (xy 35.56 50.8) (xy 35.56 53.34))
-    (stroke (width 0) (type default) (color 0 0 0 0))
-  )
   (wire (pts (xy 199.39 57.15) (xy 203.2 57.15))
     (stroke (width 0) (type default) (color 0 0 0 0))
@@
     (stroke (width 0) (type default) (color 0 0 0 0))
   )
-  (wire (pts (xy 370.84 196.85) (xy 373.38 196.85))
+  (wire (pts (xy 370.84 196.85) (xy 382.27 196.85))
     (stroke (width 0) (type default) (color 0 0 0 0))
   )
@@
     (stroke (width 0) (type default) (color 0 0 0 0))
   )
-  (wire (pts (xy 66.04 123.19) (xy 68.58 123.19))
+  (wire (pts (xy 66.04 123.19) (xy 81.28 123.19))
     (stroke (width 0) (type default) (color 0 0 0 0))
   )
@@
     (effects (font (size 1.27 1.27)) (justify left bottom))
   )
+  (label "SDA" (at 74.93 123.19 0)
+    (effects (font (size 1.27 1.27)) (justify left bottom))
+  )
   (label "Heater_Input" (at 233.68 25.4 0)
     (effects (font (size 1.27 1.27)) (justify left bottom))
   )
+  (label "COM" (at 323.85 93.98 0)
+    (effects (font (size 1.27 1.27)) (justify left bottom))
+  )
   (label "Heater_Input" (at 33.02 228.6 0)
     (effects (font (size 1.27 1.27)) (justify left bottom))
   )
+  (label "COM_CAP" (at 336.55 93.98 0)
+    (effects (font (size 1.27 1.27)) (justify left bottom))
+  )
+  (label "SDA" (at 373.38 196.85 0)
+    (effects (font (size 1.27 1.27)) (justify left bottom))
+  )
   (label "Temp2" (at 34.29 120.65 180)
     (effects (font (size 1.27 1.27)) (justify right bottom))
+  )
+  (label "CSP" (at 353.06 81.28 0)
+    (effects (font (size 1.27 1.27)) (justify left bottom))
+  )
+  (label "SCL" (at 74.93 120.65 0)
+    (effects (font (size 1.27 1.27)) (justify left bottom))
+  )
+  (label "SCL" (at 373.38 199.39 0)
+    (effects (font (size 1.27 1.27)) (justify left bottom))
+  )
+  (label "BMS_SW_OUT" (at 334.01 48.26 0)
+    (effects (font (size 1.27 1.27)) (justify left bottom))
+  )
+  (label "MPPT" (at 264.16 93.98 0)
+    (effects (font (size 1.27 1.27)) (justify left bottom))
   )
   (global_label "IN_SOLAR+" (shape input) (at 342.9 191.77 180) (fields_autoplaced)
@@
     )
   )
-  (hierarchical_label "SDA" (shape input) (at 68.58 123.19 0)
+  (hierarchical_label "SDA" (shape input) (at 81.28 123.19 0)
     (effects (font (size 1.27 1.27)) (justify left))
   )
-  (hierarchical_label "SCL" (shape input) (at 373.38 199.39 0)
+  (hierarchical_label "SCL" (shape input) (at 382.27 199.39 0)
     (effects (font (size 1.27 1.27)) (justify left))
   )
@@
     (effects (font (size 1.27 1.27)) (justify left))
   )
-  (hierarchical_label "SDA" (shape input) (at 373.38 196.85 0)
+  (hierarchical_label "SDA" (shape input) (at 382.27 196.85 0)
     (effects (font (size 1.27 1.27)) (justify left))
   )
@@
     (effects (font (size 1.27 1.27)) (justify left))
   )
-  (hierarchical_label "SCL" (shape input) (at 68.58 120.65 0)
+  (hierarchical_label "SCL" (shape input) (at 81.28 120.65 0)
     (effects (font (size 1.27 1.27)) (justify left))
   )
@@
     (property "Reference" "J13" (id 0) (at 35.56 161.925 0))
     (property "Value" "USB_A" (id 1) (at 35.56 164.465 0))
-    (property "Footprint" "Connector_USB:USB_A_Molex_105057_Vertical" (id 2) (at 39.37 176.53 0)
+    (property "Footprint" "SamacSys_Parts:USB1040GFLB" (id 2) (at 39.37 176.53 0)
       (effects (font (size 1.27 1.27)) hide)
     )
@@
     (pin "1")
   )
-  (symbol (lib_id "power:GND") (at 35.56 55.88 0) (unit 1)
-    (in_bom yes) (on_board yes) (fields_autoplaced)
-    (property "Reference" "#PWR0130" (id 0) (at 35.56 62.23 0)
-      (effects (font (size 1.27 1.27)) hide)
-    )
-    (property "Value" "GND" (id 1) (at 35.56 60.96 0)
-      (effects (font (size 1.27 1.27)) hide)
-    )
-    (property "Footprint" "" (id 2) (at 35.56 55.88 0)
-      (effects (font (size 1.27 1.27)) hide)
-    )
-    (property "Datasheet" "" (id 3) (at 35.56 55.88 0)
+  (symbol (lib_id "power:GND") (at 40.64 44.45 0) (unit 1)
+    (in_bom yes) (on_board yes) (fields_autoplaced)
+    (property "Reference" "#PWR0130" (id 0) (at 40.64 50.8 0)
+      (effects (font (size 1.27 1.27)) hide)
+    )
+    (property "Value" "GND" (id 1) (at 40.64 49.53 0)
+      (effects (font (size 1.27 1.27)) hide)
+    )
+    (property "Footprint" "" (id 2) (at 40.64 44.45 0)
+      (effects (font (size 1.27 1.27)) hide)
+    )
+    (property "Datasheet" "" (id 3) (at 40.64 44.45 0)
       (effects (font (size 1.27 1.27)) hide)
     )
@@
     (pin "1")
   )
-  (symbol (lib_id "SamacSys_Parts:140-502-415-000") (at 35.56 50.8 180) (unit 1)
-    (in_bom yes) (on_board yes) (fields_autoplaced)
-    (property "Reference" "J12" (id 0) (at 25.4 40.64 0))
-    (property "Value" "140-502-415-000" (id 1) (at 25.4 43.18 0))
-    (property "Footprint" "SamacSys_Parts:140502415000" (id 2) (at 19.05 53.34 0)
-      (effects (font (size 1.27 1.27)) (justify left) hide)
-    )
-    (property "Datasheet" "https://files.edac.net/edac/content/140/140-502-415-000%20-%20EDAC%20E-MATE%20(Pin%20Header)%20Connector.PDF" (id 3) (at 19.05 50.8 0)
-      (effects (font (size 1.27 1.27)) (justify left) hide)
-    )
-    (property "Description" "EDAC - 140-502-415-000 - PIN HEADER CONN, BRASS, 2POS, 1ROW, 2MM" (id 4) (at 19.05 48.26 0)
-      (effects (font (size 1.27 1.27)) (justify left) hide)
-    )
-    (property "Height" "5.25" (id 5) (at 19.05 45.72 0)
-      (effects (font (size 1.27 1.27)) (justify left) hide)
-    )
-    (property "Mouser Part Number" "587-140-502-415-000" (id 6) (at 19.05 43.18 0)
-      (effects (font (size 1.27 1.27)) (justify left) hide)
-    )
-    (property "Mouser Price/Stock" "https://www.mouser.co.uk/ProductDetail/EDAC/140-502-415-000?qs=zW32dvEIR3v5NSNdqekIBw%3D%3D" (id 7) (at 19.05 40.64 0)
-      (effects (font (size 1.27 1.27)) (justify left) hide)
-    )
-    (property "Manufacturer_Name" "EDAC" (id 8) (at 19.05 38.1 0)
-      (effects (font (size 1.27 1.27)) (justify left) hide)
-    )
-    (property "Manufacturer_Part_Number" "140-502-415-000" (id 9) (at 19.05 35.56 0)
-      (effects (font (size 1.27 1.27)) (justify left) hide)
-    )
-    (pin "1")
-    (pin "2")
-  )
   (symbol (lib_id "Device:LED_Small") (at 50.8 69.85 270) (unit 1)

Commit message: f
Parts:
- added C16, C31: 100n, Capacitor_SMD:C_0603_1608Metric_Pad1.08x0.95mm_HandSolder, symbol Device:C_Small
- added C74: 15n, Capacitor_SMD:C_0603_1608Metric_Pad1.08x0.95mm_HandSolder, symbol Device:C_Small
- added R33: 60, Resistor_SMD:R_0603_1608Metric_Pad0.98x0.95mm_HandSolder, symbol Device:R_Small
- added R96, R97: 10k, Resistor_SMD:R_0603_1608Metric_Pad0.98x0.95mm_HandSolder, symbol Device:R_Small
- added TP3, TP4: TestPoint, TestPoint:TestPoint_Pad_1.5x1.5mm, symbol Connector:TestPoint
- added U19, U20: TLV9161IDBVR, Package_SO:SOIC-8_3.9x4.9mm_P1.27mm, symbol Amplifier_Operational:OP179GS
- C51: value 3.5n -> 15n
- D17: footprint SamacSys_Parts:SOT95P285X140-6N -> SOT95P285X140-6N
- R63: value 45 -> 60
- R68: value X -> 300
- R70: value 120 -> 60
- R76, R77, R79, R80: value 50k+ -> 64k
- U13: footprint Package_TO_SOT_SMD:SOT-23-8_Handsoldering -> Package_TO_SOT_SMD:SOT-23-8
Connections:
- net +3V3: now also U19.7 (V+), U20.7 (V+)
- net COM: now also R33.1; no longer R70.2
- net COM_CAP: now also R70.2; no longer R70.1
- net GND: now also C16.2, C31.2, C74.2, U19.4 (V-), U20.4 (V-); no longer C51.2
- net Temp1: now also R76.1, TH1.1, U19.3 (+); no longer R79.2, TH1.2, U13.1 (AIN0)
- net Temp2: now also R77.1, TH2.1, U20.3 (+); no longer R80.2, TH2.2, U13.2 (AIN1)
- net at U13.3 (AIN2): now also TP3.1
- net at U13.4 (AIN3/REF): now also TP4.1
- new net: C51.2, C74.1
- new net: R33.2, R70.1
- new net: R79.2, TH1.2
- new net: R80.2, TH2.2
- new net Temp1_buffer: R96.1, U19.2 (-), U19.6
- new net Temp1_out: C16.1, R96.2, U13.1 (AIN0)
- new net Temp2_buffer: R97.1, U20.2 (-), U20.6
- new net Temp2_out: C31.1, R97.2, U13.2 (AIN1)
- no-connect marks 11 -> 9
Other:
- note added: "HEATER"
- note removed: "for the heater?"
- moved on the sheet: C52, C53, C54, C55, C56, D17, D18, F2, F3, FB2, J13, J14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

Commit message: h
Parts:
- removed U19, U20: TLV9161IDBVR, Package_SO:SOIC-8_3.9x4.9mm_P1.27mm, symbol Amplifier_Operational:OP179GS
- added C80: 100n, Capacitor_SMD:C_0603_1608Metric_Pad1.08x0.95mm_HandSolder, symbol Device:C_Small
- added Q12: SSM6N7002, Package_TO_SOT_SMD:SOT-363_SC-70-6_Handsoldering, symbol Device:Q_Dual_NMOS_S1G1D2S2G2D1
- added R104, R106: 10k, Resistor_SMD:R_0603_1608Metric_Pad0.98x0.95mm_HandSolder, symbol Device:R_Small
- added R105: 60, Resistor_SMD:R_0603_1608Metric_Pad0.98x0.95mm_HandSolder, symbol Device:R_Small
- added U9: TLV9062xD, Package_SO:SOIC-8_3.9x4.9mm_P1.27mm, symbol Amplifier_Operational:TLV9062xD
- C46, C47: value 10u -> 22u; footprint Capacitor_SMD:C_0603_1608Metric_Pad1.08x0.95mm_HandSolder -> Capacitor_SMD:C_0805_2012Metric_Pad1.18x1.45mm_HandSolder
- C48, C49: footprint Capacitor_SMD:C_0603_1608Metric_Pad1.08x0.95mm_HandSolder -> Capacitor_SMD:C_0805_2012Metric_Pad1.18x1.45mm_HandSolder
- D17: footprint SOT95P285X140-6N -> SamacSys_Parts:SOT95P285X140-6N
- R66: value 1k -> 60
Connections:
- net GND: now also C80.2, Q12.1 (S), Q12.4 (S), R106.1, U9.4 (V-); no longer R66.2
- net IN_SOLAR-: now also R104.2
- net Temp1: now also U9.5 (+)
- net Temp1_buffer: now also U9.6 (-), U9.7
- net Temp2: now also U9.3 (+)
- net Temp2_buffer: now also U9.1, U9.2 (-)
- new net: Q12.2 (G), Q12.3 (D), R104.1
- new net: Q12.6 (D), R66.2
- new net: Q12.5 (G), R105.1
- new net +3.3VA: C80.1, U9.8 (V+)
- new net CHG_EN: R105.2, R106.2
Other:
- moved on the sheet: D12, D13, R66
