File: Bird_detector_V1/Power.kicad_sch (KiCad schematic)
At the start: 80 parts, among them J11 Solar input, J13 USB_A, J14 batt input, Q10 SSM6N7002, Q11 DMP3028LSD, Q12 SSM6N7002, Q7 DMP3028LSD, Q8 DMP3028LSD, Q9 DMP3028LSD, U12 CN3791, U13 MAX11601, U14 INA3221, U15 APX810S05, U9 TLV9062xD

Commit message: r
Parts:
- added C82: C_Polarized_Small, symbol Device:C_Polarized_Small
Connections:
- net +BATT: now also C82.1
- net GND: now also C82.2
- net IN_SOLAR-: now also Q7.1 (S)
- net VDC: no longer Q7.1 (S)
Other:
- note added: "ADC I2C"
- moved on the sheet: Q7A
Changed lines of the file:
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@@
   (junction (at 284.48 214.63) (diameter 0) (color 0 0 0 0)
   )
+  (junction (at 104.14 48.26) (diameter 0) (color 0 0 0 0)
+  )
   (junction (at 217.17 116.84) (diameter 0) (color 0 0 0 0)
   )
@@
   (junction (at 132.08 265.43) (diameter 0) (color 0 0 0 0)
   )
-  (junction (at 210.82 48.26) (diameter 0) (color 0 0 0 0)
-  )
   (junction (at 264.16 48.26) (diameter 0) (color 0 0 0 0)
   )
@@
   (junction (at 166.37 166.37) (diameter 0) (color 0 0 0 0)
   )
+  (junction (at 24.13 261.62) (diameter 0) (color 0 0 0 0)
+  )
   (junction (at 105.41 102.87) (diameter 0) (color 0 0 0 0)
   )
@@
   (junction (at 85.09 48.26) (diameter 0) (color 0 0 0 0)
   )
+  (junction (at 30.48 242.57) (diameter 0) (color 0 0 0 0)
+  )
   (junction (at 85.09 44.45) (diameter 0) (color 0 0 0 0)
   )
@@
     (stroke (width 0) (type default) (color 0 0 0 0))
   )
-  (wire (pts (xy 24.13 242.57) (xy 40.64 242.57))
+  (wire (pts (xy 24.13 242.57) (xy 30.48 242.57))
     (stroke (width 0) (type default) (color 0 0 0 0))
   )
@@
     (stroke (width 0) (type default) (color 0 0 0 0))
   )
-  (wire (pts (xy 233.68 27.94) (xy 224.79 27.94))
+  (wire (pts (xy 127 27.94) (xy 118.11 27.94))
     (stroke (width 0) (type default) (color 0 0 0 0))
   )
@@
     (stroke (width 0) (type default) (color 0 0 0 0))
   )
-  (wire (pts (xy 233.68 25.4) (xy 233.68 27.94))
+  (wire (pts (xy 127 25.4) (xy 127 27.94))
     (stroke (width 0) (type default) (color 0 0 0 0))
   )
@@
     (stroke (width 0) (type default) (color 0 0 0 0))
   )
-  (wire (pts (xy 24.13 245.11) (xy 24.13 250.19))
+  (wire (pts (xy 24.13 245.11) (xy 24.13 261.62))
     (stroke (width 0) (type default) (color 0 0 0 0))
   )
@@
     (stroke (width 0) (type default) (color 0 0 0 0))
   )
+  (wire (pts (xy 30.48 259.08) (xy 30.48 261.62))
+    (stroke (width 0) (type default) (color 0 0 0 0))
+  )
   (wire (pts (xy 67.31 167.64) (xy 67.31 186.69))
     (stroke (width 0) (type default) (color 0 0 0 0))
@@
     (stroke (width 0) (type default) (color 0 0 0 0))
   )
+  (wire (pts (xy 104.14 48.26) (xy 113.03 48.26))
+    (stroke (width 0) (type default) (color 0 0 0 0))
+  )
   (wire (pts (xy 78.74 250.19) (xy 78.74 265.43))
     (stroke (width 0) (type default) (color 0 0 0 0))
@@
     (stroke (width 0) (type default) (color 0 0 0 0))
   )
-  (wire (pts (xy 191.77 48.26) (xy 210.82 48.26))
+  (wire (pts (xy 191.77 48.26) (xy 217.17 48.26))
     (stroke (width 0) (type default) (color 0 0 0 0))
   )
@@
     (stroke (width 0) (type default) (color 0 0 0 0))
   )
-  (wire (pts (xy 95.25 48.26) (xy 113.03 48.26))
+  (wire (pts (xy 95.25 48.26) (xy 104.14 48.26))
     (stroke (width 0) (type default) (color 0 0 0 0))
   )
@@
     (stroke (width 0) (type default) (color 0 0 0 0))
   )
+  (wire (pts (xy 30.48 242.57) (xy 40.64 242.57))
+    (stroke (width 0) (type default) (color 0 0 0 0))
+  )
   (wire (pts (xy 337.82 201.93) (xy 337.82 204.47))
     (stroke (width 0) (type default) (color 0 0 0 0))
@@
     (stroke (width 0) (type default) (color 0 0 0 0))
   )
-  (wire (pts (xy 224.79 25.4) (xy 233.68 25.4))
+  (wire (pts (xy 118.11 25.4) (xy 127 25.4))
     (stroke (width 0) (type default) (color 0 0 0 0))
   )
-  (wire (pts (xy 219.71 35.56) (xy 223.52 35.56))
+  (wire (pts (xy 113.03 35.56) (xy 116.84 35.56))
     (stroke (width 0) (type default) (color 0 0 0 0))
   )
-  (wire (pts (xy 214.63 27.94) (xy 210.82 27.94))
+  (wire (pts (xy 107.95 27.94) (xy 104.14 27.94))
     (stroke (width 0) (type default) (color 0 0 0 0))
   )
@@
     (stroke (width 0) (type default) (color 0 0 0 0))
   )
+  (wire (pts (xy 30.48 261.62) (xy 24.13 261.62))
+    (stroke (width 0) (type default) (color 0 0 0 0))
+  )
   (wire (pts (xy 162.56 242.57) (xy 160.02 242.57))
     (stroke (width 0) (type default) (color 0 0 0 0))
@@
     (stroke (width 0) (type default) (color 0 0 0 0))
   )
+  (wire (pts (xy 30.48 254) (xy 30.48 242.57))
+    (stroke (width 0) (type default) (color 0 0 0 0))
+  )
   (wire (pts (xy 43.18 48.26) (xy 50.8 48.26))
     (stroke (width 0) (type default) (color 0 0 0 0))
@@
     (stroke (width 0) (type default) (color 0 0 0 0))
   )
-  (wire (pts (xy 210.82 27.94) (xy 210.82 48.26))
+  (wire (pts (xy 104.14 27.94) (xy 104.14 48.26))
     (stroke (width 0) (type default) (color 0 0 0 0))
   )
@@
     (stroke (width 0) (type default) (color 0 0 0 0))
   )
-  (wire (pts (xy 210.82 48.26) (xy 217.17 48.26))
-    (stroke (width 0) (type default) (color 0 0 0 0))
-  )
   (wire (pts (xy 378.46 48.26) (xy 378.46 83.82))
     (stroke (width 0) (type default) (color 0 0 0 0))
@@
     (stroke (width 0) (type default) (color 0 0 0 0))
   )
+  (wire (pts (xy 24.13 261.62) (xy 24.13 264.16))
+    (stroke (width 0) (type default) (color 0 0 0 0))
+  )
   (wire (pts (xy 40.64 130.81) (xy 52.07 130.81))
     (stroke (width 0) (type default) (color 0 0 0 0))
@@
     (stroke (width 0) (type default) (color 0 0 0 0))
   )
-  (text "HEATER" (at 213.36 19.05 0)
+  (text "HEATER" (at 106.68 19.05 0)
     (effects (font (size 1.27 1.27)) (justify left bottom))
   )
@@
     (effects (font (size 1.27 1.27)) (justify left bottom))
   )
+  (text "ADC I2C" (at 336.55 142.24 0)
+    (effects (font (size 3 3)) (justify left bottom))
+  )
   (text "4.5-28V \ninput" (at 240.665 62.23 0)
     (effects (font (size 1.27 1.27)) (justify left bottom))
@@
     (effects (font (size 1.27 1.27)) (justify left bottom))
   )
-  (label "Heater_Input" (at 233.68 25.4 0)
+  (label "Heater_Input" (at 127 25.4 0)
     (effects (font (size 1.27 1.27)) (justify left bottom))
   )
@@
     (effects (font (size 1.27 1.27)) (justify left))
   )
-  (hierarchical_label "HEAT" (shape input) (at 223.52 35.56 0)
+  (hierarchical_label "HEAT" (shape input) (at 116.84 35.56 0)
     (effects (font (size 1.27 1.27)) (justify left))
   )
@@
     (pin "1")
   )
-  (symbol (lib_id "My_custom_lib:DMP2040USD") (at 219.71 27.94 270) (mirror x) (unit 1)
+  (symbol (lib_id "My_custom_lib:DMP2040USD") (at 113.03 27.94 270) (mirror x) (unit 1)
     (in_bom yes) (on_board yes)
-    (property "Reference" "Q7" (id 0) (at 212.09 21.59 90))
-    (property "Value" "DMP3028LSD" (id 1) (at 212.09 24.13 90))
-    (property "Footprint" "Package_SO:SO-8_3.9x4.9mm_P1.27mm" (id 2) (at 232.41 22.86 0)
+    (property "Reference" "Q7" (id 0) (at 105.41 21.59 90))
+    (property "Value" "DMP3028LSD" (id 1) (at 105.41 24.13 90))
+    (property "Footprint" "Package_SO:SO-8_3.9x4.9mm_P1.27mm" (id 2) (at 125.73 22.86 0)
       (effects (font (size 1.27 1.27)) hide)
     )
-    (property "Datasheet" "" (id 3) (at 224.79 35.56 0)
+    (property "Datasheet" "" (id 3) (at 118.11 35.56 0)
       (effects (font (size 1.27 1.27)) hide)
     )
@@
     (pin "1")
   )
+  (symbol (lib_id "Device:C_Polarized_Small") (at 30.48 256.54 0) (unit 1)
+    (in_bom yes) (on_board yes) (fields_autoplaced)
+    (property "Reference" "C82" (id 0) (at 33.02 254.7238 0)
+      (effects (font (size 1.27 1.27)) (justify left))
+    )
+    (property "Value" "C_Polarized_Small" (id 1) (at 33.02 257.2638 0)
+      (effects (font (size 1.27 1.27)) (justify left))
+    )
+    (property "Footprint" "" (id 2) (at 30.48 256.54 0)
+      (effects (font (size 1.27 1.27)) hide)
+    )
+    (property "Datasheet" "~" (id 3) (at 30.48 256.54 0)
+      (effects (font (size 1.27 1.27)) hide)
+    )
+    (pin "1")
+    (pin "2")
+  )
   (symbol (lib_id "Device:LED_Small") (at 289.56 83.82 0) (mirror y) (unit 1)
     (in_bom yes) (on_board yes)
@@
     (pin "2")
   )
-  (symbol (lib_id "power:GND") (at 24.13 250.19 0) (unit 1)
+  (symbol (lib_id "power:GND") (at 24.13 264.16 0) (unit 1)
     (in_bom yes) (on_board yes) (fields_autoplaced)
-    (property "Reference" "#PWR0170" (id 0) (at 24.13 256.54 0)
+    (property "Reference" "#PWR0170" (id 0) (at 24.13 270.51 0)
       (effects (font (size 1.27 1.27)) hide)
     )
-    (property "Value" "GND" (id 1) (at 24.13 255.27 0)
+    (property "Value" "GND" (id 1) (at 24.13 269.24 0)
       (effects (font (size 1.27 1.27)) hide)
     )
-    (property "Footprint" "" (id 2) (at 24.13 250.19 0)
+    (property "Footprint" "" (id 2) (at 24.13 264.16 0)
       (effects (font (size 1.27 1.27)) hide)
     )
-    (property "Datasheet" "" (id 3) (at 24.13 250.19 0)
+    (property "Datasheet" "" (id 3) (at 24.13 264.16 0)
       (effects (font (size 1.27 1.27)) hide)
     )

Commit message: K
Parts:
- C82: value C_Polarized_Small -> supercap; footprint (none) -> Z_mycustom_footprint_lib:SCMT32D755SRBB0
- F1, F2, F3: value PPTC 2A 16V -> PPTC 2.6A 16V
Connections:
- net +3V3: now also JP5.3 (B); no longer JP5.1 (A)
- net GND: now also JP5.1 (A); no longer JP5.3 (B)
- net Drain2: now reaches Q11.5 (D), Q11.6 (D), Q11.7 (D), Q11.8 (D)
- net raw_solar: now reaches F1.1, J11.2 (Pin_2), R64.1
- net ops_led: now reaches D14.1 (K), R64.2
- net Drain1: now reaches Q8.5 (D), Q8.6 (D), Q8.7 (D), Q8.8 (D)
Other:
- moved on the sheet: C56, D18, JP5, Q11A, Q9B, R81, R82, R84

Commit message: b
Other:
- title: (none) -> Bird Detection and Recognition System
Changed lines of the file:
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@@
 (kicad_sch (version 20211123) (generator eeschema)
   (paper "A3")
+  (title_block
+    (title "Bird Detection and Recognition System")
+    (rev "V0.1")
+  )
   (junction (at 278.13 83.82) (diameter 0) (color 0 0 0 0)
   )
