File: Bird_detector_V1/Power.kicad_sch (KiCad schematic)
At the start: 81 parts, among them J11 Solar input, J13 USB_A, J14 batt input, Q10 SSM6N7002, Q11 DMP3028LSD, Q12 SSM6N7002, Q7 DMP3028LSD, Q8 DMP3028LSD, Q9 DMP3028LSD, U12 CN3791, U13 MAX11601, U14 INA3221, U15 APX810S05, U9 TLV9062xD

Commit message: h
Connections:
- net Q12_GATE2: now reaches Q12.2 (G), Q12.3 (D), R104.1
- net Q12_GATE: now reaches Q12.5 (G), R105.1
Other:
- moved on the sheet: C47, C49, C50, R75

Commit message: g
Parts:
- D17: footprint SamacSys_Parts:SOT95P285X140-6N -> SOT95P285X140-6N
Other:
- note added: "AOLAR POWER INPUT AND SMPP BMS"
- note added: "BATTERY POWER INPUT + USB SWITCH"
- note added: "BMS CELLS TEMPERATURE MOITORING CIRCUITRY"
- note added: "ESD PROTECTION"
- note added: "POWER MEASUREMENT"
- note added: "USB 2.0 POWER INPUT"
- moved on the sheet: C16, C31, C44, C45, C46, C47, C48, C49, C50, C51, C52, C53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

Commit message: g
Other:
- note added: "I2C adress 001100100"
Changed lines of the file:
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@@
     (effects (font (size 3 3)) (justify left bottom))
+  )
+  (text "I2C adress 001100100" (at 252.73 208.28 0)
+    (effects (font (size 1.27 1.27)) (justify left bottom))
   )
   (label "Q12_GATE2" (at 93.98 94.615 0)
