File: Bird_detector_V1/RF.kicad_sch (KiCad schematic)
At the start: 15 parts, among them IC1 TXB0108PWR, J1 Conn_Coaxial, J2 Conn_Coaxial, J3 Conn_Coaxial, J4 USB_A, J5 SIM_Card_Shielded, J6 USB_A, U3 SIM808

Commit message: r
Parts:
- added C8: 10u, symbol Device:C_Small
- added Q1: Q_NMOS_SGD, symbol Device:Q_NMOS_SGD
- added R1: R_Small, symbol Device:R_Small
- added TP1, TP2, TP3: TestPoint, TestPoint:TestPoint_Pad_1.5x1.5mm, symbol Connector:TestPoint
Connections:
- net +3V8: now also IC1.19 (VCCB)
- net 5V-DIY: now also U3.25 (VCHG), TP3.1; no longer U3.7 (VBUS)
- net GND: now also IC1.11 (GND), C8.2, Q1.1 (S)
- net RI_INT: now reaches U3.10 (RI)
- net RI_INT: now also IC1.18 (B2)
- net DCD_INT: now reaches U3.11 (DCD)
- net DCD_INT: now also IC1.17 (B3)
- net CTS_INT: now reaches U3.12 (CTS)
- net CTS_INT: now also IC1.16 (B4)
- net RTS_INT: now reaches U3.13 (RTS)
- net RTS_INT: now also IC1.15 (B5)
- net RX_INT: now reaches U3.14 (TXD)
- net RX_INT: now also IC1.14 (B6)
- net TX_INT: now reaches U3.15 (RXD)
- net TX_INT: now also IC1.13 (B7)
- net at U3.16 (RESET): now also TP2.1
- net STAT_INT: now reaches U3.49 (STATUS)
- net STAT_INT: now also IC1.12 (B8)
- net at U3.8 (PWRKEY): now also Q1.3 (D)
- net DTR_INT: now reaches U3.9 (DTR)
- net DTR_INT: now also IC1.20 (B1)
- net +3V3: now reaches IC1.1 (A1)
- net +3V3: now also IC1.2 (VCCA)
- net RI: now reaches IC1.3 (A2)
- net DCD: now reaches IC1.4 (A3)
- net CTS: now reaches IC1.5 (A4)
- net RTS: now reaches IC1.6 (A5)
- net RX: now reaches IC1.7 (A6)
- net TX: now reaches IC1.8 (A7)
- net STAT: now reaches IC1.9 (A8)
- net at U3.17 (V_RTC): now also U3.7 (VDD_EXT), C8.1
- new net: Q1.2 (G), R1.2
- new net ENABLE: R1.1
- no-connect marks 12 -> 24
Other:
- note added: "VCHG NEEDS 4.3-7V"
- note added: "super_cap?"
- moved on the sheet: C1, C2, C3, C4, C5, C6, C7, IC1, J1, J2, J3, J4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

Commit message: g
Parts:
- removed C1: C_Small, symbol Device:C_Small
- added C? (x6): DNP, Capacitor_SMD:C_0603_1608Metric_Pad1.08x0.95mm_HandSolder, symbol Device:C_Small
- added C?: 1u, Capacitor_SMD:C_0603_1608Metric_Pad1.08x0.95mm_HandSolder, symbol Device:C_Small
- added D? (x2): D5V0P4UR6SO-7, SOT95P285X140-6N, symbol SamacSys_Parts:D5V0P4UR6SO-7
- added IC1: TXB0108PWR, SamacSys_Parts:SOP65P640X120-20N, symbol SamacSys_Parts:TXB0108PWR
- added R? (x3): 0, Resistor_SMD:R_0603_1608Metric_Pad0.98x0.95mm_HandSolder, symbol Device:R_Small
- C2: renamed from C4; footprint (none) -> Capacitor_SMD:C_0603_1608Metric_Pad1.08x0.95mm_HandSolder
- C3: renamed from C5; footprint (none) -> Capacitor_SMD:C_0603_1608Metric_Pad1.08x0.95mm_HandSolder
- C4: renamed from C6; footprint (none) -> Capacitor_SMD:C_0603_1608Metric_Pad1.08x0.95mm_HandSolder
- C5: renamed from C2; value C_Small -> gap
- C6: renamed from C7; footprint (none) -> Capacitor_SMD:C_0603_1608Metric_Pad1.08x0.95mm_HandSolder
- C7: renamed from C8; footprint (none) -> Capacitor_SMD:C_0603_1608Metric_Pad1.08x0.95mm_HandSolder
- IC2: renamed from IC1; footprint SOP65P640X120-20N -> SamacSys_Parts:SOP65P640X120-20N
- R1: footprint (none) -> Resistor_SMD:R_0603_1608Metric_Pad0.98x0.95mm_HandSolder
- renumbered C3 to C1, J4 to J1, J5 to J2, J1 to J3, J6 to J4, J2 to J5, J3 to J6, U3 to U1
Connections:
- net +1V8: now also C?.1
- net +3V3: now also IC2.10 (OE), IC1.10 (OE), IC1.2 (VCCA)
- net +3V8: now also IC1.19 (VCCB)
- net D+: now also D?.6 (I/O4)
- net D-: now also D?.4 (I/O3)
- net D2-: now also D?.1 (I/O1), D?.6 (I/O4)
- net GND: now also C?.2, C?.2, C?.2, C?.2, C?.2, C?.2, C?.2, D?.2 (VSS), D?.2 (VSS), IC1.11 (GND)
- net SCL: now also IC1.9 (A8); no longer U1.39 (SCL)
- net SDA: now also IC1.8 (A7); no longer U1.38 (SDA)
- net STAT: now also IC1.7 (A6); no longer IC2.9 (A8)
- net STAT_INT: now also IC1.14 (B6); no longer IC2.12 (B8)
- net at J6.1 (In): now also C?.1, R?.2; no longer U1.35 (GPS_RF_IN)
- net RESET_INT: now reaches TP2.1, U1.16 (RESET)
- net RESET_INT: now also IC2.12 (B8)
- net at U1.53 (ANT_BT): now also C?.1, R?.1; no longer J5.1 (In)
- net at U1.66 (GSM_RF_IN): now also C?.1, R?.1; no longer J3.1 (In)
- net 5V-in2: now reaches C5.1, J4.1 (VBUS)
- net 5V-in2: now also D?.5 (VCC)
- new net: C?.1, J5.1 (In), R?.2
- new net: C?.1, R?.1, U1.35 (GPS_RF_IN)
- new net: C?.1, J3.1 (In), R?.2
- new net RESET_GSM: IC2.9 (A8)
- new net SCL_INT: IC1.13 (B7), U1.39 (SCL)
- new net SDA_INT: IC1.12 (B8), U1.38 (SDA)
Other:
- note added: "1v8 3v3 ? TVS goes here"
- note added: "Add some TVS and the parasitic capacitance should not exceed 50pF."
- note added: "high is high power is used or it will soon start maybe use a led + change SMPS operation made low when in sleep or not transmiting RF"
- note removed: "1v8 TVS goes here"
- moved on the sheet: C5, IC2, J1, J2, J3, J5, J6, Q1, R1, TP1, TP2, U1A

Commit message: g
Parts:
- gave numbers to parts that had none: 12
- renumbered C7 to C10, C1 to C4, C2 to C5, C3 to C6, C4 to C7, C5 to C8, C6 to C9

Commit message: f
Parts:
- removed D1: D5V0P4UR6SO-7, SOT95P285X140-6N, symbol SamacSys_Parts:D5V0P4UR6SO-7
- removed IC1: TXB0108PWR, SamacSys_Parts:SOP65P640X120-20N, symbol SamacSys_Parts:TXB0108PWR
- removed J1: USB_A, Connector_USB:USB_A_Molex_105057_Vertical, symbol Connector:USB_A
- removed Q1: Q_NMOS_SGD, symbol Device:Q_NMOS_SGD
- added D1, D2, D3, D4: LED_Small, symbol Device:LED_Small
- added D5: D5V0P4UR6SO-7, SOT95P285X140-6N, symbol SamacSys_Parts:D5V0P4UR6SO-7
- added D6: z, Diode_SMD:D_SOD-123, symbol Device:D_Zener_Small
- added Q1, Q2, Q3, Q4: SSM6N7002, symbol Device:Q_Dual_NMOS_S1G1D2S2G2D1
- added R1, R10, R13, R15, R18, R2, R9: 100, Resistor_SMD:R_0603_1608Metric_Pad0.98x0.95mm_HandSolder, symbol Device:R_Small
- added R11, R12, R16, R19, R6: 100k, Resistor_SMD:R_0603_1608Metric_Pad0.98x0.95mm_HandSolder, symbol Device:R_Small
- added R14, R17, R7, R8: X, Resistor_SMD:R_0603_1608Metric_Pad0.98x0.95mm_HandSolder, symbol Device:R_Small
- added R4, R5: 10k, Resistor_SMD:R_0603_1608Metric_Pad0.98x0.95mm_HandSolder, symbol Device:R_Small
- added SW1: SW_SPST, SamacSys_Parts:PTS526SK15SMTR2LFS, symbol Switch:SW_SPST
- R3: renamed from R1; value R_Small -> 100
- renumbered D2 to D7, IC2 to IC1, J2 to J1, J3 to J2, J4 to J3, J5 to J4, J6 to J5, R2 to R20, R3 to R21, R4 to R22
Connections:
- net +3V3: now also D5.5 (VCC), R1.2, R13.2, R2.2
- net +3V8: now also D1.2 (A), D2.2 (A), D3.2 (A), D4.2 (A), D6.1 (K), R4.1, R5.2
- net ENABLE: now also R6.2
- net GND: now also D5.2 (VSS), D6.2 (A), Q1.1 (S), Q3.1 (S), Q3.4 (S), Q4.1 (S), Q4.4 (S), R11.1, R12.1, R16.1, R19.1, R6.1, SW1.1 (A)
- net RESET_GSM: now also SW1.2 (B)
- net SCL: now also Q2.4 (S)
- net SCL_INT: now also Q2.3 (D), R5.1
- net SDA: now also Q2.1 (S)
- net SDA_INT: now also Q2.6 (D), R4.2
- net STAT: now also Q1.4 (S)
- net STAT_INT: now also Q1.3 (D), R18.2, R19.2
- net at R3.2: now also Q1.2 (G)
- net PRWKEY: now reaches U1.8 (PWRKEY)
- net PRWKEY: now also Q1.6 (D)
- net at J1.2 (RST), U1.32 (SIM_RST): now also D5.3 (I/O2)
- net at J1.3 (CLK), U1.31 (SIM_CLK): now also D5.6 (I/O4)
- net at J1.7 (I/O), U1.30 (SIM_DATA): now also D5.1 (I/O1)
- net IPPS: now reaches U1.37 (IPPS)
- net IPPS: now also R15.2, R16.2
- net NETLIGHT: now reaches U1.50 (NETLIGHT)
- net NETLIGHT: now also R11.2, R9.2
- net RF_SYNC: now reaches U1.63 (RF_SYNS)
- net RF_SYNC: now also R10.2, R12.2
- new net: D2.1 (K), R8.2
- new net: Q4.6 (D), R14.1
- new net: D3.1 (K), R14.2
- new net: D1.1 (K), R7.2
- new net: Q4.3 (D), R17.1
- new net: D4.1 (K), R17.2
- new net: Q3.3 (D), R7.1
- new net: Q3.5 (G), R9.1
- new net: Q2.2 (G), R1.1
- new net: Q2.5 (G), R2.1
- new net: Q1.5 (G), R13.1
- new net: Q3.2 (G), R10.1
- new net: Q4.5 (G), R18.1
- new net: Q3.6 (D), R8.1
- new net: Q4.2 (G), R15.1
- no-connect marks 24 -> 28
Other:
- moved on the sheet: C1, C12, C14, C2, C3, D7, R21, R22, R3, TP1, TP2

Commit message: j
Parts:
- D1, D2, D3, D4: footprint (none) -> LED_SMD:LED_0603_1608Metric_Pad1.05x0.95mm_HandSolder
- D5, D7: footprint SOT95P285X140-6N -> SamacSys_Parts:SOT95P285X140-6N
Changed lines of the file:
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@@
       (effects (font (size 1.27 1.27)) (justify right))
     )
-    (property "Footprint" "" (id 2) (at 303.53 50.8 90)
+    (property "Footprint" "LED_SMD:LED_0603_1608Metric_Pad1.05x0.95mm_HandSolder" (id 2) (at 303.53 50.8 90)
       (effects (font (size 1.27 1.27)) hide)
     )
@@
       (effects (font (size 1.27 1.27)) (justify right))
     )
-    (property "Footprint" "" (id 2) (at 241.3 48.26 90)
+    (property "Footprint" "LED_SMD:LED_0603_1608Metric_Pad1.05x0.95mm_HandSolder" (id 2) (at 241.3 48.26 90)
       (effects (font (size 1.27 1.27)) hide)
     )
@@
       (effects (font (size 1.27 1.27)) (justify right))
     )
-    (property "Footprint" "" (id 2) (at 361.95 87.63 90)
+    (property "Footprint" "LED_SMD:LED_0603_1608Metric_Pad1.05x0.95mm_HandSolder" (id 2) (at 361.95 87.63 90)
       (effects (font (size 1.27 1.27)) hide)
     )
@@
       (effects (font (size 1.27 1.27)) (justify right))
     )
-    (property "Footprint" "" (id 2) (at 290.83 114.3 90)
+    (property "Footprint" "LED_SMD:LED_0603_1608Metric_Pad1.05x0.95mm_HandSolder" (id 2) (at 290.83 114.3 90)
       (effects (font (size 1.27 1.27)) hide)
     )
@@
     (property "Reference" "D5" (id 0) (at 77.47 132.08 0))
     (property "Value" "D5V0P4UR6SO-7" (id 1) (at 77.47 134.62 0))
-    (property "Footprint" "SOT95P285X140-6N" (id 2) (at 67.31 147.32 0)
+    (property "Footprint" "SamacSys_Parts:SOT95P285X140-6N" (id 2) (at 67.31 147.32 0)
       (effects (font (size 1.27 1.27)) (justify left) hide)
     )
@@
     (property "Reference" "D7" (id 0) (at 374.65 236.22 0))
     (property "Value" "D5V0P4UR6SO-7" (id 1) (at 374.65 238.76 0))
-    (property "Footprint" "SOT95P285X140-6N" (id 2) (at 384.81 241.3 0)
-      (effects (font (size 1.27 1.27)) (justify left) hide)
-    )
+    (property "Footprint" "SamacSys_Parts:SOT95P285X140-6N" (id 2) (at 384.81 241.3 0)
+      (effects (font (size 1.27 1.27)) (justify left) hide)
+    )

Commit message: f
Parts:
- removed TP1: TestPoint, TestPoint:TestPoint_Pad_1.5x1.5mm, symbol Connector:TestPoint
- added Q4: SSM6N7002, Package_TO_SOT_SMD:SOT-363_SC-70-6_Handsoldering, symbol Device:Q_Dual_NMOS_S1G1D2S2G2D1
- added R15: 100, Resistor_SMD:R_0603_1608Metric_Pad0.98x0.95mm_HandSolder, symbol Device:R_Small
- added R16: 100k, Resistor_SMD:R_0603_1608Metric_Pad0.98x0.95mm_HandSolder, symbol Device:R_Small
- added R8: 1k, Resistor_SMD:R_0603_1608Metric_Pad0.98x0.95mm_HandSolder, symbol Device:R_Small
- C8: value gap -> DNP
- C9: value 10u -> DNP
- Q1: renamed from Q3; footprint (none) -> Package_TO_SOT_SMD:SOT-363_SC-70-6_Handsoldering
- Q2: footprint (none) -> Package_TO_SOT_SMD:SOT-363_SC-70-6_Handsoldering
- Q3: renamed from Q1; footprint (none) -> Package_TO_SOT_SMD:SOT-363_SC-70-6_Handsoldering
- Q5: renamed from Q4; footprint (none) -> Package_TO_SOT_SMD:SOT-363_SC-70-6_Handsoldering
- renumbered D4 to D3, D3 to D4, R13 to R10, R3 to R11, R10 to R12, R6 to R13, R12 to R14, R14 to R18, R18 to R19, R15 to R20, R19 to R21, R16 to R22, R20 to R23, R21 to R24, R22 to R25, R4 to R3, R5 to R4, R7 to R5, R8 to R6, R9 to R7, R11 to R9, TP2 to TP1, TP3 to TP2
Connections:
- net +3V8: now also R8.2
- net GND: now also Q4.1 (S), Q4.4 (S), R16.1; no longer Q1.1 (S)
- net RF_SYNC: now also Q4.6 (D), R15.2, R16.2, R8.1
- net at R12.1: now also Q4.5 (G); no longer Q1.2 (G)
- net at R6.1: now also Q4.3 (D); no longer Q1.6 (D)
- new net: Q4.2 (G), R15.1
Other:
- moved on the sheet: D1, D2, D3, D4, Q1A, Q1B, Q2A, Q2B, Q3A, Q3B, Q5A, Q5B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

Commit message: R
Other:
- note added: "GNNS/GSM POWER"
- note added: "GSM/GNSS DATA+ RF +SIM"
- note added: "LEDS"
- note added: "LEVEL SHIFTERS"
- moved on the sheet: C1, C10, C11, C12, C13, C14, C2, C3, C4, C5, C6, C7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

Commit message: v
Parts:
- added C3: 10u, Capacitor_SMD:C_0603_1608Metric_Pad1.08x0.95mm_HandSolder, symbol Device:C_Small
- C2: renamed from C4; footprint (none) -> Capacitor_SMD:CP_Elec_8x10.5
- J2: value Conn_Coaxial -> GSM; footprint Connector_Coaxial:SMA_Amphenol_901-143_Horizontal -> Z_mycustom_footprint_lib:SMA_Amphenol_901-143_Horizontal_no_edgecuts
- J4: value Conn_Coaxial -> BT; footprint Connector_Coaxial:SMA_Amphenol_901-143_Horizontal -> Z_mycustom_footprint_lib:SMA_Amphenol_901-143_Horizontal_no_edgecuts
- J5: value Conn_Coaxial -> GNSS; footprint Connector_Coaxial:SMA_Amphenol_901-143_Horizontal -> Z_mycustom_footprint_lib:SMA_Amphenol_901-143_Horizontal_no_edgecuts
- renumbered C9 to C10, C10 to C11, C11 to C12, C12 to C13, C13 to C14, C14 to C15, C5 to C4, C6 to C5, C7 to C6, C2 to C7, C3 to C8, C8 to C9, D4 to D2, D2 to D4, Q5 to Q3, Q3 to Q4, Q4 to Q5, R19 to R10, R9 to R11, R22 to R12, R21 to R13, R10 to R14, R11 to R15, R13 to R16, R6 to R17, R8 to R18, R12 to R19, R14 to R20, R15 to R21, R16 to R22, R18 to R6, R17 to R7, R7 to R8, R20 to R9, TP2 to TP1, TP1 to TP2
Connections:
- net +3V8: now also C3.1
- net D2+: now also D7.3 (I/O2)
- net D2-: now also D7.4 (I/O3); no longer D7.1 (I/O1), D7.6 (I/O4)
- net GND: now also C3.2
- net GNSS_RF2: now reaches C15.1, J5.1 (In), R25.2
- net BT_RF1: now reaches C12.1, R24.1, U1.53 (ANT_BT)
- net GSM_RF1: now reaches C7.1, R23.1, U1.66 (GSM_RF_IN)
- net SIM_RST: now reaches J1.2 (RST), U1.32 (SIM_RST)
- net SIM_RST: now also D5.6 (I/O4); no longer D5.3 (I/O2)
- net SIM_CLK: now reaches J1.3 (CLK), U1.31 (SIM_CLK)
- net SIM_CLK: now also D5.1 (I/O1); no longer D5.6 (I/O4)
- net SIM_IO: now reaches J1.7 (I/O), U1.30 (SIM_DATA)
- net SIM_IO: now also D5.3 (I/O2); no longer D5.1 (I/O1)
- net BT_RF2: now reaches C13.1, J4.1 (In), R24.2
- net GNSS_RF1: now reaches C14.1, R25.1, U1.35 (GPS_RF_IN)
- net GSM_RF2: now reaches C8.1, J2.1 (In), R23.2
Other:
- moved on the sheet: C1, C12, C13, C14, C15, C4, C5, C6, C7, C8, D1, D2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
