File: Bird_detector_V1/RF.kicad_sch (KiCad schematic)
At the start: 62 parts, among them IC1 TXB0108PWR, J1 SIM_Card_Shielded, J2 GSM, J3 USB_A, J4 BT, J5 GNSS, Q1 SSM6N7002, Q2 SSM6N7002, Q3 SSM6N7002, Q4 SSM6N7002, Q5 SSM6N7002, SW1 SW_SPST, U1 SIM808

Commit message: f
Parts:
- added JP2: LED_on/off, Connector_PinHeader_2.54mm:PinHeader_1x03_P2.54mm_Vertical, symbol Jumper:Jumper_3_Bridged12
- added NT1: NetTie_2, NetTie:NetTie-2_SMD_Pad0.5mm, symbol Device:NetTie_2
- renumbered C4 to C10, C5 to C12, C6 to C13, C10 to C14, C9 to C15, C7 to C2, C12 to C3, C14 to C4, C8 to C5, C13 to C6, C15 to C7, C2 to C8, C3 to C9, D5 to D1, D6 to D2, D1 to D3, D2 to D5, D7 to D6, D3 to D7, J4 to J3, J5 to J4, J3 to J5, Q2 to Q1, Q4 to Q2, Q1 to Q3, Q5 to Q4, Q3 to Q5, R16 to R1, R25 to R10, R8 to R12, R5 to R13, R20 to R14, R19 to R15, R17 to R16, R12 to R17, R9 to R18, R6 to R19, R15 to R2, R22 to R20, R13 to R22, R18 to R23, R10 to R24, R7 to R25, R1 to R3, R3 to R4, R4 to R5, R2 to R6, R14 to R7, R23 to R8, R24 to R9, TP2 to TP1, TP1 to TP2
Connections:
- net +3V3: now also NT1.2; no longer IC1.1 (A1), IC1.10 (OE)
- net +3V8: now also JP2.1 (A); no longer D3.2 (A), D4.2 (A), D5.2 (A), D7.2 (A)
- new net DTR: IC1.1 (A1)
- new net LED_PWR: D3.2 (A), D4.2 (A), D5.2 (A), D7.2 (A), JP2.2 (C)
- new net OE_ENABLE: IC1.10 (OE), NT1.1
- no-connect marks 28 -> 29
Other:
- moved on the sheet: D3, Q3B, R11, R12, R13

Commit message: v
Parts:
- removed unit 1 of Q3
- renumbered C14 to C10, C3 to C12, C6 to C13, C4 to C14, C7 to C15, C8 to C2, C9 to C3, C10 to C4, C12 to C5, C13 to C6, C2 to C7, C5 to C8, C15 to C9, D5 to D1, D3 to D2, D7 to D3, D1 to D5, D2 to D6, D6 to D7, J5 to J3, J3 to J4, J4 to J5, JP2 to JP1, Q3 to Q1, Q1 to Q2, Q5 to Q3, Q2 to Q4, Q4 to Q5, R3 to R1, R24 to R10, R17 to R11, R11 to R12, R22 to R13, R7 to R14, R2 to R15, R1 to R16, R16 to R17, R23 to R18, R15 to R19, R6 to R2, R14 to R20, R20 to R22, R8 to R23, R9 to R24, R10 to R25, R4 to R3, R5 to R4, R19 to R5, R13 to R6, R25 to R7, R18 to R8, R12 to R9, TP2 to TP1, TP1 to TP2

Commit message: v
Parts:
- J3: footprint Connector_USB:USB_A_Molex_105057_Vertical -> Connector_PinHeader_2.54mm:PinHeader_1x04_P2.54mm_Vertical
Changed lines of the file:
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@@
     (property "Reference" "J3" (id 0) (at 383.54 194.945 0))
     (property "Value" "USB_A" (id 1) (at 383.54 197.485 0))
-    (property "Footprint" "Connector_USB:USB_A_Molex_105057_Vertical" (id 2) (at 379.73 209.55 0)
+    (property "Footprint" "Connector_PinHeader_2.54mm:PinHeader_1x04_P2.54mm_Vertical" (id 2) (at 379.73 209.55 0)
       (effects (font (size 1.27 1.27)) hide)
     )

Commit message: f
Parts:
- removed C6: 33p, Capacitor_SMD:C_0603_1608Metric_Pad1.08x0.95mm_HandSolder, symbol Device:C_Small
- D5, D7: footprint SamacSys_Parts:SOT95P285X140-6N -> SOT95P285X140-6N
- D6: value z -> 5v1
- IC1: footprint SamacSys_Parts:SOP65P640X120-20N -> SOP65P640X120-20N
- R1, R10, R14, R15, R19, R2, R21, R8, R9: value 100 -> 60
- R17, R5, R6, R7: value X -> 300
Changed lines of the file:
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@@
   (junction (at 370.84 134.62) (diameter 0) (color 0 0 0 0)
   )
-  (junction (at 294.64 193.04) (diameter 0) (color 0 0 0 0)
-  )
   (junction (at 312.42 129.54) (diameter 0) (color 0 0 0 0)
   )
@@
   (junction (at 314.96 223.52) (diameter 0) (color 0 0 0 0)
   )
-  (junction (at 304.8 182.88) (diameter 0) (color 0 0 0 0)
-  )
   (junction (at 322.58 223.52) (diameter 0) (color 0 0 0 0)
   )
@@
     (stroke (width 0) (type default) (color 0 0 0 0))
   )
-  (wire (pts (xy 304.8 182.88) (xy 304.8 185.42))
-    (stroke (width 0) (type default) (color 0 0 0 0))
-  )
   (wire (pts (xy 309.88 223.52) (xy 312.42 223.52))
     (stroke (width 0) (type default) (color 0 0 0 0))
@@
     (stroke (width 0) (type default) (color 0 0 0 0))
   )
-  (wire (pts (xy 294.64 182.88) (xy 304.8 182.88))
+  (wire (pts (xy 294.64 182.88) (xy 317.5 182.88))
     (stroke (width 0) (type default) (color 0 0 0 0))
   )
@@
     (stroke (width 0) (type default) (color 0 0 0 0))
   )
-  (wire (pts (xy 304.8 182.88) (xy 317.5 182.88))
-    (stroke (width 0) (type default) (color 0 0 0 0))
-  )
   (wire (pts (xy 68.58 165.1) (xy 121.92 165.1))
     (stroke (width 0) (type default) (color 0 0 0 0))
@@
     (stroke (width 0) (type default) (color 0 0 0 0))
   )
-  (wire (pts (xy 304.8 193.04) (xy 304.8 190.5))
-    (stroke (width 0) (type default) (color 0 0 0 0))
-  )
   (wire (pts (xy 292.1 129.54) (xy 312.42 129.54))
     (stroke (width 0) (type default) (color 0 0 0 0))
@@
     (stroke (width 0) (type default) (color 0 0 0 0))
   )
-  (wire (pts (xy 294.64 193.04) (xy 304.8 193.04))
-    (stroke (width 0) (type default) (color 0 0 0 0))
-  )
   (wire (pts (xy 287.02 193.04) (xy 287.02 190.5))
     (stroke (width 0) (type default) (color 0 0 0 0))
@@
       (effects (font (size 1.27 1.27)) (justify right))
     )
-    (property "Value" "X" (id 1) (at 337.82 44.4499 0)
+    (property "Value" "300" (id 1) (at 337.82 44.4499 0)
       (effects (font (size 1.27 1.27)) (justify right))
     )
@@
       (effects (font (size 1.27 1.27)) (justify right))
     )
-    (property "Value" "X" (id 1) (at 393.7 46.9899 0)
+    (property "Value" "300" (id 1) (at 393.7 46.9899 0)
       (effects (font (size 1.27 1.27)) (justify right))
     )
@@
     (pin "2")
   )
-  (symbol (lib_name "SIM808_1") (lib_id "My_custom_lib:SIM808") (at 132.08 220.98 0) (unit 1)
+  (symbol (lib_id "My_custom_lib:SIM808") (at 132.08 220.98 0) (unit 1)
     (in_bom yes) (on_board yes) (fields_autoplaced)
     (property "Reference" "U1" (id 0) (at 164.465 183.9212 0))
@@
     (pin "18")
     (pin "2")
+    (pin "25")
     (pin "28")
     (pin "3")
@@
     (in_bom yes) (on_board yes) (fields_autoplaced)
     (property "Reference" "R9" (id 0) (at 269.24 54.61 90))
-    (property "Value" "100" (id 1) (at 269.24 57.15 90))
+    (property "Value" "60" (id 1) (at 269.24 57.15 90))
     (property "Footprint" "Resistor_SMD:R_0603_1608Metric_Pad0.98x0.95mm_HandSolder" (id 2) (at 269.24 60.96 0)
       (effects (font (size 1.27 1.27)) hide)
@@
       (effects (font (size 1.27 1.27)) (justify right))
     )
-    (property "Value" "X" (id 1) (at 284.48 46.9899 0)
+    (property "Value" "300" (id 1) (at 284.48 46.9899 0)
       (effects (font (size 1.27 1.27)) (justify right))
     )
@@
     (property "Reference" "D5" (id 0) (at 82.55 144.78 0))
     (property "Value" "D5V0P4UR6SO-7" (id 1) (at 82.55 147.32 0))
-    (property "Footprint" "SamacSys_Parts:SOT95P285X140-6N" (id 2) (at 72.39 160.02 0)
+    (property "Footprint" "SOT95P285X140-6N" (id 2) (at 72.39 160.02 0)
       (effects (font (size 1.27 1.27)) (justify left) hide)
     )
@@
     (pin "1")
   )
-  (symbol (lib_name "Conn_Coaxial_1") (lib_id "Connector:Conn_Coaxial") (at 220.98 190.5 0) (unit 1)
+  (symbol (lib_id "Connector:Conn_Coaxial") (at 220.98 190.5 0) (unit 1)
     (in_bom yes) (on_board yes) (fields_autoplaced)
     (property "Reference" "J2" (id 0) (at 223.52 189.5231 0)
@@
     (pin "2")
   )
-  (symbol (lib_id "Device:C_Small") (at 304.8 187.96 0) (unit 1)
-    (in_bom yes) (on_board yes) (fields_autoplaced)
-    (property "Reference" "C6" (id 0) (at 307.34 186.6962 0)
-      (effects (font (size 1.27 1.27)) (justify left))
-    )
-    (property "Value" "33p" (id 1) (at 307.34 189.2362 0)
-      (effects (font (size 1.27 1.27)) (justify left))
-    )
-    (property "Footprint" "Capacitor_SMD:C_0603_1608Metric_Pad1.08x0.95mm_HandSolder" (id 2) (at 304.8 187.96 0)
-      (effects (font (size 1.27 1.27)) hide)
-    )
-    (property "Datasheet" "~" (id 3) (at 304.8 187.96 0)
-      (effects (font (size 1.27 1.27)) hide)
-    )
-    (pin "1")
-    (pin "2")
-  )
   (symbol (lib_id "Device:R_Small") (at 55.88 81.28 90) (unit 1)
     (in_bom yes) (on_board yes) (fields_autoplaced)
     (property "Reference" "R15" (id 0) (at 55.88 74.93 90))
-    (property "Value" "100" (id 1) (at 55.88 77.47 90))
+    (property "Value" "60" (id 1) (at 55.88 77.47 90))
     (property "Footprint" "Resistor_SMD:R_0603_1608Metric_Pad0.98x0.95mm_HandSolder" (id 2) (at 55.88 81.28 0)
       (effects (font (size 1.27 1.27)) hide)
@@
     (in_bom yes) (on_board yes) (fields_autoplaced)
     (property "Reference" "R21" (id 0) (at 358.14 118.11 90))
-    (property "Value" "100" (id 1) (at 358.14 120.65 90))
+    (property "Value" "60" (id 1) (at 358.14 120.65 90))
     (property "Footprint" "Resistor_SMD:R_0603_1608Metric_Pad0.98x0.95mm_HandSolder" (id 2) (at 358.14 124.46 0)
       (effects (font (size 1.27 1.27)) hide)
@@
     (property "Reference" "IC1" (id 0) (at 64.77 172.72 0))
     (property "Value" "TXB0108PWR" (id 1) (at 64.77 175.26 0))
-    (property "Footprint" "SamacSys_Parts:SOP65P640X120-20N" (id 2) (at 74.93 177.8 0)
+    (property "Footprint" "SOP65P640X120-20N" (id 2) (at 74.93 177.8 0)
       (effects (font (size 1.27 1.27)) (justify left) hide)
     )
@@
       (effects (font (size 1.27 1.27)) (justify right))
     )
-    (property "Value" "100" (id 1) (at 111.76 41.9099 0)
+    (property "Value" "60" (id 1) (at 111.76 41.9099 0)
       (effects (font (size 1.27 1.27)) (justify right))
     )
@@
       (effects (font (size 1.27 1.27)) (justify left))
     )
-    (property "Value" "z" (id 1) (at 254 187.96 90)
+    (property "Value" "5v1" (id 1) (at 254 187.96 90)
       (effects (font (size 1.27 1.27)) (justify left))
     )
@@
     (in_bom yes) (on_board yes) (fields_autoplaced)
     (property "Reference" "R19" (id 0) (at 299.72 113.03 90))
-    (property "Value" "100" (id 1) (at 299.72 115.57 90))
+    (property "Value" "60" (id 1) (at 299.72 115.57 90))
     (property "Footprint" "Resistor_SMD:R_0603_1608Metric_Pad0.98x0.95mm_HandSolder" (id 2) (at 299.72 119.38 0)
       (effects (font (size 1.27 1.27)) hide)
@@
       (effects (font (size 1.27 1.27)) (justify right))
     )
-    (property "Value" "X" (id 1) (at 314.96 105.4099 0)
+    (property "Value" "300" (id 1) (at 314.96 105.4099 0)
       (effects (font (size 1.27 1.27)) (justify right))
     )
@@
     (property "Reference" "D7" (id 0) (at 367.03 226.06 0))
     (property "Value" "D5V0P4UR6SO-7" (id 1) (at 367.03 228.6 0))
-    (property "Footprint" "SamacSys_Parts:SOT95P285X140-6N" (id 2) (at 377.19 241.3 0)
+    (property "Footprint" "SOT95P285X140-6N" (id 2) (at 377.19 241.3 0)
       (effects (font (size 1.27 1.27)) (justify left) hide)
     )
@@
     (in_bom yes) (on_board yes) (fields_autoplaced)
     (property "Reference" "R10" (id 0) (at 378.46 54.61 90))
-    (property "Value" "100" (id 1) (at 378.46 57.15 90))
+    (property "Value" "60" (id 1) (at 378.46 57.15 90))
     (property "Footprint" "Resistor_SMD:R_0603_1608Metric_Pad0.98x0.95mm_HandSolder" (id 2) (at 378.46 60.96 0)
       (effects (font (size 1.27 1.27)) hide)
@@
       (effects (font (size 1.27 1.27)) (justify right))
     )
-    (property "Value" "100" (id 1) (at 60.96 41.9099 0)
+    (property "Value" "60" (id 1) (at 60.96 41.9099 0)
       (effects (font (size 1.27 1.27)) (justify right))
     )
@@
       (effects (font (size 1.27 1.27)) (justify right))
     )
-    (property "Value" "100" (id 1) (at 111.76 77.4699 0)
+    (property "Value" "60" (id 1) (at 111.76 77.4699 0)
       (effects (font (size 1.27 1.27)) (justify right))
     )
@@
     (in_bom yes) (on_board yes) (fields_autoplaced)
     (property "Reference" "R8" (id 0) (at 322.58 52.07 90))
-    (property "Value" "100" (id 1) (at 322.58 54.61 90))
+    (property "Value" "60" (id 1) (at 322.58 54.61 90))
     (property "Footprint" "Resistor_SMD:R_0603_1608Metric_Pad0.98x0.95mm_HandSolder" (id 2) (at 322.58 58.42 0)
       (effects (font (size 1.27 1.27)) hide)

Commit message: h
Parts:
- C3, C4: value 10u -> 22u; footprint Capacitor_SMD:C_0603_1608Metric_Pad1.08x0.95mm_HandSolder -> Capacitor_SMD:C_0805_2012Metric_Pad1.18x1.45mm_HandSolder
- D5, D7: footprint SOT95P285X140-6N -> SamacSys_Parts:SOT95P285X140-6N
- IC1: footprint SOP65P640X120-20N -> SamacSys_Parts:SOP65P640X120-20N
Changed lines of the file:
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@@
       (effects (font (size 1.27 1.27)) (justify left))
     )
-    (property "Value" "10u" (id 1) (at 280.67 189.2362 0)
-      (effects (font (size 1.27 1.27)) (justify left))
-    )
-    (property "Footprint" "Capacitor_SMD:C_0603_1608Metric_Pad1.08x0.95mm_HandSolder" (id 2) (at 278.13 187.96 0)
+    (property "Value" "22u" (id 1) (at 280.67 189.2362 0)
+      (effects (font (size 1.27 1.27)) (justify left))
+    )
+    (property "Footprint" "Capacitor_SMD:C_0805_2012Metric_Pad1.18x1.45mm_HandSolder" (id 2) (at 278.13 187.96 0)
       (effects (font (size 1.27 1.27)) hide)
     )
@@
       (effects (font (size 1.27 1.27)) (justify left))
     )
-    (property "Value" "10u" (id 1) (at 289.56 189.2362 0)
-      (effects (font (size 1.27 1.27)) (justify left))
-    )
-    (property "Footprint" "Capacitor_SMD:C_0603_1608Metric_Pad1.08x0.95mm_HandSolder" (id 2) (at 287.02 187.96 0)
+    (property "Value" "22u" (id 1) (at 289.56 189.2362 0)
+      (effects (font (size 1.27 1.27)) (justify left))
+    )
+    (property "Footprint" "Capacitor_SMD:C_0805_2012Metric_Pad1.18x1.45mm_HandSolder" (id 2) (at 287.02 187.96 0)
       (effects (font (size 1.27 1.27)) hide)
     )
@@
     (property "Reference" "D5" (id 0) (at 82.55 144.78 0))
     (property "Value" "D5V0P4UR6SO-7" (id 1) (at 82.55 147.32 0))
-    (property "Footprint" "SOT95P285X140-6N" (id 2) (at 72.39 160.02 0)
+    (property "Footprint" "SamacSys_Parts:SOT95P285X140-6N" (id 2) (at 72.39 160.02 0)
       (effects (font (size 1.27 1.27)) (justify left) hide)
     )
@@
     (property "Reference" "IC1" (id 0) (at 64.77 172.72 0))
     (property "Value" "TXB0108PWR" (id 1) (at 64.77 175.26 0))
-    (property "Footprint" "SOP65P640X120-20N" (id 2) (at 74.93 177.8 0)
+    (property "Footprint" "SamacSys_Parts:SOP65P640X120-20N" (id 2) (at 74.93 177.8 0)
       (effects (font (size 1.27 1.27)) (justify left) hide)
     )
@@
     (property "Reference" "D7" (id 0) (at 367.03 226.06 0))
     (property "Value" "D5V0P4UR6SO-7" (id 1) (at 367.03 228.6 0))
-    (property "Footprint" "SOT95P285X140-6N" (id 2) (at 377.19 241.3 0)
-      (effects (font (size 1.27 1.27)) (justify left) hide)
-    )
+    (property "Footprint" "SamacSys_Parts:SOT95P285X140-6N" (id 2) (at 377.19 241.3 0)
+      (effects (font (size 1.27 1.27)) (justify left) hide)
+    )

Commit message: r
Parts:
- added C81: 100n, Capacitor_SMD:C_0603_1608Metric_Pad1.08x0.95mm_HandSolder, symbol Device:C_Small
Connections:
- net +3V3: now also C81.1
- net GND: now also C81.2
Changed lines of the file:
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@@
   (junction (at 294.64 182.88) (diameter 0) (color 0 0 0 0)
+  )
+  (junction (at 20.32 166.37) (diameter 0) (color 0 0 0 0)
   )
   (junction (at 332.74 223.52) (diameter 0) (color 0 0 0 0)
@@
     (stroke (width 0) (type default) (color 0 0 0 0))
   )
+  (wire (pts (xy 25.4 177.8) (xy 25.4 175.26))
+    (stroke (width 0) (type default) (color 0 0 0 0))
+  )
+  (wire (pts (xy 20.32 166.37) (xy 20.32 182.88))
+    (stroke (width 0) (type default) (color 0 0 0 0))
+  )
   (wire (pts (xy 68.58 93.98) (xy 68.58 91.44))
     (stroke (width 0) (type default) (color 0 0 0 0))
@@
     (stroke (width 0) (type default) (color 0 0 0 0))
   )
-  (wire (pts (xy 20.32 172.72) (xy 20.32 182.88))
+  (wire (pts (xy 20.32 162.56) (xy 20.32 166.37))
     (stroke (width 0) (type default) (color 0 0 0 0))
   )
@@
     (stroke (width 0) (type default) (color 0 0 0 0))
   )
+  (wire (pts (xy 25.4 166.37) (xy 20.32 166.37))
+    (stroke (width 0) (type default) (color 0 0 0 0))
+  )
   (wire (pts (xy 294.64 182.88) (xy 294.64 185.42))
     (stroke (width 0) (type default) (color 0 0 0 0))
@@
   )
   (wire (pts (xy 302.26 223.52) (xy 304.8 223.52))
+    (stroke (width 0) (type default) (color 0 0 0 0))
+  )
+  (wire (pts (xy 25.4 170.18) (xy 25.4 166.37))
     (stroke (width 0) (type default) (color 0 0 0 0))
   )
@@
     (pin "1")
     (pin "2")
+  )
+  (symbol (lib_id "power:GND") (at 25.4 177.8 0) (unit 1)
+    (in_bom yes) (on_board yes) (fields_autoplaced)
+    (property "Reference" "#PWR0236" (id 0) (at 25.4 184.15 0)
+      (effects (font (size 1.27 1.27)) hide)
+    )
+    (property "Value" "GND" (id 1) (at 25.4 182.88 0)
+      (effects (font (size 1.27 1.27)) hide)
+    )
+    (property "Footprint" "" (id 2) (at 25.4 177.8 0)
+      (effects (font (size 1.27 1.27)) hide)
+    )
+    (property "Datasheet" "" (id 3) (at 25.4 177.8 0)
+      (effects (font (size 1.27 1.27)) hide)
+    )
+    (pin "1")
   )
   (symbol (lib_id "power:+3V3") (at 58.42 33.02 0) (unit 1)
@@
     (pin "2")
   )
-  (symbol (lib_id "power:+3V3") (at 20.32 172.72 0) (unit 1)
-    (in_bom yes) (on_board yes) (fields_autoplaced)
-    (property "Reference" "#PWR020" (id 0) (at 20.32 176.53 0)
-      (effects (font (size 1.27 1.27)) hide)
-    )
-    (property "Value" "+3V3" (id 1) (at 20.32 167.005 0))
-    (property "Footprint" "" (id 2) (at 20.32 172.72 0)
-      (effects (font (size 1.27 1.27)) hide)
-    )
-    (property "Datasheet" "" (id 3) (at 20.32 172.72 0)
+  (symbol (lib_id "power:+3V3") (at 20.32 162.56 0) (unit 1)
+    (in_bom yes) (on_board yes) (fields_autoplaced)
+    (property "Reference" "#PWR020" (id 0) (at 20.32 166.37 0)
+      (effects (font (size 1.27 1.27)) hide)
+    )
+    (property "Value" "+3V3" (id 1) (at 20.32 156.845 0))
+    (property "Footprint" "" (id 2) (at 20.32 162.56 0)
+      (effects (font (size 1.27 1.27)) hide)
+    )
+    (property "Datasheet" "" (id 3) (at 20.32 162.56 0)
       (effects (font (size 1.27 1.27)) hide)
     )
@@
       (effects (font (size 1.27 1.27)) hide)
     )
+    (pin "1")
+    (pin "2")
+  )
+  (symbol (lib_id "Device:C_Small") (at 25.4 172.72 0) (unit 1)
+    (in_bom yes) (on_board yes) (fields_autoplaced)
+    (property "Reference" "C81" (id 0) (at 27.94 171.4562 0)
+      (effects (font (size 1.27 1.27)) (justify left))
+    )
+    (property "Value" "100n" (id 1) (at 27.94 173.9962 0)
+      (effects (font (size 1.27 1.27)) (justify left))
+    )
+    (property "Footprint" "Capacitor_SMD:C_0603_1608Metric_Pad1.08x0.95mm_HandSolder" (id 2) (at 25.4 172.72 0)
+      (effects (font (size 1.27 1.27)) hide)
+    )
+    (property "Datasheet" "~" (id 3) (at 25.4 172.72 0)
+      (effects (font (size 1.27 1.27)) hide)
+    )

Commit message: K
Parts:
- added U21: eSIM, Z_mycustom_footprint_lib:eSIM, symbol My_custom_lib:eSIM
Connections:
- net +1V8: now also U21.8 (VCC)
- net GND: now also U21.1 (GND)
- net SIM_CLK: now also U21.6 (CLK)
- net SIM_IO: now also U21.2 (NC/IO), U21.3 (IO/NC)
- net SIM_RST: now also U21.7 (RST)
Changed lines of the file:
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@@
+    (stroke (width 0) (type default) (color 0 0 0 0))
+  )
+  (wire (pts (xy 190.5 142.24) (xy 190.5 144.78))
     (stroke (width 0) (type default) (color 0 0 0 0))
   )
@@
     (stroke (width 0) (type default) (color 0 0 0 0))
   )
+  (wire (pts (xy 167.64 134.62) (xy 177.8 134.62))
+    (stroke (width 0) (type default) (color 0 0 0 0))
+  )
   (wire (pts (xy 109.22 139.7) (xy 109.22 142.24))
     (stroke (width 0) (type default) (color 0 0 0 0))
@@
     (stroke (width 0) (type default) (color 0 0 0 0))
   )
+  (wire (pts (xy 167.64 129.54) (xy 177.8 129.54))
+    (stroke (width 0) (type default) (color 0 0 0 0))
+  )
   (wire (pts (xy 93.98 182.88) (xy 93.98 180.34))
     (stroke (width 0) (type default) (color 0 0 0 0))
@@
     (stroke (width 0) (type default) (color 0 0 0 0))
   )
+  (wire (pts (xy 167.64 132.08) (xy 177.8 132.08))
+    (stroke (width 0) (type default) (color 0 0 0 0))
+  )
   (wire (pts (xy 269.24 193.04) (xy 269.24 195.58))
     (stroke (width 0) (type default) (color 0 0 0 0))
@@
     (stroke (width 0) (type default) (color 0 0 0 0))
   )
+  (wire (pts (xy 190.5 116.84) (xy 190.5 119.38))
+    (stroke (width 0) (type default) (color 0 0 0 0))
+  )
   (wire (pts (xy 345.44 236.22) (xy 345.44 238.76))
     (stroke (width 0) (type default) (color 0 0 0 0))
@@
     (stroke (width 0) (type default) (color 0 0 0 0))
   )
+  (wire (pts (xy 167.64 127) (xy 167.64 129.54))
+    (stroke (width 0) (type default) (color 0 0 0 0))
+  )
   (wire (pts (xy 266.7 182.88) (xy 278.13 182.88))
     (stroke (width 0) (type default) (color 0 0 0 0))
@@
   )
   (wire (pts (xy 322.58 220.98) (xy 322.58 223.52))
+    (stroke (width 0) (type default) (color 0 0 0 0))
+  )
+  (wire (pts (xy 167.64 127) (xy 177.8 127))
     (stroke (width 0) (type default) (color 0 0 0 0))
   )
@@
     (effects (font (size 1.27 1.27)) (justify left bottom))
   )
+  (label "SIM_RST" (at 167.64 134.62 0)
+    (effects (font (size 1.27 1.27)) (justify left bottom))
+  )
   (label "SIM_CLK" (at 106.68 157.48 0)
     (effects (font (size 1.27 1.27)) (justify left bottom))
@@
     (effects (font (size 1.27 1.27)) (justify right bottom))
   )
+  (label "SIM_IO" (at 167.64 127 0)
+    (effects (font (size 1.27 1.27)) (justify left bottom))
+  )
   (label "DTR" (at 43.18 180.34 0)
     (effects (font (size 1.27 1.27)) (justify left bottom))
@@
   )
   (label "BT_RF2" (at 203.2 238.76 0)
+    (effects (font (size 1.27 1.27)) (justify left bottom))
+  )
+  (label "SIM_CLK" (at 167.64 132.08 0)
     (effects (font (size 1.27 1.27)) (justify left bottom))
   )
@@
     (pin "1")
   )
+  (symbol (lib_id "My_custom_lib:eSIM") (at 187.96 127 0) (unit 1)
+    (in_bom yes) (on_board yes) (fields_autoplaced)
+    (property "Reference" "U21" (id 0) (at 192.5194 116.84 0)
+      (effects (font (size 1.27 1.27)) (justify left))
+    )
+    (property "Value" "eSIM" (id 1) (at 192.5194 119.38 0)
+      (effects (font (size 1.27 1.27)) (justify left))
+    )
+    (property "Footprint" "Z_mycustom_footprint_lib:eSIM" (id 2) (at 187.96 114.3 0)
+      (effects (font (size 1.27 1.27)) hide)
+    )
+    (property "Datasheet" "" (id 3) (at 187.96 114.3 0)
+      (effects (font (size 1.27 1.27)) hide)
+    )
+    (pin "1")
+    (pin "2")
+    (pin "3")
+    (pin "4")
+    (pin "5")
+    (pin "6")
+    (pin "7")
+    (pin "8")
+  )
   (symbol (lib_id "Connector:SIM_Card_Shielded") (at 147.32 139.7 0) (unit 1)
-    (in_bom yes) (on_board yes) (fields_autoplaced)
-    (property "Reference" "J1" (id 0) (at 164.465 138.4299 0)
-      (effects (font (size 1.27 1.27)) (justify left))
-    )
-    (property "Value" "SIM_Card_Shielded" (id 1) (at 164.465 140.9699 0)
+    (in_bom yes) (on_board yes)
+    (property "Reference" "J1" (id 0) (at 147.32 124.46 0)
+      (effects (font (size 1.27 1.27)) (justify left))
+    )
+    (property "Value" "SIM_Card_Shielded" (id 1) (at 142.24 127 0)
       (effects (font (size 1.27 1.27)) (justify left))
     )
@@
     )
     (property "Datasheet" "" (id 3) (at 383.54 220.98 0)
+      (effects (font (size 1.27 1.27)) hide)
+    )
+    (pin "1")
+  )
+  (symbol (lib_id "power:GND") (at 190.5 144.78 0) (unit 1)
+    (in_bom yes) (on_board yes) (fields_autoplaced)
+    (property "Reference" "#PWR0238" (id 0) (at 190.5 151.13 0)
+      (effects (font (size 1.27 1.27)) hide)
+    )
+    (property "Value" "GND" (id 1) (at 190.5 149.86 0)
+      (effects (font (size 1.27 1.27)) hide)
+    )
+    (property "Footprint" "" (id 2) (at 190.5 144.78 0)
+      (effects (font (size 1.27 1.27)) hide)
+    )
+    (property "Datasheet" "" (id 3) (at 190.5 144.78 0)
       (effects (font (size 1.27 1.27)) hide)
     )
@@
       (effects (font (size 1.27 1.27)) hide)
     )
+    (pin "1")
+  )
+  (symbol (lib_id "power:+1V8") (at 190.5 116.84 0) (unit 1)
+    (in_bom yes) (on_board yes) (fields_autoplaced)
+    (property "Reference" "#PWR0237" (id 0) (at 190.5 120.65 0)
+      (effects (font (size 1.27 1.27)) hide)
+    )
+    (property "Value" "+1V8" (id 1) (at 190.5 111.76 0))
+    (property "Footprint" "" (id 2) (at 190.5 116.84 0)
+      (effects (font (size 1.27 1.27)) hide)
+    )
+    (property "Datasheet" "" (id 3) (at 190.5 116.84 0)
+      (effects (font (size 1.27 1.27)) hide)
+    )

Commit message: b
Other:
- title: (none) -> Bird Detection and Recognition System
Changed lines of the file:
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@@
 (kicad_sch (version 20211123) (generator eeschema)
   (paper "A3")
+  (title_block
+    (title "Bird Detection and Recognition System")
+    (rev "V0.1")
+  )
   (junction (at 96.52 53.34) (diameter 0) (color 0 0 0 0)
   )
