File: Bird_detector_V1/MCU.kicad_sch (KiCad schematic)
At the start: 2 parts, among them U1 ESP32-S3-MINI-1, U2 ESP32-S3-WROOM-1

Commit message: g
Parts:
- renumbered U1 to U2, U2 to U3
Changed lines of the file:
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@@
 (kicad_sch (version 20211123) (generator eeschema)
   (paper "A3")
+  (wire (pts (xy 31.75 233.68) (xy 31.75 237.49))
+    (stroke (width 0) (type default) (color 0 0 0 0))
+  )
+  (wire (pts (xy 29.21 238.76) (xy 29.21 233.68))
+    (stroke (width 0) (type default) (color 0 0 0 0))
+  )
   (wire (pts (xy 221.615 54.61) (xy 221.615 57.15))
     (stroke (width 0) (type default) (color 0 0 0 0))
   )
+  (wire (pts (xy 36.83 233.68) (xy 36.83 237.49))
+    (stroke (width 0) (type default) (color 0 0 0 0))
+  )
+  (wire (pts (xy 34.29 233.68) (xy 34.29 237.49))
+    (stroke (width 0) (type default) (color 0 0 0 0))
+  )
+  (wire (pts (xy 54.61 229.87) (xy 54.61 232.41))
+    (stroke (width 0) (type default) (color 0 0 0 0))
+  )
   (wire (pts (xy 219.075 54.61) (xy 219.075 57.15))
     (stroke (width 0) (type default) (color 0 0 0 0))
   )
+  (wire (pts (xy 57.15 229.87) (xy 57.15 232.41))
+    (stroke (width 0) (type default) (color 0 0 0 0))
+  )
+  (hierarchical_label "DTR" (shape input) (at 39.37 256.54 180)
+    (effects (font (size 1.27 1.27)) (justify right))
+  )
+  (hierarchical_label "SCK" (shape input) (at 36.83 233.68 90)
+    (effects (font (size 1.27 1.27)) (justify left))
+  )
+  (hierarchical_label "STAT" (shape input) (at 71.12 177.8 180)
+    (effects (font (size 1.27 1.27)) (justify right))
+  )
+  (hierarchical_label "CTS" (shape input) (at 39.37 266.7 180)
+    (effects (font (size 1.27 1.27)) (justify right))
+  )
+  (hierarchical_label "SD" (shape input) (at 31.75 233.68 90)
+    (effects (font (size 1.27 1.27)) (justify left))
+  )
+  (hierarchical_label "RX" (shape input) (at 39.37 271.78 180)
+    (effects (font (size 1.27 1.27)) (justify right))
+  )
+  (hierarchical_label "RTS" (shape input) (at 39.37 269.24 180)
+    (effects (font (size 1.27 1.27)) (justify right))
+  )
+  (hierarchical_label "SDA" (shape input) (at 54.61 232.41 270)
+    (effects (font (size 1.27 1.27)) (justify right))
+  )
+  (hierarchical_label "DCD" (shape input) (at 39.37 264.16 180)
+    (effects (font (size 1.27 1.27)) (justify right))
+  )
+  (hierarchical_label "RI" (shape input) (at 39.37 261.62 180)
+    (effects (font (size 1.27 1.27)) (justify right))
+  )
+  (hierarchical_label "RESET_AUDIO" (shape input) (at 29.21 233.68 90)
+    (effects (font (size 1.27 1.27)) (justify left))
+  )
+  (hierarchical_label "RESET_GSM" (shape input) (at 39.37 276.86 180)
+    (effects (font (size 1.27 1.27)) (justify right))
+  )
+  (hierarchical_label "ENABLE" (shape input) (at 80.01 243.84 180)
+    (effects (font (size 1.27 1.27)) (justify right))
+  )
+  (hierarchical_label "TX" (shape input) (at 39.37 274.32 180)
+    (effects (font (size 1.27 1.27)) (justify right))
+  )
+  (hierarchical_label "WS" (shape input) (at 34.29 233.68 90)
+    (effects (font (size 1.27 1.27)) (justify left))
+  )
+  (hierarchical_label "SCL" (shape input) (at 57.15 232.41 270)
+    (effects (font (size 1.27 1.27)) (justify right))
+  )
   (symbol (lib_id "Espressif:ESP32-S3-MINI-1") (at 117.475 83.82 0) (unit 1)
     (in_bom yes) (on_board yes) (fields_autoplaced)
-    (property "Reference" "U1" (id 0) (at 116.84 44.45 0))
+    (property "Reference" "U2" (id 0) (at 116.84 44.45 0))
     (property "Value" "ESP32-S3-MINI-1" (id 1) (at 116.84 46.99 0))
     (property "Footprint" "Espressif:ESP32-S3-MINI-1" (id 2) (at 117.475 125.73 0)
@@
   (symbol (lib_id "Espressif:ESP32-S3-WROOM-1") (at 118.11 162.56 0) (unit 1)
     (in_bom yes) (on_board yes) (fields_autoplaced)
-    (property "Reference" "U2" (id 0) (at 117.475 123.19 0))
+    (property "Reference" "U3" (id 0) (at 117.475 123.19 0))
     (property "Value" "ESP32-S3-WROOM-1" (id 1) (at 117.475 125.73 0))
     (property "Footprint" "Espressif:ESP32-S3-WROOM-1" (id 2) (at 118.11 201.93 0)
@@
   (symbol (lib_id "power:GND") (at 221.615 57.15 0) (unit 1)
     (in_bom yes) (on_board yes) (fields_autoplaced)
-    (property "Reference" "#PWR020" (id 0) (at 221.615 63.5 0)
+    (property "Reference" "#PWR036" (id 0) (at 221.615 63.5 0)
       (effects (font (size 1.27 1.27)) hide)
     )
@@
   (symbol (lib_id "power:GND") (at 219.075 57.15 0) (unit 1)
     (in_bom yes) (on_board yes) (fields_autoplaced)
-    (property "Reference" "#PWR019" (id 0) (at 219.075 63.5 0)
-      (effects (font (size 1.27 1.27)) hide)
-    )
+    (property "Reference" "#PWR035" (id 0) (at 219.075 63.5 0)
+      (effects (font (size 1.27 1.27)) hide)
+    )

Commit message: f
Changed lines of the file:
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@@
+    (effects (font (size 1.27 1.27)) (justify right))
+  )
+  (hierarchical_label "DATA3{slash}CS" (shape input) (at 104.14 243.84 180)
     (effects (font (size 1.27 1.27)) (justify right))
   )
   (hierarchical_label "SCK" (shape input) (at 36.83 233.68 90)
     (effects (font (size 1.27 1.27)) (justify left))
+  )
+  (hierarchical_label "DATA2" (shape input) (at 104.14 241.3 180)
+    (effects (font (size 1.27 1.27)) (justify right))
   )
   (hierarchical_label "STAT" (shape input) (at 71.12 177.8 180)
@@
   )
   (hierarchical_label "RX" (shape input) (at 39.37 271.78 180)
+    (effects (font (size 1.27 1.27)) (justify right))
+  )
+  (hierarchical_label "DATA0" (shape input) (at 104.14 256.54 180)
     (effects (font (size 1.27 1.27)) (justify right))
   )
@@
     (effects (font (size 1.27 1.27)) (justify right))
   )
+  (hierarchical_label "CMD" (shape input) (at 104.14 246.38 180)
+    (effects (font (size 1.27 1.27)) (justify right))
+  )
   (hierarchical_label "RESET_AUDIO" (shape input) (at 29.21 233.68 90)
     (effects (font (size 1.27 1.27)) (justify left))
@@
     (effects (font (size 1.27 1.27)) (justify right))
   )
+  (hierarchical_label "DATA1" (shape input) (at 104.14 259.08 180)
+    (effects (font (size 1.27 1.27)) (justify right))
+  )
   (hierarchical_label "ENABLE" (shape input) (at 80.01 243.84 180)
     (effects (font (size 1.27 1.27)) (justify right))
   )
+  (hierarchical_label "SCLK" (shape input) (at 104.14 251.46 180)
+    (effects (font (size 1.27 1.27)) (justify right))
+  )
   (hierarchical_label "TX" (shape input) (at 39.37 274.32 180)
+    (effects (font (size 1.27 1.27)) (justify right))
+  )
+  (hierarchical_label "CARD_DET" (shape input) (at 76.2 264.16 270)
     (effects (font (size 1.27 1.27)) (justify right))
   )
@@
   (symbol (lib_id "power:GND") (at 221.615 57.15 0) (unit 1)
     (in_bom yes) (on_board yes) (fields_autoplaced)
-    (property "Reference" "#PWR045" (id 0) (at 221.615 63.5 0)
+    (property "Reference" "#PWR056" (id 0) (at 221.615 63.5 0)
       (effects (font (size 1.27 1.27)) hide)
     )
@@
   (symbol (lib_id "power:GND") (at 219.075 57.15 0) (unit 1)
     (in_bom yes) (on_board yes) (fields_autoplaced)
-    (property "Reference" "#PWR044" (id 0) (at 219.075 63.5 0)
+    (property "Reference" "#PWR055" (id 0) (at 219.075 63.5 0)
       (effects (font (size 1.27 1.27)) hide)
     )

Commit message: j
Parts:
- removed U2: ESP32-S3-MINI-1, Espressif:ESP32-S3-MINI-1, symbol Espressif:ESP32-S3-MINI-1
Connections:
- net GND: now also U3.1 (GND), U3.40 (GND), U3.41 (GND)
- net D-: now reaches U3.13 (GPIO19/U1RTS/ADC2_CH8/CLK_OUT2/USB_D-)
- net D+: now reaches U3.14 (GPIO20/U1CTS/ADC2_CH9/CLK_OUT1/USB_D+)
- net +3V3: now reaches U3.2 (3V3)
Other:
- moved on the sheet: U3
Changed lines of the file:
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@@
 (kicad_sch (version 20211123) (generator eeschema)
   (paper "A3")
+  (junction (at 186.69 148.59) (diameter 0) (color 0 0 0 0)
+  )
+  (junction (at 186.69 151.13) (diameter 0) (color 0 0 0 0)
+  )
+  (wire (pts (xy 186.69 148.59) (xy 186.69 151.13))
+    (stroke (width 0) (type default) (color 0 0 0 0))
+  )
+  (wire (pts (xy 182.88 151.13) (xy 186.69 151.13))
+    (stroke (width 0) (type default) (color 0 0 0 0))
+  )
+  (wire (pts (xy 182.88 146.05) (xy 186.69 146.05))
+    (stroke (width 0) (type default) (color 0 0 0 0))
+  )
+  (wire (pts (xy 182.88 148.59) (xy 186.69 148.59))
+    (stroke (width 0) (type default) (color 0 0 0 0))
+  )
   (wire (pts (xy 31.75 233.68) (xy 31.75 237.49))
     (stroke (width 0) (type default) (color 0 0 0 0))
@@
     (stroke (width 0) (type default) (color 0 0 0 0))
   )
-  (wire (pts (xy 221.615 54.61) (xy 221.615 57.15))
-    (stroke (width 0) (type default) (color 0 0 0 0))
-  )
   (wire (pts (xy 36.83 233.68) (xy 36.83 237.49))
     (stroke (width 0) (type default) (color 0 0 0 0))
   )
+  (wire (pts (xy 17.78 148.59) (xy 64.77 148.59))
+    (stroke (width 0) (type default) (color 0 0 0 0))
+  )
   (wire (pts (xy 34.29 233.68) (xy 34.29 237.49))
     (stroke (width 0) (type default) (color 0 0 0 0))
   )
+  (wire (pts (xy 182.88 88.9) (xy 185.42 88.9))
+    (stroke (width 0) (type default) (color 0 0 0 0))
+  )
   (wire (pts (xy 54.61 229.87) (xy 54.61 232.41))
     (stroke (width 0) (type default) (color 0 0 0 0))
   )
-  (wire (pts (xy 219.075 54.61) (xy 219.075 57.15))
+  (wire (pts (xy 182.88 86.36) (xy 185.42 86.36))
+    (stroke (width 0) (type default) (color 0 0 0 0))
+  )
+  (wire (pts (xy 186.69 146.05) (xy 186.69 148.59))
+    (stroke (width 0) (type default) (color 0 0 0 0))
+  )
+  (wire (pts (xy 186.69 151.13) (xy 186.69 153.67))
     (stroke (width 0) (type default) (color 0 0 0 0))
   )
@@
     (stroke (width 0) (type default) (color 0 0 0 0))
   )
+  (global_label "D+" (shape input) (at 185.42 86.36 0) (fields_autoplaced)
+    (effects (font (size 1.27 1.27)) (justify left))
+    (property "Intersheet References" "${INTERSHEET_REFS}" (id 0) (at 190.6755 86.2806 0)
+      (effects (font (size 1.27 1.27)) (justify left) hide)
+    )
+  )
+  (global_label "D-" (shape input) (at 185.42 88.9 0) (fields_autoplaced)
+    (effects (font (size 1.27 1.27)) (justify left))
+    (property "Intersheet References" "${INTERSHEET_REFS}" (id 0) (at 190.6755 88.8206 0)
+      (effects (font (size 1.27 1.27)) (justify left) hide)
+    )
+  )
   (hierarchical_label "DTR" (shape input) (at 39.37 256.54 180)
     (effects (font (size 1.27 1.27)) (justify right))
@@
     (effects (font (size 1.27 1.27)) (justify right))
   )
-  (hierarchical_label "STAT" (shape input) (at 71.12 177.8 180)
+  (hierarchical_label "STAT" (shape input) (at 72.39 215.9 180)
     (effects (font (size 1.27 1.27)) (justify right))
   )
@@
     (effects (font (size 1.27 1.27)) (justify right))
   )
-  (hierarchical_label "CARD_DET" (shape input) (at 76.2 264.16 270)
+  (hierarchical_label "CARD_DET" (shape input) (at 104.14 262.89 180)
     (effects (font (size 1.27 1.27)) (justify right))
   )
@@
     (effects (font (size 1.27 1.27)) (justify right))
   )
-  (symbol (lib_id "Espressif:ESP32-S3-MINI-1") (at 117.475 83.82 0) (unit 1)
-    (in_bom yes) (on_board yes) (fields_autoplaced)
-    (property "Reference" "U2" (id 0) (at 116.84 44.45 0))
-    (property "Value" "ESP32-S3-MINI-1" (id 1) (at 116.84 46.99 0))
-    (property "Footprint" "Espressif:ESP32-S3-MINI-1" (id 2) (at 117.475 125.73 0)
-      (effects (font (size 1.27 1.27)) hide)
-    )
-    (property "Datasheet" "https://www.espressif.com/sites/default/files/documentation/esp32-s3-mini-1_mini-1u_datasheet_en.pdf" (id 3) (at 117.475 128.27 0)
+  (symbol (lib_id "power:+3V3") (at 17.78 148.59 0) (unit 1)
+    (in_bom yes) (on_board yes) (fields_autoplaced)
+    (property "Reference" "#PWR?" (id 0) (at 17.78 152.4 0)
+      (effects (font (size 1.27 1.27)) hide)
+    )
+    (property "Value" "+3V3" (id 1) (at 17.78 143.51 0))
+    (property "Footprint" "" (id 2) (at 17.78 148.59 0)
+      (effects (font (size 1.27 1.27)) hide)
+    )
+    (property "Datasheet" "" (id 3) (at 17.78 148.59 0)
       (effects (font (size 1.27 1.27)) hide)
     )
     (pin "1")
-    (pin "10")
-    (pin "11")
-    (pin "12")
-    (pin "13")
-    (pin "14")
-    (pin "15")
-    (pin "16")
-    (pin "17")
-    (pin "18")
-    (pin "19")
-    (pin "2")
-    (pin "20")
-    (pin "21")
-    (pin "22")
-    (pin "23")
-    (pin "24")
-    (pin "25")
-    (pin "26")
-    (pin "27")
-    (pin "28")
-    (pin "29")
-    (pin "3")
-    (pin "30")
-    (pin "31")
-    (pin "32")
-    (pin "33")
-    (pin "34")
-    (pin "35")
-    (pin "36")
-    (pin "37")
-    (pin "38")
-    (pin "39")
-    (pin "4")
-    (pin "40")
-    (pin "41")
-    (pin "42")
-    (pin "43")
-    (pin "44")
-    (pin "45")
-    (pin "46")
-    (pin "5")
-    (pin "6")
-    (pin "7")
-    (pin "8")
-    (pin "9")
-  )
-  (symbol (lib_id "Espressif:ESP32-S3-WROOM-1") (at 118.11 162.56 0) (unit 1)
-    (in_bom yes) (on_board yes) (fields_autoplaced)
-    (property "Reference" "U3" (id 0) (at 117.475 123.19 0))
-    (property "Value" "ESP32-S3-WROOM-1" (id 1) (at 117.475 125.73 0))
-    (property "Footprint" "Espressif:ESP32-S3-WROOM-1" (id 2) (at 118.11 201.93 0)
-      (effects (font (size 1.27 1.27)) hide)
-    )
-    (property "Datasheet" "https://www.espressif.com/sites/default/files/documentation/esp32-s3-wroom-1_wroom-1u_datasheet_en.pdf" (id 3) (at 118.11 204.47 0)
+  )
+  (symbol (lib_id "Espressif:ESP32-S3-WROOM-1") (at 124.46 118.11 0) (unit 1)
+    (in_bom yes) (on_board yes) (fields_autoplaced)
+    (property "Reference" "U3" (id 0) (at 123.825 78.74 0))
+    (property "Value" "ESP32-S3-WROOM-1" (id 1) (at 123.825 81.28 0))
+    (property "Footprint" "Espressif:ESP32-S3-WROOM-1" (id 2) (at 124.46 157.48 0)
+      (effects (font (size 1.27 1.27)) hide)
+    )
+    (property "Datasheet" "https://www.espressif.com/sites/default/files/documentation/esp32-s3-wroom-1_wroom-1u_datasheet_en.pdf" (id 3) (at 124.46 160.02 0)
       (effects (font (size 1.27 1.27)) hide)
     )
@@
     (pin "9")
   )
-  (symbol (lib_id "power:GND") (at 221.615 57.15 0) (unit 1)
-    (in_bom yes) (on_board yes) (fields_autoplaced)
-    (property "Reference" "#PWR056" (id 0) (at 221.615 63.5 0)
-      (effects (font (size 1.27 1.27)) hide)
-    )
-    (property "Value" "GND" (id 1) (at 221.615 62.23 0)
-      (effects (font (size 1.27 1.27)) hide)
-    )
-    (property "Footprint" "" (id 2) (at 221.615 57.15 0)
-      (effects (font (size 1.27 1.27)) hide)
-    )
-    (property "Datasheet" "" (id 3) (at 221.615 57.15 0)
+  (symbol (lib_id "power:GND") (at 186.69 153.67 0) (unit 1)
+    (in_bom yes) (on_board yes) (fields_autoplaced)
+    (property "Reference" "#PWR055" (id 0) (at 186.69 160.02 0)
+      (effects (font (size 1.27 1.27)) hide)
+    )
+    (property "Value" "GND" (id 1) (at 186.69 158.75 0)
+      (effects (font (size 1.27 1.27)) hide)
+    )
+    (property "Footprint" "" (id 2) (at 186.69 153.67 0)
+      (effects (font (size 1.27 1.27)) hide)
+    )
+    (property "Datasheet" "" (id 3) (at 186.69 153.67 0)
       (effects (font (size 1.27 1.27)) hide)
     )
     (pin "1")
   )
-  (symbol (lib_id "power:GND") (at 219.075 57.15 0) (unit 1)
-    (in_bom yes) (on_board yes) (fields_autoplaced)
-    (property "Reference" "#PWR055" (id 0) (at 219.075 63.5 0)
-      (effects (font (size 1.27 1.27)) hide)
-    )
-    (property "Value" "GND" (id 1) (at 219.075 62.23 0)
-      (effects (font (size 1.27 1.27)) hide)
-    )
-    (property "Footprint" "" (id 2) (at 219.075 57.15 0)
-      (effects (font (size 1.27 1.27)) hide)
-    )
-    (property "Datasheet" "" (id 3) (at 219.075 57.15 0)
-      (effects (font (size 1.27 1.27)) hide)
-    )
+  (symbol (lib_id "power:+3V3") (at 31.75 86.36 0) (unit 1)
+    (in_bom yes) (on_board yes) (fields_autoplaced)
+    (property "Reference" "#PWR?" (id 0) (at 31.75 90.17 0)
+      (effects (font (size 1.27 1.27)) hide)
+    )
+    (property "Value" "+3V3" (id 1) (at 31.75 81.28 0))
+    (property "Footprint" "" (id 2) (at 31.75 86.36 0)
+      (effects (font (size 1.27 1.27)) hide)
+    )
+    (property "Datasheet" "" (id 3) (at 31.75 86.36 0)
+      (effects (font (size 1.27 1.27)) hide)
+    )

Commit message: f
Parts:
- renumbered U3 to U2
Changed lines of the file:
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@@
   (symbol (lib_id "power:+3V3") (at 17.78 148.59 0) (unit 1)
     (in_bom yes) (on_board yes) (fields_autoplaced)
-    (property "Reference" "#PWR?" (id 0) (at 17.78 152.4 0)
+    (property "Reference" "#PWR057" (id 0) (at 17.78 152.4 0)
       (effects (font (size 1.27 1.27)) hide)
     )
@@
   (symbol (lib_id "Espressif:ESP32-S3-WROOM-1") (at 124.46 118.11 0) (unit 1)
     (in_bom yes) (on_board yes) (fields_autoplaced)
-    (property "Reference" "U3" (id 0) (at 123.825 78.74 0))
+    (property "Reference" "U2" (id 0) (at 123.825 78.74 0))
     (property "Value" "ESP32-S3-WROOM-1" (id 1) (at 123.825 81.28 0))
     (property "Footprint" "Espressif:ESP32-S3-WROOM-1" (id 2) (at 124.46 157.48 0)
@@
   (symbol (lib_id "power:GND") (at 186.69 153.67 0) (unit 1)
     (in_bom yes) (on_board yes) (fields_autoplaced)
-    (property "Reference" "#PWR055" (id 0) (at 186.69 160.02 0)
+    (property "Reference" "#PWR058" (id 0) (at 186.69 160.02 0)
       (effects (font (size 1.27 1.27)) hide)
     )
@@
   (symbol (lib_id "power:+3V3") (at 31.75 86.36 0) (unit 1)
     (in_bom yes) (on_board yes) (fields_autoplaced)
-    (property "Reference" "#PWR?" (id 0) (at 31.75 90.17 0)
+    (property "Reference" "#PWR056" (id 0) (at 31.75 90.17 0)
       (effects (font (size 1.27 1.27)) hide)
     )

Commit message: v
Parts:
- added C16, C19, C21: 100n, Capacitor_SMD:C_0603_1608Metric_Pad1.08x0.95mm_HandSolder, symbol Device:C_Small
- added C17, C18: 10u, Capacitor_SMD:C_0603_1608Metric_Pad1.08x0.95mm_HandSolder, symbol Device:C_Small
- added C20: 1u+, Capacitor_SMD:C_0603_1608Metric_Pad1.08x0.95mm_HandSolder, symbol Device:C_Small
- added D8, D9: LED_Small, LED_SMD:LED_0603_1608Metric_Pad1.05x0.95mm_HandSolder, symbol Device:LED_Small
- added JP1, JP2: Jumper_2_Open, Jumper:SolderJumper-2_P1.3mm_Open_RoundedPad1.0x1.5mm, symbol Jumper:Jumper_2_Open
- added Q6: BC847BS, symbol Device:Q_Dual_NPN_NPN_E1B1C2E2B2C1
- added R26: 1k, Resistor_SMD:R_0603_1608Metric_Pad0.98x0.95mm_HandSolder, symbol Device:R_Small
- added R27: 22k, Resistor_SMD:R_0603_1608Metric_Pad0.98x0.95mm_HandSolder, symbol Device:R_Small
- added R28: 47k, Resistor_SMD:R_0603_1608Metric_Pad0.98x0.95mm_HandSolder, symbol Device:R_Small
- added R29: 10K, Resistor_SMD:R_0603_1608Metric_Pad0.98x0.95mm_HandSolder, symbol Device:R_Small
- added R30, R31: X, Resistor_SMD:R_0603_1608Metric_Pad0.98x0.95mm_HandSolder, symbol Device:R_Small
- added R32: 10k+, Resistor_SMD:R_0603_1608Metric_Pad0.98x0.95mm_HandSolder, symbol Device:R_Small
- added R33, R34, R35: 10k, Resistor_SMD:R_0603_1608Metric_Pad0.98x0.95mm_HandSolder, symbol Device:R_Small
- added SW2: MCU_RESET, SamacSys_Parts:PTS526SK15SMTR2LFS, symbol Switch:SW_SPST
- added U2: CP2102N-Axx-xQFN24, Package_DFN_QFN:QFN-24-1EP_4x4mm_P0.5mm_EP2.6x2.6mm, symbol Interface_USB:CP2102N-Axx-xQFN24
- renumbered U2 to U3
Connections:
- net +3V3: now also C17.1, C18.1, C19.1, R32.2, R35.2
- net D+: now also JP1.2 (B), U2.3 (D+); no longer U3.14 (GPIO20/U1CTS/ADC2_CH9/CLK_OUT1/USB_D+)
- net D-: now also JP2.2 (B), U2.4 (D-); no longer U3.13 (GPIO19/U1RTS/ADC2_CH8/CLK_OUT2/USB_D-)
- net GND: now also C16.2, C17.2, C18.2, C19.2, C20.2, C21.2, R28.2, R29.2, SW2.2 (B), U2.2 (GND), U2.25 (GND)
- net GPIO_17: now reaches U3.10 (GPIO17/U1TXD/ADC2_CH6)
- net GPIO_18: now reaches U3.11 (GPIO18/U1RXD/ADC2_CH7/CLK_OUT3)
- net GPIO_08: now reaches U3.12 (GPIO8/TOUCH8/ADC1_CH7/SUBSPICS1)
- net GPIO_03: now reaches U3.15 (GPIO3/TOUCH3/ADC1_CH2)
- net GPIO_46: now reaches U3.16 (GPIO46)
- net GPIO_09: now reaches U3.17 (GPIO9/TOUCH9/ADC1_CH8/FSPIHD/SUBSPIHD)
- net GPIO_10: now reaches U3.18 (GPIO10/TOUCH10/ADC1_CH9/FSPICS0/FSPIIO4/SUBSPICS0)
- net GPIO_11: now reaches U3.19 (GPIO11/TOUCH11/ADC2_CH0/FSPID/FSPIIO5/SUBSPID)
- net GPIO_12: now reaches U3.20 (GPIO12/TOUCH12/ADC2_CH1/FSPICLK/FSPIIO6/SUBSPICLK)
- net GPIO_13: now reaches U3.21 (GPIO13/TOUCH13/ADC2_CH2/FSPIQ/FSPIIO7/SUBSPIQ)
- net GPIO_14: now reaches U3.22 (GPIO14/TOUCH14/ADC2_CH3/FSPIWP/FSPIDQS/SUBSPIWP)
- net GPIO_21: now reaches U3.23 (GPIO21)
- net GPIO_47: now reaches U3.24 (GPIO47/SPICLK_P/SUBSPICLK_P_DIFF)
- net GPIO_48: now reaches U3.25 (GPIO48/SPICLK_N/SUBSPICLK_N_DIFF)
- net GPIO_45: now reaches U3.26 (GPIO45)
- net BOOT: now reaches U3.27 (GPIO0/BOOT)
- net BOOT: now also C21.1, Q6.3 (C2), R35.1
- net GPIO_35: now reaches U3.28 (SPIIO6/GPIO35/FSPID/SUBSPID)
- net GPIO_36: now reaches U3.29 (SPIIO7/GPIO36/FSPICLK/SUBSPICLK)
- net EN: now reaches U3.3 (EN)
- net EN: now also C20.1, Q6.6 (C1), R32.1, SW2.1 (A)
- net GPIO_37: now reaches U3.30 (SPIDQS/GPIO37/FSPIQ/SUBSPIQ)
- net GPIO_38: now reaches U3.31 (GPIO38/FSPIWP/SUBSPIWP)
- net GPIO_39: now reaches U3.32 (MTCK/GPIO39/CLK_OUT3/SUBSPICS1)
- net GPIO_40: now reaches U3.33 (MTDO/GPIO40/CLK_OUT2)
- net GPIO_41: now reaches U3.34 (MTDI/GPIO41/CLK_OUT1)
- net GPIO_42: now reaches U3.35 (MTMS/GPIO42)
- net UART0_RX: now reaches U3.36 (U0RXD/GPIO44/CLK_OUT2)
- net UART0_RX: now also U2.21 (TXD)
- net UART0_TX: now reaches U3.37 (U0TXD/GPIO43/CLK_OUT1)
- net UART0_TX: now also U2.20 (RXD)
- net GPIO_02: now reaches U3.38 (GPIO2/TOUCH2/ADC1_CH1)
- net GPIO_01: now reaches U3.39 (GPIO1/TOUCH1/ADC1_CH0)
- net GPIO_04: now reaches U3.4 (GPIO4/TOUCH4/ADC1_CH3)
- net GPIO_05: now reaches U3.5 (GPIO5/TOUCH5/ADC1_CH4)
- net GPIO_06: now reaches U3.6 (GPIO6/TOUCH6/ADC1_CH5)
- net GPIO_07: now reaches U3.7 (GPIO7/TOUCH7/ADC1_CH6)
- net GPIO_15: now reaches U3.8 (GPIO15/U0RTS/ADC2_CH4/XTAL_32K_P)
- net GPIO_16: now reaches U3.9 (GPIO16/U0CTS/ADC2_CH5/XTAL_32K_NH5)
- new net: R29.1, U2.15 (~{SUSPEND})
- new net: D9.1 (K), R31.2
- new net: D8.1 (K), R30.2
- new net +5V: R27.1
- new net BASE1: Q6.2 (B1), R33.1
- new net BASE2: Q6.5 (B2), R34.2
- new net ESP32_D+: JP1.1 (A), U3.14 (GPIO20/U1CTS/ADC2_CH9/CLK_OUT1/USB_D+)
- new net ESP32_D-: JP2.1 (A), U3.13 (GPIO19/U1RTS/ADC2_CH8/CLK_OUT2/USB_D-)
- new net RXT: R31.1, U2.13 (~{RXT}/GPIO.1)
- new net TXT: R30.1, U2.14 (~{TXT}/GPIO.0)
- new net VBUS_DETECT_CP: R27.2, R28.1, U2.8 (VBUS)
- new net VDD_CP: C16.1, U2.6 (VDD), U2.7 (VREGIN)
- new net VIO: D8.2 (A), D9.2 (A), R26.2, U2.5 (VIO)
- new net ~{CTS}: U2.18 (~{CTS})
- new net ~{DCD}: U2.24 (~{DCD})
- new net ~{DSR}: U2.22 (~{DSR})
- new net ~{DTR}: Q6.4 (E2), R33.2, U2.23 (~{DTR})
- new net ~{RI}: U2.1 (~{RI}/CLK)
- new net ~{RST_CP}: R26.1, U2.9 (~{RST})
- new net ~{RTS}: Q6.1 (E1), R34.1, U2.19 (~{RTS})
- no-connect marks 0 -> 6
Other:
- note added: "ESP32-S3 has four strapping pins: • GPIO0 • GPIO45 • GPIO46 • GPIO3 GPIO0, GPIO45 and GPIO46 are connected to the chip's internal weak pull-up/pull-down during the chip reset. GPIO3 is floating by default"
- note added: "Internal Pull-up/down 45k Max IC typical current: source 40mA sink 28mA EN pin TTL: 0.75*Vcc+ HIGH 0.25*Vcc- LOW"
- note added: "RC delay"
- moved on the sheet: U3
