File: Bird_detector_V1/MCU.kicad_sch (KiCad schematic)
At the start: 24 parts, among them Q6 BC847BS, SW2 MCU_RESET, U2 CP2102N-Axx-xQFN24, U3 ESP32-S3-WROOM-1

Commit message: f
Parts:
- removed JP1, JP2: Jumper_2_Open, Jumper:SolderJumper-2_P1.3mm_Open_RoundedPad1.0x1.5mm, symbol Jumper:Jumper_2_Open
- added C19, C56: 100n, Capacitor_SMD:C_0603_1608Metric_Pad1.08x0.95mm_HandSolder, symbol Device:C_Small
- added C57: 4.7n, Capacitor_SMD:C_0603_1608Metric_Pad1.08x0.95mm_HandSolder, symbol Device:C_Small
- added J12: Screw_Terminal_01x03, TerminalBlock:TerminalBlock_Altech_AK300-3_P5.00mm, symbol Connector:Screw_Terminal_01x03
- added JP1: ADR0, Jumper:SolderJumper-3_P1.3mm_Bridged12_RoundedPad1.0x1.5mm_NumberLabels, symbol Jumper:SolderJumper_3_Bridged12
- added NT2: NetTie_2, NetTie:NetTie-2_SMD_Pad0.5mm, symbol Device:NetTie_2
- added R72, R73: 10k, Resistor_SMD:R_0603_1608Metric_Pad0.98x0.95mm_HandSolder, symbol Device:R_Small
- added R74, R76: 60, Resistor_SMD:R_0603_1608Metric_Pad0.98x0.95mm_HandSolder, symbol Device:R_Small
- added R75: 300, Resistor_SMD:R_0603_1608Metric_Pad0.98x0.95mm_HandSolder, symbol Device:R_Small
- added U14: 74LVC1G08, Package_TO_SOT_SMD:SOT-23-5_HandSoldering, symbol 74xGxx:74LVC1G08
- added U15: MCP2561-H-SN, Package_SO:SOIC-8_3.9x4.9mm_P1.27mm, symbol Interface_CAN_LIN:MCP2561-H-SN
- added U3: BME280, Package_LGA:Bosch_LGA-8_2.5x2.5mm_P0.65mm_ClockwisePinNumbering, symbol Sensor:BME280
- C20: value 1u+ -> z
- R27: renamed from R32; value 10k+ -> y
- renumbered C17 to C16, C18 to C17, C19 to C18, C16 to C22, R29 to R26, R35 to R28, R26 to R29, R34 to R30, R33 to R31, R27 to R32, R28 to R33, R30 to R34, R31 to R35, U3 to U2, U2 to U4
Connections:
- net GND is gone; now on net +3V3: C16.2, C17.2, C18.2, C20.2, C21.2, C22.2, R26.2, R33.2, SW2.2 (B), U2.1 (GND), U2.40 (GND), U2.41 (GND), U4.2 (GND), U4.25 (GND)
- net GPIO_04 is gone; now on net CARD_DET: U2.4 (GPIO4/TOUCH4/ADC1_CH3)
- net GPIO_05 is gone; now on net DATA1: U2.5 (GPIO5/TOUCH5/ADC1_CH4)
- net GPIO_06 is gone; now on net DATA0: U2.6 (GPIO6/TOUCH6/ADC1_CH5)
- net GPIO_07 is gone; now on net SCLK: U2.7 (GPIO7/TOUCH7/ADC1_CH6)
- net GPIO_08 is gone; now on net DCD: U2.12 (GPIO8/TOUCH8/ADC1_CH7/SUBSPICS1)
- net GPIO_09 is gone; now on net STAT: U2.17 (GPIO9/TOUCH9/ADC1_CH8/FSPIHD/SUBSPIHD)
- net GPIO_10 is gone; now on net RESET_GSM: U2.18 (GPIO10/TOUCH10/ADC1_CH9/FSPICS0/FSPIIO4/SUBSPICS0)
- net GPIO_11 is gone; now on net TX: U2.19 (GPIO11/TOUCH11/ADC2_CH0/FSPID/FSPIIO5/SUBSPID)
- net GPIO_12 is gone; now on net RX: U2.20 (GPIO12/TOUCH12/ADC2_CH1/FSPICLK/FSPIIO6/SUBSPICLK)
- net GPIO_13 is gone; now on net RTS: U2.21 (GPIO13/TOUCH13/ADC2_CH2/FSPIQ/FSPIIO7/SUBSPIQ)
- net GPIO_14 is gone; now on net CTS: U2.22 (GPIO14/TOUCH14/ADC2_CH3/FSPIWP/FSPIDQS/SUBSPIWP)
- net GPIO_15 is gone; now on net CMD: U2.8 (GPIO15/U0RTS/ADC2_CH4/XTAL_32K_P)
- net GPIO_16 is gone; now on net DATA3/CS: U2.9 (GPIO16/U0CTS/ADC2_CH5/XTAL_32K_NH5)
- net GPIO_17 is gone; now on net DATA2: U2.10 (GPIO17/U1TXD/ADC2_CH6)
- net GPIO_18 is gone; now on net RI: U2.11 (GPIO18/U1RXD/ADC2_CH7/CLK_OUT3)
- net GPIO_21 is gone; now on net SD: U2.23 (GPIO21)
- net GPIO_35 is gone; now on net SCL: U2.28 (SPIIO6/GPIO35/FSPID/SUBSPID)
- net GPIO_36 is gone; now on net SDA: U2.29 (SPIIO7/GPIO36/FSPICLK/SUBSPICLK)
- net GPIO_37 is gone; now on net DTR: U2.30 (SPIDQS/GPIO37/FSPIQ/SUBSPIQ)
- net GPIO_38 is gone; now on net RESET_AUDIO: U2.31 (GPIO38/FSPIWP/SUBSPIWP)
- net GPIO_47 is gone; now on net WS: U2.24 (GPIO47/SPICLK_P/SUBSPICLK_P_DIFF)
- net GPIO_48 is gone; now on net SCK: U2.25 (GPIO48/SPICLK_N/SUBSPICLK_N_DIFF)
- net +3V3: now also C19.1, C19.2, C56.1, C56.2, C57.2, J12.3 (Pin_3), JP1.1 (A), JP1.3 (B), NT2.2, R72.2, R73.1, U14.3 (GND), U14.5 (VCC), U15.2 (VSS), U15.3 (VDD), U3.1 (GND), U3.6 (VDDIO), U3.7 (GND), U3.8 (VDD); no longer R27.2
- net ENABLE: now also U14.4
- net GPIO_01: now also U14.2
- net GPIO_02: now also U15.8 (STBY)
- net GPIO_41: now also U15.4 (RXD)
- net GPIO_42: now also U15.1 (TXD)
- net SCL: now also R73.2, U3.4 (SCK)
- net SDA: now also R72.1, U3.3 (SDI)
- net ESP32_D+ renamed USB_OTG_D+
- net ESP32_D- renamed USB_OTG_D-
- new net: C57.1, R74.1, R75.2, R76.2
- new net: JP1.2 (C), U3.5 (SDO)
- new net CAN_H: J12.1 (Pin_1), R76.1, U15.7 (CANH)
- new net CAN_L: J12.2 (Pin_2), R74.2, U15.6 (CANL)
- new net CSB: NT2.1, U3.2 (CSB)
- new net PG_3V3: R27.2
- new net PG_3V8: U14.1
- new net SPLIT: R75.1, U15.5 (SPLIT)
- no-connect marks 6 -> 9
Other:
- note added: "Danger pins"
- note added: "Free pins"
- note added: "GSM UART + COMMANDS"
- note added: "I2C BUS"
- note added: "I2S BUS"
- note added: "NMOS and gate?"
- note added: "NOTE: PG 1Meg R so for delay in ms is cap rating in nF ex: 15ms => 15nF"
- note added: "RC delay recomanded min 10ms wanted 15-20ms"
- note added: "SD CARD data SPI/2/4bit"
- note removed: "RC delay"

Commit message: v
Parts:
- removed U14: 74LVC1G08, Package_TO_SOT_SMD:SOT-23-5_HandSoldering, symbol 74xGxx:74LVC1G08
- added C16: 4p7-10p, Capacitor_SMD:C_0603_1608Metric_Pad1.08x0.95mm_HandSolder, symbol Device:C_Small
- added C18: 100n, Capacitor_SMD:C_0603_1608Metric_Pad1.08x0.95mm_HandSolder, symbol Device:C_Small
- added J6: USB1046-GF-0190-L-B-A, USB1046GF0190LBA, symbol SamacSys_Parts:USB1046-GF-0190-L-B-A
- added Q1: SSM6N7002, Package_TO_SOT_SMD:SOT-363_SC-70-6_Handsoldering, symbol Device:Q_Dual_NMOS_S1G1D2S2G2D1
- added R27: 1Meg, Resistor_SMD:R_0603_1608Metric_Pad0.98x0.95mm_HandSolder, symbol Device:R_Small
- added R93: 10k, Resistor_SMD:R_0603_1608Metric_Pad0.98x0.95mm_HandSolder, symbol Device:R_Small
- added R94: 100, Resistor_SMD:R_0603_1608Metric_Pad0.98x0.95mm_HandSolder, symbol Device:R_Small
- added R95: 100k, Resistor_SMD:R_0603_1608Metric_Pad0.98x0.95mm_HandSolder, symbol Device:R_Small
- added U6: 74LVC1G08, Package_SO:TSOP-5_1.65x3.05mm_P0.95mm, symbol My_custom_lib:74LVC1G08
- renumbered C22 to C17, C16 to C19, C17 to C20, C18 to C21, C56 to C22, C20 to C23, C57 to C24, C21 to C25, C19 to C26, J12 to J7, JP1 to JP2, R29 to R26, R32 to R28, R33 to R29, R26 to R30, R34 to R31, R35 to R32, R27 to R33, R31 to R34, R72 to R35, R73 to R36, R74 to R37, R75 to R38, R76 to R39, R30 to R40, R28 to R41, U4 to U2, U2 to U3, U15 to U4, U3 to U5
Connections:
- net +3V3: now also U6.5 (VCC); no longer C17.2, C19.2, C20.2, C21.2, C22.2, C23.2, C24.2, C25.2, C26.2, J7.3 (Pin_3), JP2.1 (A), R29.2, R30.2, SW2.2 (B), U2.2 (GND), U2.25 (GND), U3.1 (GND), U3.40 (GND), U3.41 (GND), U4.2 (VSS), U5.1 (GND), U5.7 (GND)
- net ENABLE: now also U6.4
- net GPIO_01: now also U6.1
- net GPIO_40: now also R94.2, R95.2
- net PG_3V8: now also U6.2
- net USB_OTG_D+: now also J6.3
- net USB_OTG_D-: now also J6.2
- net ~{RST_CP}: now also C18.1
- new net: Q1.2 (G), R94.1
- new net GND: C16.2, C17.2, C18.2, C19.2, C20.2, C21.2, C22.2, C23.2, C24.2, C25.2, C26.2, J6.4, J7.3 (Pin_3), JP2.1 (A), Q1.1 (S), R27.2, R29.2, R30.2, R95.1, SW2.2 (B), U2.2 (GND), U2.25 (GND), U3.1 (GND), U3.40 (GND), U3.41 (GND), U4.2 (VSS), U5.1 (GND), U5.7 (GND), U6.3 (GND)
- new net HEAT: Q1.6 (D), R93.2
- new net Shield3: C16.1, J6.MH1, J6.MH2, R27.1
- new net VBUS: J6.1
- new net VDC: R93.1
- no-connect marks 9 -> 8
Other:
- note added: "Heater controll"
- note removed: "NMOS and gate?"
- moved on the sheet: C19, C20, C21, C26, J7, U3

Commit message: v
Parts:
- removed C16: 4p7-10p, Capacitor_SMD:C_0603_1608Metric_Pad1.08x0.95mm_HandSolder, symbol Device:C_Small
- removed J6: USB1046-GF-0190-L-B-A, USB1046GF0190LBA, symbol SamacSys_Parts:USB1046-GF-0190-L-B-A
- removed R27: 1Meg, Resistor_SMD:R_0603_1608Metric_Pad0.98x0.95mm_HandSolder, symbol Device:R_Small
Connections:
- net GPIO_39 renamed INT_EXTENDER
- no-connect marks 8 -> 7

Commit message: f
Parts:
- removed R33: y, Resistor_SMD:R_0603_1608Metric_Pad0.98x0.95mm_HandSolder, symbol Device:R_Small
- added C32: DNP, Capacitor_SMD:C_0603_1608Metric_Pad1.08x0.95mm_HandSolder, symbol Device:C_Small
- added C75: 4.7n, Capacitor_SMD:C_0603_1608Metric_Pad1.08x0.95mm_HandSolder, symbol Device:C_Small
- C23: value z -> 15n
- R30: value 10K -> 10k
- R31, R32: value X -> 300
- R94: value 100 -> 60
Connections:
- net EN is gone; now on net PG_3V3: C23.1, Q6.6 (C1), SW2.1 (A), U3.3 (EN)
- net +3V3: now also C75.1
- net GND: now also C32.2, C75.2
- net PG_3V3: now also C32.1
Other:
- moved on the sheet: C19, C20, C21

Commit message: h
Parts:
- removed C19: 10u, Capacitor_SMD:C_0603_1608Metric_Pad1.08x0.95mm_HandSolder, symbol Device:C_Small
- added NT3, NT4: NetTie_2, NetTie:NetTie-2_SMD_Pad0.5mm, symbol Device:NetTie_2
- added R100, R101: ESD, Resistor_SMD:R_0603_1608Metric_Pad0.98x0.95mm_HandSolder, symbol Device:R_Small
- C20: value 10u -> 22u; footprint Capacitor_SMD:C_0603_1608Metric_Pad1.08x0.95mm_HandSolder -> Capacitor_SMD:C_0805_2012Metric_Pad1.18x1.45mm_HandSolder
- Q6: footprint (none) -> Package_TO_SOT_SMD:SOT-363_SC-70-6_Handsoldering
Connections:
- net CAN_H: now also R101.1
- net CAN_L: now also R100.1
- net GND: now also R100.2, R101.2
- net SCL: now also NT4.1; no longer U3.28 (SPIIO6/GPIO35/FSPID/SUBSPID)
- net SDA: now also NT3.1; no longer U3.29 (SPIIO7/GPIO36/FSPICLK/SUBSPICLK)
- new net GPIO_35: NT4.2, U3.28 (SPIIO6/GPIO35/FSPID/SUBSPID)
- new net GPIO_36: NT3.2, U3.29 (SPIIO7/GPIO36/FSPICLK/SUBSPICLK)
Other:
- added sheet test (untitled.kicad_sch)
- moved on the sheet: J7

Commit message: r
Parts:
- added R107, R108: 10k, Resistor_SMD:R_0603_1608Metric_Pad0.98x0.95mm_HandSolder, symbol Device:R_Small
Connections:
- net GPIO_46 is gone; now on net CHG_EN: U3.16 (GPIO46)
- net +3V3: now also R107.2, R108.1
- net SCL: now also R108.2
- net SDA: now also R107.1
- no-connect marks 7 -> 6
Other:
- note added: "Straping pin that is in pull down default. There is a 100k discrete pull down too."
- moved on the sheet: Q1A, R93, R94, R95

Commit message: K
Parts:
- removed NT2: NetTie_2, NetTie:NetTie-2_SMD_Pad0.5mm, symbol Device:NetTie_2
- added R109: 300, Resistor_SMD:R_0603_1608Metric_Pad0.98x0.95mm_HandSolder, symbol Device:R_Small
Connections:
- net CSB is gone; now on net +3V3: U5.2 (CSB)
- net RESET_AUDIO: now also R109.1; no longer U3.31 (GPIO38/FSPIWP/SUBSPIWP)
- new net GPIO_38: R109.2, U3.31 (GPIO38/FSPIWP/SUBSPIWP)

Commit message: b
Parts:
- added J18: Conn_02x02_Odd_Even, Connector_PinHeader_2.54mm:PinHeader_2x02_P2.54mm_Vertical_SMD, symbol Connector_Generic:Conn_02x02_Odd_Even
Connections:
- net +3V3: now also J18.2 (Pin_2)
- net CAN_H: now also J7.3 (Pin_3); no longer J7.1 (Pin_1)
- net GND: now also J7.1 (Pin_1), J18.3 (Pin_3); no longer J7.3 (Pin_3)
- net SCL: now also J18.1 (Pin_1)
- net SDA: now also J18.4 (Pin_4)
Other:
- title: (none) -> Bird Detection and Recognition System
Changed lines of the file:
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@@
 (kicad_sch (version 20211123) (generator eeschema)
   (paper "A3")
+  (title_block
+    (title "Bird Detection and Recognition System")
+    (rev "V0.1")
+  )
   (junction (at 317.5 168.91) (diameter 0) (color 0 0 0 0)
   )
@@
     (stroke (width 0) (type default) (color 0 0 0 0))
   )
+  (wire (pts (xy 257.81 237.49) (xy 257.81 241.3))
+    (stroke (width 0) (type default) (color 0 0 0 0))
+  )
   (wire (pts (xy 247.65 176.53) (xy 247.65 189.23))
     (stroke (width 0) (type default) (color 0 0 0 0))
@@
     (stroke (width 0) (type default) (color 0 0 0 0))
   )
+  (wire (pts (xy 270.51 234.95) (xy 278.13 234.95))
+    (stroke (width 0) (type default) (color 0 0 0 0))
+  )
   (wire (pts (xy 185.42 93.98) (xy 191.77 93.98))
     (stroke (width 0) (type default) (color 0 0 0 0))
@@
     (stroke (width 0) (type default) (color 0 0 0 0))
   )
+  (wire (pts (xy 270.51 237.49) (xy 279.4 237.49))
+    (stroke (width 0) (type default) (color 0 0 0 0))
+  )
   (wire (pts (xy 54.61 119.38) (xy 71.12 119.38))
     (stroke (width 0) (type default) (color 0 0 0 0))
@@
     (stroke (width 0) (type default) (color 0 0 0 0))
   )
+  (wire (pts (xy 278.13 231.14) (xy 278.13 234.95))
+    (stroke (width 0) (type default) (color 0 0 0 0))
+  )
   (wire (pts (xy 64.77 71.12) (xy 71.12 71.12))
     (stroke (width 0) (type default) (color 0 0 0 0))
@@
   )
   (wire (pts (xy 139.7 181.61) (xy 139.7 185.42))
+    (stroke (width 0) (type default) (color 0 0 0 0))
+  )
+  (wire (pts (xy 257.81 234.95) (xy 248.92 234.95))
     (stroke (width 0) (type default) (color 0 0 0 0))
   )
@@
     (effects (font (size 1.27 1.27)) (justify left bottom))
   )
+  (label "SCL" (at 248.92 234.95 0)
+    (effects (font (size 1.27 1.27)) (justify left bottom))
+  )
   (label "GPIO_17" (at 81.28 196.85 0)
     (effects (font (size 1.27 1.27)) (justify left bottom))
@@
   (label "TXT" (at 314.96 82.55 0)
     (effects (font (size 1.27 1.27)) (justify left bottom))
+  )
+  (label "SDA" (at 279.4 237.49 180)
+    (effects (font (size 1.27 1.27)) (justify right bottom))
   )
   (label "CAN_L" (at 227.33 181.61 0)
@@
     (pin "5")
   )
+  (symbol (lib_id "power:GND") (at 257.81 241.3 0) (unit 1)
+    (in_bom yes) (on_board yes) (fields_autoplaced)
+    (property "Reference" "#PWR0224" (id 0) (at 257.81 247.65 0)
+      (effects (font (size 1.27 1.27)) hide)
+    )
+    (property "Value" "GND" (id 1) (at 257.81 246.38 0)
+      (effects (font (size 1.27 1.27)) hide)
+    )
+    (property "Footprint" "" (id 2) (at 257.81 241.3 0)
+      (effects (font (size 1.27 1.27)) hide)
+    )
+    (property "Datasheet" "" (id 3) (at 257.81 241.3 0)
+      (effects (font (size 1.27 1.27)) hide)
+    )
+    (pin "1")
+  )
   (symbol (lib_id "Device:R_Small") (at 147.32 187.96 0) (unit 1)
     (in_bom yes) (on_board yes) (fields_autoplaced)
@@
     )
     (property "Datasheet" "" (id 3) (at 317.5 210.82 0)
+      (effects (font (size 1.27 1.27)) hide)
+    )
+    (pin "1")
+  )
+  (symbol (lib_id "power:+3V3") (at 278.13 231.14 0) (unit 1)
+    (in_bom yes) (on_board yes) (fields_autoplaced)
+    (property "Reference" "#PWR0227" (id 0) (at 278.13 234.95 0)
+      (effects (font (size 1.27 1.27)) hide)
+    )
+    (property "Value" "+3V3" (id 1) (at 278.13 226.06 0))
+    (property "Footprint" "" (id 2) (at 278.13 231.14 0)
+      (effects (font (size 1.27 1.27)) hide)
+    )
+    (property "Datasheet" "" (id 3) (at 278.13 231.14 0)
       (effects (font (size 1.27 1.27)) hide)
     )
@@
     (pin "8")
   )
+  (symbol (lib_id "Connector_Generic:Conn_02x02_Odd_Even") (at 262.89 234.95 0) (unit 1)
+    (in_bom yes) (on_board yes) (fields_autoplaced)
+    (property "Reference" "J18" (id 0) (at 264.16 227.965 0))
+    (property "Value" "Conn_02x02_Odd_Even" (id 1) (at 264.16 230.505 0))
+    (property "Footprint" "Connector_PinHeader_2.54mm:PinHeader_2x02_P2.54mm_Vertical_SMD" (id 2) (at 262.89 234.95 0)
+      (effects (font (size 1.27 1.27)) hide)
+    )
+    (property "Datasheet" "~" (id 3) (at 262.89 234.95 0)
+      (effects (font (size 1.27 1.27)) hide)
+    )
+    (pin "1")
+    (pin "2")
+    (pin "3")
+    (pin "4")
+  )
   (symbol (lib_id "power:GND") (at 222.25 208.28 0) (unit 1)
     (in_bom yes) (on_board yes) (fields_autoplaced)
@@
     (pin "2")
   )
-  (symbol (lib_id "Connector:Screw_Terminal_01x03") (at 265.43 181.61 0) (unit 1)
-    (in_bom yes) (on_board yes) (fields_autoplaced)
-    (property "Reference" "J7" (id 0) (at 267.97 180.3399 0)
-      (effects (font (size 1.27 1.27)) (justify left))
-    )
-    (property "Value" "Screw_Terminal_01x03" (id 1) (at 267.97 182.8799 0)
-      (effects (font (size 1.27 1.27)) (justify left))
-    )
+  (symbol (lib_id "Connector:Screw_Terminal_01x03") (at 265.43 181.61 0) (mirror x) (unit 1)
+    (in_bom yes) (on_board yes) (fields_autoplaced)
+    (property "Reference" "J7" (id 0) (at 265.43 172.72 0))
+    (property "Value" "Screw_Terminal_01x03" (id 1) (at 265.43 175.26 0))
     (property "Footprint" "TerminalBlock:TerminalBlock_Altech_AK300-3_P5.00mm" (id 2) (at 265.43 181.61 0)
       (effects (font (size 1.27 1.27)) hide)
