File: Bird_detector_V1/MCU.kicad_sch (KiCad schematic)
At the start: 48 parts, among them J18 Conn_02x02_Odd_Even, J7 Screw_Terminal_01x03, Q1 SSM6N7002, Q6 BC847BS, SW2 MCU_RESET, U2 CP2102N-Axx-xQFN24, U3 ESP32-S3-WROOM-1, U4 MCP2561-H-SN, U5 BME280, U6 74LVC1G08

Commit message: h
Parts:
- added C76, C77: 100n, Capacitor_SMD:C_0603_1608Metric_Pad1.08x0.95mm_HandSolder, symbol Device:C_Small
- added C78: 22u, Capacitor_SMD:C_0805_2012Metric_Pad1.18x1.45mm_HandSolder, symbol Device:C_Small
- added JP10: ADR0, Jumper:SolderJumper-3_P1.3mm_Bridged12_RoundedPad1.0x1.5mm_NumberLabels, symbol Jumper:SolderJumper_3_Bridged12
- added U19: MMA8452, Package_DFN_QFN:QFN-16-1EP_3x3mm_P0.5mm_EP1.45x1.45mm, symbol My_custom_lib:MMA8452
- J7: value Screw_Terminal_01x03 -> CAN
Connections:
- net +3V3: now also C76.1, C77.1, C78.1, JP10.3 (B), U19.1 (VDDIO), U19.14 (VDD)
- net GND: now also C76.2, C78.2, JP10.1 (A), U19.10 (GND), U19.12 (GND), U19.13 (NC), U19.15 (NC), U19.16 (NC), U19.3 (NC), U19.5 (GND), U19.8 (NC)
- net SCL: now also U19.4 (SCL)
- net SDA: now also U19.6 (SDA)
- new net: C77.2, U19.2 (BYP)
- new net: JP10.2 (C), U19.7 (SA0)
Other:
- note added: "Danger free pins:"
- note added: "Free safe pins:"
- note removed: "Danger pins"
- note removed: "Free pins"
- moved on the sheet: C17, C18, C20, C21, C22, C23, C24, C25, C32, D8, D9, J18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

Commit message: g
Connections:
- net COMMON_NODE: now reaches C24.1, R37.1, R38.2, R39.2
- net ADRESS_BME280: now reaches JP2.2 (C), U5.5 (SDO)
Changed lines of the file:
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@@
   (title_block
     (title "Bird Detection and Recognition System")
+    (date "2022-11-23")
     (rev "V0.1")
+    (comment 1 "Designed by: Kecs Robert Alfred")
+    (comment 2 "Verified by: Kecs Robert Alfred")
+    (comment 3 "Layout by: Kecs Robert Alfred")
   )
   (junction (at 275.59 69.85) (diameter 0) (color 0 0 0 0)
@@
     (effects (font (size 1.27 1.27)) (justify left bottom))
   )
+  (label "ADRESS_BME280" (at 213.36 248.92 0)
+    (effects (font (size 0.5 0.5)) (justify left bottom))
+  )
   (label "~{DTR}" (at 325.12 54.61 0)
     (effects (font (size 1.27 1.27)) (justify left bottom))
@@
     (effects (font (size 1.27 1.27)) (justify left bottom))
   )
+  (label "COMMON_NODE" (at 151.13 196.85 180)
+    (effects (font (size 0.5 0.5)) (justify right bottom))
+  )
   (label "GPIO_38" (at 50.8 218.44 0)

Commit message: f
Other:
- note added: "SD CARD data SPI/1bit/4bit"
- note removed: "SD CARD data SPI/2/4bit"
Changed lines of the file:
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@@
     (effects (font (size 1.27 1.27)) (justify left bottom))
   )
-  (text "SD CARD data\nSPI/2/4bit" (at 69.85 191.77 0)
+  (text "SD CARD data\nSPI/1bit/4bit" (at 69.85 191.77 0)
     (effects (font (size 1.27 1.27)) (justify left bottom))
   )

Commit message: g
Parts:
- J18: value Conn_02x02_Odd_Even -> PINS
Other:
- note added: "ACCELEROMETER"
- note added: "AIR MONITORING SENSORS"
- note added: "BOOOT & RESET"
- note added: "CAN BUS INTERFACE"
- note added: "I2C PULL UPS"
- note added: "MCU"
- note added: "USB TO UART BRIDGE PROGRAMER"
- moved on the sheet: C17, C18, C20, C21, C22, C23, C24, C25, C26, C32, C76, C77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

Commit message: g
Other:
- note added: "I2C adress 001110X"
Changed lines of the file:
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@@
+    (effects (font (size 1.27 1.27)) (justify left bottom))
+  )
+  (text "I2C adress 001110X" (at 208.28 274.32 0)
     (effects (font (size 1.27 1.27)) (justify left bottom))
   )
