File: Bird_detector_V1/_autosave-Power.kicad_sch (KiCad schematic)
At the start: 47 parts, among them J10 backup, J11 140-502-415-000, J12 USB_A, J9 ntc 10k, Q7 DMP2040USD, Q8 DMP2040USD, SW3 BMS_RESET, U10 INA3221, U8 MP2615, U9 APX810S05

Commit message: r
Parts:
- removed C38: 100n, Capacitor_SMD:C_0603_1608Metric_Pad1.08x0.95mm_HandSolder, symbol Device:C_Small
- removed C39: 22u+, Capacitor_SMD:C_0603_1608Metric_Pad1.08x0.95mm_HandSolder, symbol Device:C_Small
- removed C40: 10u+, Capacitor_SMD:C_0603_1608Metric_Pad1.08x0.95mm_HandSolder, symbol Device:C_Small
- removed C41, C42: 1u, Capacitor_SMD:C_0603_1608Metric_Pad1.08x0.95mm_HandSolder, symbol Device:C_Small
- removed D10, D11: LED_Small, LED_SMD:LED_0603_1608Metric_Pad1.05x0.95mm_HandSolder, symbol Device:LED_Small
- removed J9: ntc 10k, Connector_PinSocket_2.54mm:PinSocket_1x02_P2.54mm_Vertical, symbol Connector_Generic:Conn_01x02
- removed JP5: leds, Connector_PinHeader_2.54mm:PinHeader_1x03_P2.54mm_Vertical, symbol Jumper:Jumper_3_Bridged12
- removed L1: 6u8, Z_mycustom_footprint_lib:inductor 6x6mm, symbol Device:L
- removed R50: 50m, Resistor_SMD:R_0805_2012Metric, symbol Device:R_Small
- removed R51: 100K, Resistor_SMD:R_0603_1608Metric_Pad0.98x0.95mm_HandSolder, symbol Device:R_Small
- removed R52, R53: 1k, Resistor_SMD:R_0603_1608Metric_Pad0.98x0.95mm_HandSolder, symbol Device:R_Small
- removed R54: 100k, Resistor_SMD:R_0603_1608Metric_Pad0.98x0.95mm_HandSolder, symbol Device:R_Small
- removed R57: 10k, Resistor_SMD:R_0603_1608Metric_Pad0.98x0.95mm_HandSolder, symbol Device:R_Small
- removed SW3: BMS_RESET, SamacSys_Parts:PTS526SK15SMTR2LFS, symbol Switch:SW_SPST
- removed U8: MP2615, SamacSys_Parts:MP2615GQZ, symbol My_custom_lib:MP2615
Connections:
- no-connect marks 9 -> 8
Other:
- note removed: "0.2W max"
- note removed: "4.5-18V absolute max input Buck only"
- note removed: "CELL: 1 short to VCC for single cell OR 2 connect to GND for 2 cell SEL: 1 pull up for 4.1V (longer cell live) 2 pull down or float for 4.2V (more storage)"
- note removed: "CHGOK: Charging completion indicator. When this pin goes logic low, the device is charging. The pin becomes an open drain once the charge is completed or suspended. ACOK: Valid input supply indicator. A logic low on this pin indicates the presence of a valid input power supply."
- note removed: "T_p (seconds) = 0.46 X C (uF) t_trickle (minutes) = 62.8 X C (uF)"
- note removed: "switching frequency 760KHz Inductor: DC resistance less than 50mΩ"
- moved on the sheet: U?
