File: Bird_detector_V1/Bird_detector_V1.kicad_pcb (KiCad board)
At the start: 2 copper layers, 11 parts, among them IC1 TXB0108PWR, J1 Conn_Coaxial, J2 Conn_Coaxial, J3 Conn_Coaxial, J4 USB_A, J5 SIM_Card_Shielded, J6 USB_A, U1 ESP32-S3-MINI-1, U2 ESP32-S3-WROOM-1, U3 SIM808

Commit message: g
Parts:
- added C10: 100n, Capacitor_SMD:C_0603_1608Metric_Pad1.08x0.95mm_HandSolder, F.Cu at (96.1, 103.8)
- added C11: 1u, Capacitor_SMD:C_0603_1608Metric_Pad1.08x0.95mm_HandSolder, F.Cu at (87.4, 108.8)
- added C12: 1u, Capacitor_SMD:C_0603_1608Metric_Pad1.08x0.95mm_HandSolder, F.Cu at (91.7, 101.3)
- added C13: 1u, Capacitor_SMD:C_0603_1608Metric_Pad1.08x0.95mm_HandSolder, F.Cu at (91.7, 106.3)
- added C14: 100n, Capacitor_SMD:C_0603_1608Metric_Pad1.08x0.95mm_HandSolder, F.Cu at (91.7, 108.8)
- added C15: 1u, Capacitor_SMD:C_0603_1608Metric_Pad1.08x0.95mm_HandSolder, F.Cu at (91.7, 103.8)
- added C16: 100n, Capacitor_SMD:C_0603_1608Metric_Pad1.08x0.95mm_HandSolder, F.Cu at (91.7, 98.8)
- added C17: 1u, Capacitor_SMD:C_0603_1608Metric_Pad1.08x0.95mm_HandSolder, F.Cu at (100.4, 98.8)
- added C18: 100n, Capacitor_SMD:C_0603_1608Metric_Pad1.08x0.95mm_HandSolder, F.Cu at (100.4, 103.8)
- added C19: 1u, Capacitor_SMD:C_0603_1608Metric_Pad1.08x0.95mm_HandSolder, F.Cu at (104.8, 101.3)
- added C2: 10u, Capacitor_SMD:C_0603_1608Metric_Pad1.08x0.95mm_HandSolder, F.Cu at (118.4, 98.8)
- added C3: 100n, Capacitor_SMD:C_0603_1608Metric_Pad1.08x0.95mm_HandSolder, F.Cu at (114.0, 101.3)
- added C4: 33p, Capacitor_SMD:C_0603_1608Metric_Pad1.08x0.95mm_HandSolder, F.Cu at (118.4, 101.3)
- added C6: 10u, Capacitor_SMD:C_0603_1608Metric_Pad1.08x0.95mm_HandSolder, F.Cu at (114.0, 103.8)
- added C7: 10u, Capacitor_SMD:C_0603_1608Metric_Pad1.08x0.95mm_HandSolder, F.Cu at (114.0, 98.8)
- added C8: 10u, Capacitor_SMD:C_0603_1608Metric_Pad1.08x0.95mm_HandSolder, F.Cu at (87.4, 98.8)
- added C9: 100n, Capacitor_SMD:C_0603_1608Metric_Pad1.08x0.95mm_HandSolder, F.Cu at (87.4, 101.3)
- added CA1: 1u, Capacitor_SMD:C_0603_1608Metric_Pad1.08x0.95mm_HandSolder, F.Cu at (96.1, 108.8)
- added CA2: 1u, Capacitor_SMD:C_0603_1608Metric_Pad1.08x0.95mm_HandSolder, F.Cu at (100.4, 101.3)
- added CA3: 1u, Capacitor_SMD:C_0603_1608Metric_Pad1.08x0.95mm_HandSolder, F.Cu at (96.1, 101.3)
- added CA4: 1u, Capacitor_SMD:C_0603_1608Metric_Pad1.08x0.95mm_HandSolder, F.Cu at (96.1, 98.8)
- added CA5: 1u, Capacitor_SMD:C_0603_1608Metric_Pad1.08x0.95mm_HandSolder, F.Cu at (104.8, 98.8)
- added CA6: 1u, Capacitor_SMD:C_0603_1608Metric_Pad1.08x0.95mm_HandSolder, F.Cu at (87.4, 103.8)
- added FB1: MZ1608-102Y, Resistor_SMD:R_0603_1608Metric_Pad0.98x0.95mm_HandSolder, F.Cu at (143.3, 100.8)
- added FB2: MH2029-401Y, Resistor_SMD:R_0805_2012Metric_Pad1.20x1.40mm_HandSolder, F.Cu at (155.0, 96.4)
- added IC1: TXB0108PWR, SamacSys_Parts:SOP65P640X120-20N, F.Cu at (134.1, 113.3)
- added JP1: ADR1, Jumper:SolderJumper-3_P1.3mm_Bridged12_RoundedPad1.0x1.5mm_NumberLabels, F.Cu at (138.3, 103.0)
- added JP2: ADR0, Jumper:SolderJumper-3_P1.3mm_Bridged12_RoundedPad1.0x1.5mm_NumberLabels, F.Cu at (144.5, 96.7)
- added R1: R_Small, Resistor_SMD:R_0603_1608Metric_Pad0.98x0.95mm_HandSolder, F.Cu at (122.7, 98.8)
- added R2: 2k, Resistor_SMD:R_0603_1608Metric_Pad0.98x0.95mm_HandSolder, F.Cu at (87.4, 106.3)
- added R3: 2k, Resistor_SMD:R_0603_1608Metric_Pad0.98x0.95mm_HandSolder, F.Cu at (96.1, 106.3)
- added TP1: TestPoint, TestPoint:TestPoint_Pad_1.5x1.5mm, F.Cu at (143.8, 111.0)
- added TP2: TestPoint, TestPoint:TestPoint_Pad_1.5x1.5mm, F.Cu at (140.3, 114.5)
- added TP3: TestPoint, TestPoint:TestPoint_Pad_1.5x1.5mm, F.Cu at (140.3, 111.0)
- added TP4: TestPoint, TestPoint:TestPoint_Pad_1.5x1.5mm, F.Cu at (142.9, 103.9)
- added U4: TLV320ADC3100, Package_DFN_QFN:VQFN-24-1EP_4x4mm_P0.5mm_EP2.45x2.45mm_ThermalVias, F.Cu at (132.8, 98.1)
- added U5: MIC5317, Package_TO_SOT_SMD:SOT-23-5_HandSoldering, F.Cu at (132.5, 103.5)
- added U6: MIC5317, Package_TO_SOT_SMD:SOT-23-5_HandSoldering, F.Cu at (138.8, 97.3)
- C5: renamed from C2; value C_Small -> gap
- renumbered IC1 to IC2, J4 to J1, J5 to J2, J1 to J3, J6 to J4, J2 to J5, J3 to J6, U3 to U1, U1 to U2, U2 to U3
Connections:
- IC2 pad 1: unconnected-(IC1-Pad1) -> +3V3
- IC2 pad 10: unconnected-(IC1-Pad10) -> +3V3
- IC2 pad 11: unconnected-(IC1-Pad11) -> GND
- IC2 pad 12: unconnected-(IC1-Pad12) -> /GSM+GPS/RESET_INT
- IC2 pad 13: unconnected-(IC1-Pad13) -> /GSM+GPS/TX_INT
- IC2 pad 14: unconnected-(IC1-Pad14) -> /GSM+GPS/RX_INT
- IC2 pad 15: unconnected-(IC1-Pad15) -> /GSM+GPS/RTS_INT
- IC2 pad 16: unconnected-(IC1-Pad16) -> /GSM+GPS/CTS_INT
- IC2 pad 17: unconnected-(IC1-Pad17) -> /GSM+GPS/DCD_INT
- IC2 pad 18: unconnected-(IC1-Pad18) -> /GSM+GPS/RI_INT
- IC2 pad 19: unconnected-(IC1-Pad19) -> +3V8
- IC2 pad 2: unconnected-(IC1-Pad2) -> +3V3
- IC2 pad 20: unconnected-(IC1-Pad20) -> /GSM+GPS/DTR_INT
- IC2 pad 3: unconnected-(IC1-Pad3) -> /GSM+GPS/RI
- IC2 pad 4: unconnected-(IC1-Pad4) -> /GSM+GPS/DCD
- IC2 pad 5: unconnected-(IC1-Pad5) -> /GSM+GPS/CTS
- IC2 pad 6: unconnected-(IC1-Pad6) -> /GSM+GPS/RTS
- IC2 pad 7: unconnected-(IC1-Pad7) -> /GSM+GPS/RX
- IC2 pad 8: unconnected-(IC1-Pad8) -> /GSM+GPS/TX
- IC2 pad 9: unconnected-(IC1-Pad9) -> /GSM+GPS/RESET
- U1 pad 10: unconnected-(U3-Pad10) (its old number) -> /GSM+GPS/RI_INT
- U1 pad 11: unconnected-(U3-Pad11) (its old number) -> /GSM+GPS/DCD_INT
- U1 pad 12: unconnected-(U3-Pad12) (its old number) -> /GSM+GPS/CTS_INT
- U1 pad 13: unconnected-(U3-Pad13) (its old number) -> /GSM+GPS/RTS_INT
- U1 pad 14: unconnected-(U3-Pad14) (its old number) -> /GSM+GPS/RX_INT
- U1 pad 15: unconnected-(U3-Pad15) (its old number) -> /GSM+GPS/TX_INT
- U1 pad 16: unconnected-(U3-Pad16) (its old number) -> /GSM+GPS/RESET_INT
- U1 pad 17: unconnected-(U3-Pad17) (its old number) -> Net-(U1-Pad17)
- U1 pad 25: (no net) -> /GSM+GPS/5V-DIY
- U1 pad 38: SDA -> /GSM+GPS/SDA_INT
- U1 pad 39: SCL -> /GSM+GPS/SCL_INT
- U1 pad 49: unconnected-(U3-Pad49) -> /GSM+GPS/STAT_INT
- U1 pad 7: /GSM+GPS/5V-DIY -> Net-(U1-Pad17)
- U1 pad 8: unconnected-(U3-Pad8) (its old number) -> Net-(U1-Pad8)
- U1 pad 9: unconnected-(U3-Pad9) (its old number) -> /GSM+GPS/DTR_INT

Commit message: g
Parts:
- added C1: 1u, Capacitor_SMD:C_0603_1608Metric_Pad1.08x0.95mm_HandSolder, F.Cu at (96.0, 117.6)
- added C11: DNP, Capacitor_SMD:C_0603_1608Metric_Pad1.08x0.95mm_HandSolder, F.Cu at (91.7, 117.6)
- added C12: DNP, Capacitor_SMD:C_0603_1608Metric_Pad1.08x0.95mm_HandSolder, F.Cu at (96.0, 125.1)
- added C13: DNP, Capacitor_SMD:C_0603_1608Metric_Pad1.08x0.95mm_HandSolder, F.Cu at (100.4, 117.6)
- added C14: DNP, Capacitor_SMD:C_0603_1608Metric_Pad1.08x0.95mm_HandSolder, F.Cu at (100.4, 120.1)
- added C2: DNP, Capacitor_SMD:C_0603_1608Metric_Pad1.08x0.95mm_HandSolder, F.Cu at (91.7, 120.1)
- added C3: DNP, Capacitor_SMD:C_0603_1608Metric_Pad1.08x0.95mm_HandSolder, F.Cu at (96.0, 120.1)
- added D1: D5V0P4UR6SO-7, SamacSys_Parts:SOT95P285X140-6N, F.Cu at (86.8, 123.3)
- added D2: D5V0P4UR6SO-7, SamacSys_Parts:SOT95P285X140-6N, F.Cu at (86.8, 118.7)
- added R2: 0, Resistor_SMD:R_0603_1608Metric_Pad0.98x0.95mm_HandSolder, F.Cu at (96.0, 122.6)
- added R3: 0, Resistor_SMD:R_0603_1608Metric_Pad0.98x0.95mm_HandSolder, F.Cu at (91.7, 122.6)
- added R4: 0, Resistor_SMD:R_0603_1608Metric_Pad0.98x0.95mm_HandSolder, F.Cu at (91.7, 125.1)
- renumbered C7 to C10, C8 to C15, C9 to C16, C10 to C17, C11 to C18, C12 to C19, C13 to C20, C14 to C21, C15 to C22, C16 to C23, C17 to C24, C18 to C25, C19 to C26, C2 to C5, C3 to C6, C4 to C7, C5 to C8, C6 to C9, R2 to R5, R3 to R6
Connections:
- net Net-(C5-Pad1) renamed /GSM+GPS/5V-in2
- J3 pad 1: Net-(J3-Pad1) -> Net-(C3-Pad1)
- J5 pad 1: Net-(J5-Pad1) -> Net-(C12-Pad1)
- J6 pad 1: Net-(J6-Pad1) -> Net-(C14-Pad1)
- U1 pad 35: Net-(J6-Pad1) -> Net-(C13-Pad1)
- U1 pad 53: Net-(J5-Pad1) -> Net-(C11-Pad1)
- U1 pad 66: Net-(J3-Pad1) -> Net-(C2-Pad1)

Commit message: j
Parts:
- removed C15: 10u, Capacitor_SMD:C_0603_1608Metric_Pad1.08x0.95mm_HandSolder
- removed C16: 100n, Capacitor_SMD:C_0603_1608Metric_Pad1.08x0.95mm_HandSolder
- removed D1: D5V0P4UR6SO-7, SamacSys_Parts:SOT95P285X140-6N
- removed the IC1 at (134.1, 113.3)
- removed the J1 at (172.4, 76.4)
- removed TP4: TestPoint, TestPoint:TestPoint_Pad_1.5x1.5mm
- added C27: 10u, Capacitor_SMD:C_0603_1608Metric_Pad1.08x0.95mm_HandSolder, F.Cu at (106.7, 162.8)
- added C28: 22u, Capacitor_SMD:C_0603_1608Metric_Pad1.08x0.95mm_HandSolder, F.Cu at (106.7, 138.2)
- added C29: 22u, Capacitor_SMD:C_0603_1608Metric_Pad1.08x0.95mm_HandSolder, F.Cu at (115.4, 138.2)
- added C30: 22u, Capacitor_SMD:C_0603_1608Metric_Pad1.08x0.95mm_HandSolder, F.Cu at (111.0, 138.2)
- added C31: 22u, Capacitor_SMD:C_0603_1608Metric_Pad1.08x0.95mm_HandSolder, F.Cu at (122.6, 134.1)
- added D5: D5V0P4UR6SO-7, SamacSys_Parts:SOT95P285X140-6N, F.Cu at (152.6, 124.1)
- added D6: z, Diode_SMD:D_SOD-123, F.Cu at (142.3, 131.7)
- added D8: D5V0P4UR6SO-7, SamacSys_Parts:SOT95P285X140-6N, F.Cu at (124.2, 130.5)
- added J6: MEM2051, Z_mycustom_footprint_lib:MEM2051-00-195-00, F.Cu at (113.6, 152.2)
- added J8: USB_A, Connector_USB:USB_A_Molex_105057_Vertical, F.Cu at (109.5, 128.5)
- added Q5: DMP2040USD, Package_SO:SO-8_3.9x4.9mm_P1.27mm, F.Cu at (108.7, 133.7)
- added Q6: DMP2040USD, Package_SO:SO-8_3.9x4.9mm_P1.27mm, F.Cu at (125.8, 125.0)
- added R1: 100, Resistor_SMD:R_0603_1608Metric_Pad0.98x0.95mm_HandSolder, F.Cu at (160.4, 130.2)
- added R10: 100, Resistor_SMD:R_0603_1608Metric_Pad0.98x0.95mm_HandSolder, F.Cu at (150.3, 133.8)
- added R11: 100k, Resistor_SMD:R_0603_1608Metric_Pad0.98x0.95mm_HandSolder, F.Cu at (151.7, 131.3)
- added R12: 100k, Resistor_SMD:R_0603_1608Metric_Pad0.98x0.95mm_HandSolder, F.Cu at (152.2, 127.7)
- added R13: 100, Resistor_SMD:R_0603_1608Metric_Pad0.98x0.95mm_HandSolder, F.Cu at (159.0, 132.7)
- added R14: X, Resistor_SMD:R_0603_1608Metric_Pad0.98x0.95mm_HandSolder, F.Cu at (141.6, 134.7)
- added R15: 100, Resistor_SMD:R_0603_1608Metric_Pad0.98x0.95mm_HandSolder, F.Cu at (159.0, 135.2)
- added R16: 100k, Resistor_SMD:R_0603_1608Metric_Pad0.98x0.95mm_HandSolder, F.Cu at (156.5, 127.7)
- added R17: X, Resistor_SMD:R_0603_1608Metric_Pad0.98x0.95mm_HandSolder, F.Cu at (147.3, 131.3)
- added R18: 100, Resistor_SMD:R_0603_1608Metric_Pad0.98x0.95mm_HandSolder, F.Cu at (160.9, 125.5)
- added R19: 100k, Resistor_SMD:R_0603_1608Metric_Pad0.98x0.95mm_HandSolder, F.Cu at (145.9, 134.7)
- added R2: 100, Resistor_SMD:R_0603_1608Metric_Pad0.98x0.95mm_HandSolder, F.Cu at (145.9, 137.2)
- added R25: 100k, Resistor_SMD:R_0603_1608Metric_Pad0.98x0.95mm_HandSolder, F.Cu at (124.3, 143.9)
- added R4: 10k, Resistor_SMD:R_0603_1608Metric_Pad0.98x0.95mm_HandSolder, F.Cu at (154.6, 133.8)
- added R5: 10k, Resistor_SMD:R_0603_1608Metric_Pad0.98x0.95mm_HandSolder, F.Cu at (156.0, 130.2)
- added R6: 100k, Resistor_SMD:R_0603_1608Metric_Pad0.98x0.95mm_HandSolder, F.Cu at (154.6, 136.3)
- added R7: X, Resistor_SMD:R_0603_1608Metric_Pad0.98x0.95mm_HandSolder, F.Cu at (157.5, 123.0)
- added R8: X, Resistor_SMD:R_0603_1608Metric_Pad0.98x0.95mm_HandSolder, F.Cu at (150.3, 136.3)
- added R9: 100, Resistor_SMD:R_0603_1608Metric_Pad0.98x0.95mm_HandSolder, F.Cu at (141.6, 137.2)
- added SW1: SW_SPST, SamacSys_Parts:PTS526SK15SMTR2LFS, F.Cu at (144.9, 125.9)
- added U7: APX810S05, Package_TO_SOT_SMD:SOT-23, F.Cu at (132.5, 124.0)
- added U8: TPS63020DSJR, Z_mycustom_footprint_lib:TPS63020, F.Cu at (116.5, 133.5)
- R3: renamed from R1; value R_Small -> 100
- renumbered D2 to D7, IC2 to IC1, J2 to J1, J3 to J2, J4 to J3, J5 to J4, J6 to J5, R2 to R20, R3 to R21, R4 to R22, R5 to R23, R6 to R24
Connections:
- net Net-(Q1-Pad3) renamed /GSM+GPS/PRWKEY
- FB2 pad 1: unconnected-(FB2-Pad1) -> VBUS
- FB2 pad 2: unconnected-(FB2-Pad2) -> Net-(F3-Pad1)
- U1 pad 37: unconnected-(U1-Pad37) -> /GSM+GPS/IPPS
- U1 pad 50: unconnected-(U1-Pad50) -> /GSM+GPS/NETLIGHT
- U1 pad 63: unconnected-(U1-Pad63) -> /GSM+GPS/RF_SYNC

Commit message: f
Parts:
- removed Q5: DMP2040USD, Package_SO:SO-8_3.9x4.9mm_P1.27mm
- removed TP3: TestPoint, TestPoint:TestPoint_Pad_1.5x1.5mm
- added C15: 100n, Capacitor_SMD:C_0603_1608Metric_Pad1.08x0.95mm_HandSolder, F.Cu at (-101.1, 124.9)
- added C16: 1u, Capacitor_SMD:C_0603_1608Metric_Pad1.08x0.95mm_HandSolder, F.Cu at (-101.1, 122.4)
- added C32: 100n, Capacitor_SMD:C_0603_1608Metric_Pad1.08x0.95mm_HandSolder, F.Cu at (-134.0, 124.9)
- added C33: 100n, Capacitor_SMD:C_0603_1608Metric_Pad1.08x0.95mm_HandSolder, F.Cu at (-138.3, 127.4)
- added C34: 100n, Capacitor_SMD:C_0603_1608Metric_Pad1.08x0.95mm_HandSolder, F.Cu at (-131.9, 115.3)
- added C35: 22u, Capacitor_SMD:C_0603_1608Metric_Pad1.08x0.95mm_HandSolder, F.Cu at (-27.4, 66.5)
- added C36: 22u, Capacitor_SMD:C_0603_1608Metric_Pad1.08x0.95mm_HandSolder, F.Cu at (-31.8, 69.0)
- added C37: 22u, Capacitor_SMD:C_0603_1608Metric_Pad1.08x0.95mm_HandSolder, F.Cu at (-39.2, 74.5)
- added C38: 22u, Capacitor_SMD:C_0603_1608Metric_Pad1.08x0.95mm_HandSolder, F.Cu at (-27.4, 71.5)
- added C39: 100n, Capacitor_SMD:C_0603_1608Metric_Pad1.08x0.95mm_HandSolder, F.Cu at (-31.8, 71.5)
- added C40: 22u, Capacitor_SMD:C_0603_1608Metric_Pad1.08x0.95mm_HandSolder, F.Cu at (-39.2, 82.0)
- added C41: 22u, Capacitor_SMD:C_0603_1608Metric_Pad1.08x0.95mm_HandSolder, F.Cu at (-23.1, 61.5)
- added C42: 22u, Capacitor_SMD:C_0603_1608Metric_Pad1.08x0.95mm_HandSolder, F.Cu at (-23.1, 64.0)
- added C43: 22u, Capacitor_SMD:C_0603_1608Metric_Pad1.08x0.95mm_HandSolder, F.Cu at (-23.1, 66.5)
- added C44: 100n, Capacitor_SMD:C_0603_1608Metric_Pad1.08x0.95mm_HandSolder, F.Cu at (-30.6, 74.0)
- added D1: LED_Small, LED_SMD:LED_0603_1608Metric_Pad1.05x0.95mm_HandSolder, F.Cu at (-132.8, 87.6)
- added D10: D5V0P4UR6SO-7, SamacSys_Parts:SOT95P285X140-6N, F.Cu at (-136.7, 118.4)
- added D2: LED_Small, LED_SMD:LED_0603_1608Metric_Pad1.05x0.95mm_HandSolder, F.Cu at (-128.4, 87.6)
- added D3: LED_Small, LED_SMD:LED_0603_1608Metric_Pad1.05x0.95mm_HandSolder, F.Cu at (-128.4, 90.2)
- added D4: LED_Small, LED_SMD:LED_0603_1608Metric_Pad1.05x0.95mm_HandSolder, F.Cu at (-132.8, 90.2)
- added D9: LED_Small, LED_SMD:LED_0603_1608Metric_Pad1.05x0.95mm_HandSolder, F.Cu at (-149.5, 133.2)
- added J10: 140-502-415-000, SamacSys_Parts:140502415000, F.Cu at (-161.4, 119.5)
- added J11: USB_A, Connector_USB:USB_A_Molex_105057_Vertical, F.Cu at (-159.9, 114.5)
- added J7: 292132-3, SamacSys_Parts:SHDR3W65P0X200_1X3_780X580X710P, F.Cu at (-107.0, 117.9)
- added JP3: leds, Connector_PinHeader_2.54mm:PinHeader_1x03_P2.54mm_Vertical, F.Cu at (-153.5, 118.8)
- added JP4: ADR1, Jumper:SolderJumper-3_P1.3mm_Bridged12_RoundedPad1.0x1.5mm_NumberLabels, F.Cu at (-148.4, 124.3)
- added JP5: safe, Jumper:SolderJumper-2_P1.3mm_Open_RoundedPad1.0x1.5mm, F.Cu at (-34.9, 77.5)
- added Q7: DMP2040USD, Package_SO:SO-8_3.9x4.9mm_P1.27mm, F.Cu at (-143.6, 119.3)
- added R26: 1k, Resistor_SMD:R_0603_1608Metric_Pad0.98x0.95mm_HandSolder, F.Cu at (-95.4, 112.5)
- added R27: 2k, Resistor_SMD:R_0603_1608Metric_Pad0.98x0.95mm_HandSolder, F.Cu at (-105.7, 128.3)
- added R28: 2k, Resistor_SMD:R_0603_1608Metric_Pad0.98x0.95mm_HandSolder, F.Cu at (-91.5, 117.6)
- added R29: 100k, Resistor_SMD:R_0603_1608Metric_Pad0.98x0.95mm_HandSolder, F.Cu at (-60.5, 96.5)
- added R30: 50m, Resistor_SMD:R_0805_2012Metric, F.Cu at (-124.3, 109.2)
- added R31: 50m, Resistor_SMD:R_0805_2012Metric, F.Cu at (-128.8, 109.2)
- added R32: 100K, Resistor_SMD:R_0603_1608Metric_Pad0.98x0.95mm_HandSolder, F.Cu at (-138.3, 124.9)
- added R33: 1k, Resistor_SMD:R_0603_1608Metric_Pad0.98x0.95mm_HandSolder, F.Cu at (-134.0, 127.4)
- added R34: 1k, Resistor_SMD:R_0603_1608Metric_Pad0.98x0.95mm_HandSolder, F.Cu at (-127.6, 114.5)
- added R35: 100k, Resistor_SMD:R_0603_1608Metric_Pad0.98x0.95mm_HandSolder, F.Cu at (-142.7, 131.7)
- added R36: 100k, Resistor_SMD:R_0603_1608Metric_Pad0.98x0.95mm_HandSolder, F.Cu at (-132.8, 121.9)
- added R37: 100k, Resistor_SMD:R_0603_1608Metric_Pad0.98x0.95mm_HandSolder, F.Cu at (-142.7, 126.7)
- added R38: 10k, Resistor_SMD:R_0603_1608Metric_Pad0.98x0.95mm_HandSolder, F.Cu at (-131.9, 117.8)
- added R39: 50m, Resistor_SMD:R_0805_2012Metric, F.Cu at (-137.2, 122.2)
- added R40: 1k, Resistor_SMD:R_0603_1608Metric_Pad0.98x0.95mm_HandSolder, F.Cu at (-127.6, 117.0)
- added R41: 100k, Resistor_SMD:R_0603_1608Metric_Pad0.98x0.95mm_HandSolder, F.Cu at (-124.4, 111.9)
- added R42: 50m, Resistor_SMD:R_0805_2012Metric, F.Cu at (-143.3, 124.0)
- added R43: 1Meg, Resistor_SMD:R_0603_1608Metric_Pad0.98x0.95mm_HandSolder, F.Cu at (-34.9, 74.5)
- added R44: DNP, Resistor_SMD:R_0603_1608Metric_Pad0.98x0.95mm_HandSolder, F.Cu at (-27.4, 69.0)
- added R45: 1Meg, Resistor_SMD:R_0603_1608Metric_Pad0.98x0.95mm_HandSolder, F.Cu at (-31.8, 66.5)
- added R46: 180k, Resistor_SMD:R_0603_1608Metric_Pad0.98x0.95mm_HandSolder, F.Cu at (-27.4, 61.5)
- added R47: 1.18Meg, Resistor_SMD:R_0603_1608Metric_Pad0.98x0.95mm_HandSolder, F.Cu at (-39.2, 77.0)
- added R48: 180k, Resistor_SMD:R_0603_1608Metric_Pad0.98x0.95mm_HandSolder, F.Cu at (-39.2, 79.5)
- added R49: 1.32Meg, Resistor_SMD:R_0603_1608Metric_Pad0.98x0.95mm_HandSolder, F.Cu at (-27.4, 64.0)
- added R50: DNP, Resistor_SMD:R_0603_1608Metric_Pad0.98x0.95mm_HandSolder, F.Cu at (-31.8, 64.0)
- added R51: 1Meg, Resistor_SMD:R_0603_1608Metric_Pad0.98x0.95mm_HandSolder, F.Cu at (-18.7, 61.5)
- added R52: 200k, Resistor_SMD:R_0603_1608Metric_Pad0.98x0.95mm_HandSolder, F.Cu at (-31.8, 61.5)
- added SW2: BMS_RESET, SamacSys_Parts:PTS526SK15SMTR2LFS, F.Cu at (-142.3, 111.9)
- added U10: TPS63020DSJR, Z_mycustom_footprint_lib:TPS63020, F.Cu at (-37.9, 63.3)
- added U9: TPS63020DSJR, Z_mycustom_footprint_lib:TPS63020, F.Cu at (-37.9, 69.8)
- added Y1: SiT1602BI-13-33E-12.000000G, Crystal:Crystal_SMD_2520-4Pin_2.5x2.0mm, F.Cu at (-105.5, 124.5)
- C17: value 100n -> 1u
- C19, C26: value 1u -> 100n
- C25: value 100n -> 10u
- C27: value 10u -> 100n
- C28: value 22u -> 22u+
- C29: value 22u -> 10u+
- C30, C31: value 22u -> 1u
- C8: value gap -> DNP
- C9: value 10u -> DNP
- D8: value D5V0P4UR6SO-7 -> LED_Small; footprint SamacSys_Parts:SOT95P285X140-6N -> LED_SMD:LED_0603_1608Metric_Pad1.05x0.95mm_HandSolder
- J6: value MEM2051 -> 292132-3; footprint Z_mycustom_footprint_lib:MEM2051-00-195-00 -> SamacSys_Parts:SHDR3W65P0X200_1X3_780X580X710P
- J8: value USB_A -> MEM2051; footprint Connector_USB:USB_A_Molex_105057_Vertical -> Z_mycustom_footprint_lib:MEM2051-00-195-00
- R11, R12, R19: value 100k -> 100
- R13, R9: value 100 -> 100k
- R14: value X -> 100k
- R18: value 100 -> X
- R20: value 0 -> 100
- R21, R22: value 0 -> 100k
- R23, R24: value 2k -> 0
- R25: value 100k -> 0
- R3: value 100 -> 10k
- R5: value 10k -> X
- R6: value 100k -> X
- R7: value X -> 100
- R8: value X -> 1k
- U2: value ESP32-S3-MINI-1 -> ESP32-S3-WROOM-1; footprint Espressif:ESP32-S3-MINI-1 -> Espressif:ESP32-S3-WROOM-1
- U3: value ESP32-S3-WROOM-1 -> TLV320ADC3100; footprint Espressif:ESP32-S3-WROOM-1 -> Package_DFN_QFN:VQFN-24-1EP_4x4mm_P0.5mm_EP2.45x2.45mm_ThermalVias
- U4: value TLV320ADC3100 -> MIC5317; footprint Package_DFN_QFN:VQFN-24-1EP_4x4mm_P0.5mm_EP2.45x2.45mm_ThermalVias -> Package_TO_SOT_SMD:SOT-23-5_HandSoldering
- U6: value MIC5317 -> MP2615; footprint Package_TO_SOT_SMD:SOT-23-5_HandSoldering -> SamacSys_Parts:MP2615GQZ
- U8: value TPS63020DSJR -> INA3221; footprint Z_mycustom_footprint_lib:TPS63020 -> Package_DFN_QFN:Texas_RGV_S-PVQFN-N16_EP2.1x2.1mm
- moved J1 324.4 mm to (-155.2, 95.6)
- moved J4 324.4 mm to (-139.9, 99.3)
- moved J2 315.3 mm to (-122.8, 72.7)
- moved FB2 311.4 mm to (-154.1, 133.3)
- moved R18 295.3 mm to (-132.8, 95.2)
- moved J5 295.1 mm to (-132.5, 72.7)
- moved U1 295.1 mm to (-150.6, 73.5)
- moved U6 293.3 mm to (-152.8, 129.0)
- moved R6 289.4 mm to (-132.8, 102.8)
- moved R13 289.3 mm to (-128.5, 100.3)
- moved Q6 286.6 mm to (-160.7, 130.5)
- moved R16 286.6 mm to (-128.5, 97.7)
- moved R5 282.9 mm to (-124.1, 90.1)
- moved R2 281.2 mm to (-132.8, 100.3)
- moved U7 279.8 mm to (-147.3, 128.3)
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Connections:
- C17 pad 1: /Audio capture/RESET_AUDIO -> Net-(C17-Pad1)
- C18 pad 1: +3V8 -> +3.3VA
- C19 pad 1: Net-(C19-Pad1) -> 1V8A
- C20 pad 1: +3.3VA -> 1V8A
- C21 pad 1: 1V8A -> +3.3VA
- C22 pad 1: 1V8A -> +3.3VA
- C25 pad 1: +3.3VA -> +3V3
- C26 pad 1: +3.3VA -> IN_SYSTEM-
- C26 pad 2: GND -> IN_SYSTEM+
- C27 pad 1: +3V3 -> Net-(C27-Pad1)
- C27 pad 2: GND -> Net-(C27-Pad2)
- C28 pad 1: unconnected-(C28-Pad1) -> IN_SYSTEM-
- C28 pad 2: unconnected-(C28-Pad2) -> GND
- C29 pad 1: unconnected-(C29-Pad1) -> IN_SOLAR-
- C29 pad 2: unconnected-(C29-Pad2) -> GND
- C30 pad 1: unconnected-(C30-Pad1) -> /Power Management +BMS/VCC
- C30 pad 2: unconnected-(C30-Pad2) -> GND
- C31 pad 1: unconnected-(C31-Pad1) -> Net-(C31-Pad1)
- C31 pad 2: unconnected-(C31-Pad2) -> GND
- D8 pad 1: unconnected-(D8-Pad1) -> Net-(D8-Pad1)
- D8 pad 2: GND -> Net-(D8-Pad2)
- FB1 pad 2: Net-(C19-Pad1) -> Net-(C17-Pad1)
- J6 pad 1: /MCU+WIFI+BT/DATA2 -> unconnected-(J6-Pad1)
- J6 pad 2: /MCU+WIFI+BT/DATA3/CS -> unconnected-(J6-Pad2)
- J6 pad 3: /MCU+WIFI+BT/CMD -> unconnected-(J6-Pad3)
- J8 pad 1: VBUS -> /MCU+WIFI+BT/DATA2
- J8 pad 2: D- -> /MCU+WIFI+BT/DATA3/CS
- J8 pad 3: D+ -> /MCU+WIFI+BT/CMD
- J8 pad 4: GND -> +3V3
- J8 pad 5: unconnected-(J8-Pad5) -> /MCU+WIFI+BT/SCLK
- Q6 pad 3: Net-(F2-Pad2) -> Net-(F1-Pad2)
- R10 pad 2: /GSM+GPS/RF_SYNC -> +3V3
- R11 pad 1: GND -> /GSM+GPS/ENABLE
- R11 pad 2: /GSM+GPS/NETLIGHT -> Net-(Q3-Pad2)
- R12 pad 1: GND -> Net-(R12-Pad1)
- R13 pad 1: Net-(Q1-Pad5) (its old number) -> GND
- R13 pad 2: +3V3 -> /GSM+GPS/ENABLE
- R14 pad 1: Net-(Q4-Pad6) -> GND
- R14 pad 2: Net-(D3-Pad1) (its old number) -> /GSM+GPS/RF_SYNC
- R15 pad 2: /GSM+GPS/IPPS -> /GSM+GPS/RF_SYNC
- R16 pad 2: /GSM+GPS/IPPS -> /GSM+GPS/RF_SYNC
- R18 pad 2: /GSM+GPS/STAT_INT -> Net-(D4-Pad1)
- R19 pad 1: GND -> Net-(Q5-Pad5)
- R20 pad 1: Net-(C2-Pad1) -> Net-(Q5-Pad2)
- R20 pad 2: Net-(C3-Pad1) -> /GSM+GPS/IPPS
- R21 pad 1: Net-(C11-Pad1) -> GND
- R21 pad 2: Net-(C12-Pad1) -> /GSM+GPS/STAT_INT
- R22 pad 1: Net-(C13-Pad1) -> GND
- R22 pad 2: Net-(C14-Pad1) -> /GSM+GPS/IPPS
- R23 pad 1: Net-(CA3-Pad2) -> Net-(C2-Pad1)
- R23 pad 2: Net-(R23-Pad2) -> Net-(C3-Pad1)
- R24 pad 1: Net-(R23-Pad2) -> Net-(C11-Pad1)
- R24 pad 2: Net-(CA4-Pad2) -> Net-(C12-Pad1)
- R25 pad 1: /MCU+WIFI+BT/CARD_DET -> Net-(C13-Pad1)
- R25 pad 2: +3V3 -> Net-(C14-Pad1)
- R3 pad 1: /GSM+GPS/ENABLE -> +3V8
- R3 pad 2: Net-(Q1-Pad2) -> /GSM+GPS/SDA_INT
- R4 pad 1: +3V8 -> /GSM+GPS/SCL_INT
- R4 pad 2: /GSM+GPS/SDA_INT -> +3V8
- R5 pad 1: /GSM+GPS/SCL_INT -> Net-(Q1-Pad3)
- R5 pad 2: +3V8 -> Net-(D1-Pad1)
- R6 pad 1: GND -> Net-(R6-Pad1)
- R6 pad 2: /GSM+GPS/ENABLE -> Net-(D2-Pad1)
- R7 pad 2: Net-(D1-Pad1) -> /GSM+GPS/NETLIGHT
- R8 pad 1: Net-(Q3-Pad6) -> /GSM+GPS/RF_SYNC
- R8 pad 2: Net-(D2-Pad1) -> +3V8
- R9 pad 1: Net-(Q3-Pad5) (its old number) -> GND
- TP1 pad 1: unconnected-(TP1-Pad1) -> /GSM+GPS/RESET_INT
- TP2 pad 1: /GSM+GPS/RESET_INT -> /GSM+GPS/5V-DIY
- U2 pad 1: unconnected-(U2-Pad1) -> GND
- U2 pad 13: unconnected-(U2-Pad13) -> D-
- U2 pad 14: unconnected-(U2-Pad14) -> D+
- U2 pad 2: unconnected-(U2-Pad2) -> +3V3
- U2 pad 40: unconnected-(U2-Pad40) -> GND
- U2 pad 41: unconnected-(U2-Pad41) -> GND
- U3 pad 1: unconnected-(U3-Pad1) -> /Audio capture/SCK
- U3 pad 10: unconnected-(U3-Pad10) -> +3.3VA
- U3 pad 12: unconnected-(U3-Pad12) -> Net-(CA4-Pad2)
- U3 pad 13: unconnected-(U3-Pad13) -> GND
- U3 pad 15: unconnected-(U3-Pad15) -> Net-(JP2-Pad2)
- U3 pad 16: unconnected-(U3-Pad16) -> Net-(JP1-Pad2)
- U3 pad 17: unconnected-(U3-Pad17) -> /Audio capture/SCL
- U3 pad 18: unconnected-(U3-Pad18) -> /Audio capture/SDA
- U3 pad 2: unconnected-(U3-Pad2) -> /Audio capture/WS
- U3 pad 21: unconnected-(U3-Pad21) -> +3.3VA
- U3 pad 22: unconnected-(U3-Pad22) -> 1V8A
- U3 pad 23: unconnected-(U3-Pad23) -> GND
- U3 pad 24: unconnected-(U3-Pad24) -> /Audio capture/12MHz
- U3 pad 25: unconnected-(U3-Pad25) -> (no net)
- U3 pad 3: unconnected-(U3-Pad3) -> /Audio capture/SD
- U3 pad 4: unconnected-(U3-Pad4) -> /Audio capture/RESET_AUDIO
- U3 pad 5: unconnected-(U3-Pad5) -> Net-(R27-Pad2)
- U3 pad 6: unconnected-(U3-Pad6) -> GND
- U3 pad 7: unconnected-(U3-Pad7) -> Net-(CA3-Pad2)
- U3 pad 9: unconnected-(U3-Pad9) -> GND
- U4 pad 1: /Audio capture/SCK -> Net-(C17-Pad1)
- U4 pad 2: /Audio capture/WS -> GND
- U4 pad 3: /Audio capture/SD -> Net-(C17-Pad1)
- U4 pad 4: /Audio capture/RESET_AUDIO -> unconnected-(U4-Pad4)
- U4 pad 5: Net-(R23-Pad2) -> +3.3VA
- U5 pad 1: Net-(C19-Pad1) -> +3.3VA
- U5 pad 3: Net-(C19-Pad1) -> +3.3VA
- U5 pad 5: +3.3VA -> 1V8A
- U6 pad 1: +3.3VA -> Net-(C27-Pad1)
- U6 pad 2: GND -> IN_SYSTEM-
- U6 pad 3: +3.3VA -> /Power Management +BMS/VCC
- U6 pad 4: unconnected-(U6-Pad4) -> /Power Management +BMS/VCC
- U6 pad 5: 1V8A -> Net-(U6-Pad5)
- U7 pad 1: Net-(Q5-Pad4) -> Net-(Q6-Pad4)
- U8 pad 1: +VDC -> IN_SYSTEM-
- U8 pad 10: +VDC -> unconnected-(U8-Pad10)
- U8 pad 11: +VDC -> IN_USB_-
- U8 pad 12: +VDC -> IN_USB_+
- U8 pad 13: /GSM+GPS/RF_SYNC -> unconnected-(U8-Pad13)
- U8 pad 14: Net-(R33-Pad2) -> IN_SOLAR-
- U8 pad 2: GND -> IN_SYSTEM+
- U8 pad 3: unconnected-(U8-Pad3) -> GND
- U8 pad 4: +3V8 -> +3V3
- U8 pad 5: +3V8 -> Net-(JP4-Pad2)
- U8 pad 6: Net-(L1-Pad2) -> /Audio capture/SCL
- U8 pad 7: Net-(L1-Pad2) -> /Audio capture/SDA
- U8 pad 8: Net-(L1-Pad1) -> unconnected-(U8-Pad8)
- U8 pad 9: Net-(L1-Pad1) -> unconnected-(U8-Pad9)

Commit message: R
Parts:
- added D11: LED_Small, LED_SMD:LED_0603_1608Metric_Pad1.05x0.95mm_HandSolder, F.Cu at (-109.5, 155.3)
- added D12: MMSZ5245B, Diode_SMD:D_SOD-123, F.Cu at (-123.4, 162.3)
- added D13: MMSZ5245B, Diode_SMD:D_SOD-123, F.Cu at (-108.8, 152.4)
- added F1: PPTC 2A 16V, Fuse:Fuse_1812_4532Metric_Pad1.30x3.40mm_HandSolder, F.Cu at (-115.3, 153.2)
- added F2: PPTC 2A 16V, Fuse:Fuse_1812_4532Metric_Pad1.30x3.40mm_HandSolder, F.Cu at (-122.6, 158.1)
- added F3: PPTC 2A 16V, Fuse:Fuse_1812_4532Metric_Pad1.30x3.40mm_HandSolder, F.Cu at (-122.6, 153.2)
- added FID1: Fiducial, Fiducial:Fiducial_0.5mm_Mask1.5mm, F.Cu at (-150.8, 159.2)
- added FID2: scale, Calibration_Scale:Gauge_10mm_Type2_SilkScreenTop, F.Cu at (-141.5, 161.3)
- added FID3: kicad, Symbol:KiCad-Logo2_5mm_SilkScreen, F.Cu at (-150.8, 154.2)
- added FID4: garbage, Symbol:WEEE-Logo_4.2x6mm_SilkScreen, F.Cu at (-155.0, 161.2)
- added J9: ntc 10k, Connector_PinSocket_2.54mm:PinSocket_1x02_P2.54mm_Vertical, F.Cu at (-116.7, 158.0)
- added L2: 1.5u, Inductor_SMD:L_Wuerth_MAPI-3012, F.Cu at (-123.7, 170.8)
- added L3: 1.5u, Inductor_SMD:L_Wuerth_MAPI-3012, F.Cu at (-123.7, 175.8)
- added Q1: SSM6N7002, Package_TO_SOT_SMD:SOT-363_SC-70-6_Handsoldering, F.Cu at (-154.7, 179.2)
- added Q2: SSM6N7002, Package_TO_SOT_SMD:SOT-363_SC-70-6_Handsoldering, F.Cu at (-154.7, 175.4)
- added Q3: SSM6N7002, Package_TO_SOT_SMD:SOT-363_SC-70-6_Handsoldering, F.Cu at (-148.8, 171.5)
- added Q4: SSM6N7002, Package_TO_SOT_SMD:SOT-363_SC-70-6_Handsoldering, F.Cu at (-154.7, 171.5)
- added Q5: SSM6N7002, Package_TO_SOT_SMD:SOT-363_SC-70-6_Handsoldering, F.Cu at (-148.8, 175.4)
- added R53: 1k, Resistor_SMD:R_0603_1608Metric_Pad0.98x0.95mm_HandSolder, F.Cu at (-112.2, 157.9)
Connections:
- C29 pad 1: IN_SOLAR- -> +BATT
- R31 pad 2: IN_SOLAR- -> +BATT
- U6 pad 9: IN_SOLAR- -> +BATT
