File: Bird_detector_V1/Bird_detector_V1.kicad_pcb (KiCad board)
At the start: 2 copper layers, 165 parts, among them IC1 TXB0108PWR, J1 SIM_Card_Shielded, J10 140-502-415-000, J11 USB_A, J2 Conn_Coaxial, J3 USB_A, J4 Conn_Coaxial, J5 Conn_Coaxial, J6 292132-3, J7 292132-3, J8 MEM2051, J9 ntc 10k, Q1 SSM6N7002, Q2 SSM6N7002, Q3 SSM6N7002, Q4 SSM6N7002, Q5 SSM6N7002, Q6 DMP2040USD, Q7 DMP2040USD, SW1 SW_SPST, SW2 BMS_RESET, U1 SIM808, U10 TPS63020DSJR, U2 ESP32-S3-WROOM-1, U3 TLV320ADC3100, U4 MIC5317, U5 MIC5317, U6 MP2615, U7 APX810S05, U8 INA3221, U9 TPS63020DSJR, Y1 SiT1602BI-13-33E-12.000000G

Commit message: v
Parts:
- removed the C10 at (-91.9, 61.5)
- removed FID3: kicad, Symbol:KiCad-Logo2_5mm_SilkScreen
- removed the TP1 at (-87.9, 62.0)
- removed the U3 at (-100.7, 110.9)
- added C4: 10u, Capacitor_SMD:C_0603_1608Metric_Pad1.08x0.95mm_HandSolder, B.Cu at (177.8, 91.6)
- added C45: 100n, Capacitor_SMD:C_0603_1608Metric_Pad1.08x0.95mm_HandSolder, F.Cu at (351.5, 89.1)
- added C46: 22u, Capacitor_SMD:C_0603_1608Metric_Pad1.08x0.95mm_HandSolder, F.Cu at (452.8, 141.1)
- added C47: 22u, Capacitor_SMD:C_0603_1608Metric_Pad1.08x0.95mm_HandSolder, F.Cu at (456.6, 151.5)
- added C48: 22u, Capacitor_SMD:C_0603_1608Metric_Pad1.08x0.95mm_HandSolder, F.Cu at (456.6, 153.3)
- added C49: 22u, Capacitor_SMD:C_0603_1608Metric_Pad1.08x0.95mm_HandSolder, F.Cu at (456.5, 155.2)
- added C50: 100n, Capacitor_SMD:C_0603_1608Metric_Pad1.08x0.95mm_HandSolder, F.Cu at (449.2, 140.9)
- added C51: 22u, Capacitor_SMD:C_0603_1608Metric_Pad1.08x0.95mm_HandSolder, F.Cu at (516.0, 142.0)
- added C52: 22u, Capacitor_SMD:C_0603_1608Metric_Pad1.08x0.95mm_HandSolder, F.Cu at (518.6, 153.8)
- added C53: 22u, Capacitor_SMD:C_0603_1608Metric_Pad1.08x0.95mm_HandSolder, F.Cu at (518.6, 155.5)
- added C54: 22u, Capacitor_SMD:C_0603_1608Metric_Pad1.08x0.95mm_HandSolder, F.Cu at (513.9, 155.7)
- added C55: 100n, Capacitor_SMD:C_0603_1608Metric_Pad1.08x0.95mm_HandSolder, F.Cu at (508.1, 143.8)
- added C8: DNP, Capacitor_SMD:C_0603_1608Metric_Pad1.08x0.95mm_HandSolder, F.Cu at (389.7, 81.5)
- added CA7: 1u, Capacitor_SMD:C_0603_1608Metric_Pad1.08x0.95mm_HandSolder, F.Cu at (335.9, 116.1)
- added D14: LED_Small, LED_SMD:LED_0603_1608Metric_Pad1.05x0.95mm_HandSolder, F.Cu at (363.1, 74.0)
- added D15: D5V0P4UR6SO-7, SamacSys_Parts:SOT95P285X140-6N, F.Cu at (342.3, 90.8)
- added FID10: Cell, Z_mycustom_footprint_lib:18650 cell 3d model, B.Cu at (479.6, 104.4)
- added FID2: kicad, Symbol:KiCad-Logo2_5mm_SilkScreen, F.Cu at (408.8, 92.9)
- added FID5: Cell, Z_mycustom_footprint_lib:18650 cell 3d model, F.Cu at (435.5, 107.6)
- added FID6: garbage, Symbol:WEEE-Logo_4.2x6mm_SilkScreen, F.Cu at (418.2, 93.0)
- added FID9: Cell, Z_mycustom_footprint_lib:18650 cell 3d model, F.Cu at (450.2, 104.4)
- added H1: M3, MountingHole:MountingHole_3.2mm_M3_ISO7380_Pad_TopBottom, F.Cu at (125.0, 130.0)
- added H2: M3, MountingHole:MountingHole_3.2mm_M3_ISO7380_Pad_TopBottom, F.Cu at (185.0, 130.0)
- added H3: M3, MountingHole:MountingHole_3.2mm_M3_ISO7380_Pad_TopBottom, F.Cu at (210.0, 100.0)
- added H4: M3, MountingHole:MountingHole_3.2mm_M3_ISO7380_Pad_TopBottom, F.Cu at (185.0, 70.0)
- added H5: M3, MountingHole:MountingHole_3.2mm_M3_ISO7380_Pad_TopBottom, F.Cu at (125.0, 70.0)
- added H6: M3, MountingHole:MountingHole_3.2mm_M3_ISO7380_Pad_TopBottom, F.Cu at (100.0, 100.0)
- added J12: USB_A, Connector_USB:USB_A_Molex_105057_Vertical, F.Cu at (134.9, 122.0)
- added JP6: ADR1, Jumper:SolderJumper-3_P1.3mm_Bridged12_RoundedPad1.0x1.5mm_NumberLabels, F.Cu at (358.1, 73.8)
- added JP7: safe, Jumper:SolderJumper-2_P1.3mm_Open_RoundedPad1.0x1.5mm, F.Cu at (511.1, 143.0)
- added L1: 6u8, Z_mycustom_footprint_lib:inductor 6x6mm, F.Cu at (380.5, 171.6)
- added Q8: DMP2040USD, Package_SO:SO-8_3.9x4.9mm_P1.27mm, F.Cu at (342.9, 78.9)
- added R54: 100k, Resistor_SMD:R_0603_1608Metric_Pad0.98x0.95mm_HandSolder, F.Cu at (382.2, 185.2)
- added R55: 100k, Resistor_SMD:R_0603_1608Metric_Pad0.98x0.95mm_HandSolder, F.Cu at (358.5, 83.1)
- added R56: 100k, Resistor_SMD:R_0603_1608Metric_Pad0.98x0.95mm_HandSolder, F.Cu at (364.5, 79.0)
- added R57: 10k, Resistor_SMD:R_0603_1608Metric_Pad0.98x0.95mm_HandSolder, F.Cu at (379.0, 185.2)
- added R58: 50m, Resistor_SMD:R_0805_2012Metric, F.Cu at (349.8, 86.4)
- added R59: 1k, Resistor_SMD:R_0603_1608Metric_Pad0.98x0.95mm_HandSolder, F.Cu at (368.1, 72.0)
- added R60: 1k, Resistor_SMD:R_0603_1608Metric_Pad0.98x0.95mm_HandSolder, F.Cu at (372.4, 69.1)
- added R61: 100k, Resistor_SMD:R_0603_1608Metric_Pad0.98x0.95mm_HandSolder, F.Cu at (360.2, 76.8)
- added R62: 50m, Resistor_SMD:R_0805_2012Metric, F.Cu at (369.0, 66.4)
- added R63: 1Meg, Resistor_SMD:R_0603_1608Metric_Pad0.98x0.95mm_HandSolder, F.Cu at (452.3, 151.6)
- added R64: DNP, Resistor_SMD:R_0603_1608Metric_Pad0.98x0.95mm_HandSolder, F.Cu at (452.2, 153.5)
- added R65: 1Meg, Resistor_SMD:R_0603_1608Metric_Pad0.98x0.95mm_HandSolder, F.Cu at (452.1, 155.3)
- added R66: 180k, Resistor_SMD:R_0603_1608Metric_Pad0.98x0.95mm_HandSolder, F.Cu at (448.7, 151.6)
- added R67: 1.18Meg, Resistor_SMD:R_0603_1608Metric_Pad0.98x0.95mm_HandSolder, F.Cu at (387.5, 101.4)
- added R68: 180k, Resistor_SMD:R_0603_1608Metric_Pad0.98x0.95mm_HandSolder, F.Cu at (391.8, 101.4)
- added R69: 1.32Meg, Resistor_SMD:R_0603_1608Metric_Pad0.98x0.95mm_HandSolder, F.Cu at (513.7, 151.5)
- added R70: DNP, Resistor_SMD:R_0603_1608Metric_Pad0.98x0.95mm_HandSolder, F.Cu at (513.8, 153.6)
- added R71: 1Meg, Resistor_SMD:R_0603_1608Metric_Pad0.98x0.95mm_HandSolder, F.Cu at (518.5, 151.7)
- added R72: 200k, Resistor_SMD:R_0603_1608Metric_Pad0.98x0.95mm_HandSolder, F.Cu at (509.9, 151.7)
- added SW3: BMS_RESET, SamacSys_Parts:PTS526SK15SMTR2LFS, F.Cu at (327.3, 91.8)
- added TP2: TestPoint, TestPoint:TestPoint_Pad_1.5x1.5mm, F.Cu at (407.3, 79.3)
- added U11: TPS63020DSJR, Z_mycustom_footprint_lib:TPS63020, F.Cu at (451.4, 145.4)
- added U12: TPS63020DSJR, Z_mycustom_footprint_lib:TPS63020, F.Cu at (514.0, 147.0)
- added U2: CP2102N-Axx-xQFN24, Package_DFN_QFN:QFN-24-1EP_4x4mm_P0.5mm_EP2.6x2.6mm, F.Cu at (140.0, 124.4)
- C10: renamed from C9; moved to B.Cu
- C11, C3: value DNP -> 10u
- C15: value 100n -> DNP
- C16, C24, C30: value 1u -> 100n
- C17, C18: value 1u -> 10u
- C2: value DNP -> 220u; footprint Capacitor_SMD:C_0603_1608Metric_Pad1.08x0.95mm_HandSolder -> Capacitor_SMD:CP_Elec_8x10.5
- C20: value 1u -> 1u+
- C22: value 1u -> 4p7-10p
- C23: value 100n -> 4p7-10p
- C25: value 10u -> 220p
- C26: value 100n -> 220p
- C27, C33: value 100n -> 1u
- C28: value 22u+ -> 1u
- C29: value 10u+ -> 1u
- C35, C41, C42: value 22u -> 1u
- C36: value 22u -> 10u
- C37, C38, C43: value 22u -> 100n
- C39: value 100n -> 22u+
- C40: value 22u -> 10u+
- C5: value 10u -> 100n; moved to B.Cu
- C6: value 100n -> 33p; moved to B.Cu
- C7: value 33p -> DNP
- CA4: value 1u -> 10n?
- D10: value D5V0P4UR6SO-7 -> LED_Small; footprint SamacSys_Parts:SOT95P285X140-6N -> LED_SMD:LED_0603_1608Metric_Pad1.05x0.95mm_HandSolder
- FID4: value garbage -> Cell; footprint Symbol:WEEE-Logo_4.2x6mm_SilkScreen -> Z_mycustom_footprint_lib:18650 cell 3d model
- J10: value 140-502-415-000 -> backup; footprint SamacSys_Parts:140502415000 -> TerminalBlock:TerminalBlock_Altech_AK300-2_P5.00mm
- J11: value USB_A -> 140-502-415-000; footprint Connector_USB:USB_A_Molex_105057_Vertical -> SamacSys_Parts:140502415000
- J2: value Conn_Coaxial -> GSM; footprint Connector_Coaxial:SMA_Amphenol_901-143_Horizontal -> Z_mycustom_footprint_lib:SMA_Amphenol_901-143_Horizontal_no_edgecuts
- J4: value Conn_Coaxial -> BT; footprint Connector_Coaxial:SMA_Amphenol_901-143_Horizontal -> Z_mycustom_footprint_lib:SMA_Amphenol_901-143_Horizontal_no_edgecuts
- J5: value Conn_Coaxial -> GNSS; footprint Connector_Coaxial:SMA_Amphenol_901-143_Horizontal -> Z_mycustom_footprint_lib:SMA_Amphenol_901-143_Horizontal_no_edgecuts
- J8: moved to B.Cu
- JP1: value ADR1 -> Jumper_2_Open; footprint Jumper:SolderJumper-3_P1.3mm_Bridged12_RoundedPad1.0x1.5mm_NumberLabels -> Jumper:SolderJumper-2_P1.3mm_Open_RoundedPad1.0x1.5mm; moved to B.Cu
- JP2: value ADR0 -> Jumper_2_Open; footprint Jumper:SolderJumper-3_P1.3mm_Bridged12_RoundedPad1.0x1.5mm_NumberLabels -> Jumper:SolderJumper-2_P1.3mm_Open_RoundedPad1.0x1.5mm; moved to B.Cu
- JP3: value leds -> ADR1; footprint Connector_PinHeader_2.54mm:PinHeader_1x03_P2.54mm_Vertical -> Jumper:SolderJumper-3_P1.3mm_Bridged12_RoundedPad1.0x1.5mm_NumberLabels
- JP4: value ADR1 -> ADR0
- JP5: value safe -> leds; footprint Jumper:SolderJumper-2_P1.3mm_Open_RoundedPad1.0x1.5mm -> Connector_PinHeader_2.54mm:PinHeader_1x03_P2.54mm_Vertical
- Q6: value DMP2040USD -> BC847BS; footprint Package_SO:SO-8_3.9x4.9mm_P1.27mm -> Package_TO_SOT_SMD:SOT-363_SC-70-6_Handsoldering
- R11, R12, R20: value 100 -> 100k
- R14, R21, R41, R9: value 100k -> 100
- R18: value X -> 1k
- R27: value 2k -> 22k
- R28: value 2k -> 47k
- R29: value 100k -> 10K
- R30, R31: value 50m -> X; footprint Resistor_SMD:R_0805_2012Metric -> Resistor_SMD:R_0603_1608Metric_Pad0.98x0.95mm_HandSolder
- R32: value 100K -> 10k+
- R33, R34: value 1k -> 10k
- R35: value 100k -> 10k
- R36, R37: value 100k -> 1Meg
- R38: value 10k -> 1k
- R39: value 50m -> 1Meg; footprint Resistor_SMD:R_0805_2012Metric -> Resistor_SMD:R_0603_1608Metric_Pad0.98x0.95mm_HandSolder
- R40: value 1k -> 2k
- R42: value 50m -> 2k; footprint Resistor_SMD:R_0805_2012Metric -> Resistor_SMD:R_0603_1608Metric_Pad0.98x0.95mm_HandSolder
- R43: value 1Meg -> 1k
- R44: value DNP -> ESD supresor
- R46: value 180k -> 33k
- R47: value 1.18Meg -> 10k
- R48: value 180k -> 100k; moved to B.Cu
- R49: value 1.32Meg -> 50m; footprint Resistor_SMD:R_0603_1608Metric_Pad0.98x0.95mm_HandSolder -> Resistor_SMD:R_0805_2012Metric
- R50: value DNP -> 50m; footprint Resistor_SMD:R_0603_1608Metric_Pad0.98x0.95mm_HandSolder -> Resistor_SMD:R_0805_2012Metric
- R51: value 1Meg -> 100K
- R52: value 200k -> 1k
- R7: value 100 -> X
- R8: value 1k -> 100
- SW2: value BMS_RESET -> MCU_RESET
- U10: value TPS63020DSJR -> INA3221; footprint Z_mycustom_footprint_lib:TPS63020 -> Package_DFN_QFN:Texas_RGV_S-PVQFN-N16_EP2.1x2.1mm
- U4: value MIC5317 -> TLV320ADC3100; footprint Package_TO_SOT_SMD:SOT-23-5_HandSoldering -> Package_DFN_QFN:VQFN-24-1EP_4x4mm_P0.5mm_EP2.45x2.45mm_ThermalVias
- U5: value MIC5317 -> OP179GS; footprint Package_TO_SOT_SMD:SOT-23-5_HandSoldering -> Package_SO:SOIC-8_3.9x4.9mm_P1.27mm
- U6: value MP2615 -> MIC5317; footprint SamacSys_Parts:MP2615GQZ -> Package_TO_SOT_SMD:SOT-23-5_HandSoldering
- U7: value APX810S05 -> MIC5317; footprint Package_TO_SOT_SMD:SOT-23 -> Package_TO_SOT_SMD:SOT-23-5_HandSoldering
- U8: value INA3221 -> MP2615; footprint Package_DFN_QFN:Texas_RGV_S-PVQFN-N16_EP2.1x2.1mm -> SamacSys_Parts:MP2615GQZ
- U9: value TPS63020DSJR -> APX810S05; footprint Z_mycustom_footprint_lib:TPS63020 -> Package_TO_SOT_SMD:SOT-23
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- renumbered C8 to C9, FID2 to FID8, TP2 to TP1, U2 to U3
Connections:
- net Net-(R27-Pad2) renamed /MCU+WIFI+BT/VBUS_DETECT_CP
- C12 pad 1: Net-(C12-Pad1) -> /GSM+GPS/BT_RF1
- C13 pad 1: Net-(C13-Pad1) -> /GSM+GPS/BT_RF2
- C14 pad 1: Net-(C14-Pad1) -> /GSM+GPS/GNSS_RF1
- C15 pad 1: /Audio capture/RESET_AUDIO -> /GSM+GPS/GNSS_RF2
- C16 pad 1: +3V8 -> /MCU+WIFI+BT/VDD_CP
- C17 pad 1: Net-(C17-Pad1) -> +3V3
- C18 pad 1: +3.3VA -> +3V3
- C19 pad 1: 1V8A -> +3V3
- C2 pad 1: Net-(C2-Pad1) -> +3V8
- C20 pad 1: 1V8A -> /MCU+WIFI+BT/EN
- C21 pad 1: +3.3VA -> /MCU+WIFI+BT/BOOT
- C22 pad 1: +3.3VA -> /Audio capture/Shield1
- C23 pad 1: +3.3VA -> /Audio capture/Shield2
- C24 pad 1: +3.3VA -> /Audio capture/RESET_AUDIO
- C25 pad 1: +3V3 -> Net-(C25-Pad1)
- C26 pad 1: IN_SYSTEM- -> Net-(C26-Pad1)
- C26 pad 2: IN_SYSTEM+ -> GND
- C27 pad 1: Net-(C27-Pad1) -> +3V8
- C27 pad 2: Net-(C27-Pad2) -> GND
- C28 pad 1: IN_SYSTEM- -> Net-(C28-Pad1)
- C29 pad 1: +BATT -> +3.3VA
- C3 pad 1: Net-(C3-Pad1) -> +3V8
- C30 pad 1: /Power Management +BMS/VCC -> 1V8A
- C31 pad 1: Net-(C31-Pad1) -> 1V8A
- C32 pad 1: IN_SOLAR+ -> +3.3VA
- C32 pad 2: IN_SOLAR- -> GND
- C33 pad 1: +3V3 -> +3.3VA
- C34 pad 1: IN_USB_+ -> +3.3VA
- C34 pad 2: IN_USB_- -> GND
- C35 pad 1: +VDC -> +3.3VA
- C36 pad 1: unconnected-(C36-Pad1) -> +3V3
- C36 pad 2: unconnected-(C36-Pad2) -> GND
- C37 pad 1: unconnected-(C37-Pad1) -> IN_SYSTEM-
- C37 pad 2: unconnected-(C37-Pad2) -> IN_SYSTEM+
- C38 pad 1: unconnected-(C38-Pad1) -> /Power Management +BMS/SW
- C38 pad 2: unconnected-(C38-Pad2) -> /Power Management +BMS/BST
- C39 pad 1: Net-(C39-Pad1) -> IN_SYSTEM-
- C40 pad 1: +VDC -> +BATT
- C41 pad 1: unconnected-(C41-Pad1) -> /Power Management +BMS/VCC
- C41 pad 2: unconnected-(C41-Pad2) -> GND
- C42 pad 1: unconnected-(C42-Pad1) -> /Power Management +BMS/TMR
- C42 pad 2: unconnected-(C42-Pad2) -> GND
- C43 pad 1: unconnected-(C43-Pad1) -> IN_SOLAR+
- C43 pad 2: unconnected-(C43-Pad2) -> IN_SOLAR-
- C44 pad 1: Net-(C44-Pad1) -> +3V3
- C7 pad 1: +3V8 -> /GSM+GPS/GSM_RF1
- CA4 pad 1: Net-(CA4-Pad1) -> Net-(C25-Pad1)
- CA5 pad 1: Net-(CA5-Pad1) -> Net-(C26-Pad1)
- CA5 pad 2: Net-(CA4-Pad1) -> Net-(CA5-Pad2)
- CA6 pad 1: Net-(CA5-Pad1) -> GND
- CA6 pad 2: GND -> Net-(C26-Pad1)
- D10 pad 1: unconnected-(D10-Pad1) -> Net-(D10-Pad1)
- D10 pad 2: GND -> /Power Management +BMS/BMS_LED
- D11 pad 2: GND -> /Power Management +BMS/BMS_LED
- D5 pad 1: Net-(D5-Pad1) -> /GSM+GPS/SIM_CLK
- D5 pad 3: Net-(D5-Pad3) -> /GSM+GPS/SIM_IO
- D5 pad 6: Net-(D5-Pad6) -> /GSM+GPS/SIM_RST
- D7 pad 1: D2- -> unconnected-(D7-Pad1)
- D7 pad 3: unconnected-(D7-Pad3) -> D2+
- D7 pad 4: unconnected-(D7-Pad4) -> D2-
- D7 pad 6: D2- -> unconnected-(D7-Pad6)
- D8 pad 2: Net-(D8-Pad2) -> /MCU+WIFI+BT/VIO
- D9 pad 2: Net-(D8-Pad2) -> /MCU+WIFI+BT/VIO
- F1 pad 2: Net-(Q6-Pad3) -> Net-(F1-Pad2)
- F2 pad 1: Net-(J10-Pad2) -> Net-(F2-Pad1)
- FB1 pad 2: Net-(C17-Pad1) -> Net-(C28-Pad1)
- J1 pad 2: Net-(D5-Pad3) -> /GSM+GPS/SIM_RST
- J1 pad 3: Net-(D5-Pad6) -> /GSM+GPS/SIM_CLK
- J1 pad 7: Net-(D5-Pad1) -> /GSM+GPS/SIM_IO
- J10 pad 2: Net-(J10-Pad2) -> Net-(F2-Pad1)
- J11 pad 1: VBUS -> GND
- J11 pad 2: D- -> Net-(F2-Pad1)
- J2 pad 1: Net-(C3-Pad1) -> /GSM+GPS/GSM_RF2
- J4 pad 1: Net-(C12-Pad1) -> /GSM+GPS/BT_RF2
- J5 pad 1: Net-(C14-Pad1) -> /GSM+GPS/GNSS_RF2
- J6 pad 2: unconnected-(J6-Pad2) -> /Audio capture/Shield1
- J7 pad 1: unconnected-(J7-Pad1) -> GND
- J7 pad 2: unconnected-(J7-Pad2) -> /Audio capture/Shield2
- J7 pad 3: unconnected-(J7-Pad3) -> Net-(J7-Pad3)
- J9 pad 1: Net-(J9-Pad1) -> /Power Management +BMS/NTC
- JP1 pad 1: +3.3VA -> /MCU+WIFI+BT/ESP32_D+
- JP1 pad 2: Net-(JP1-Pad2) -> D+
- JP2 pad 1: +3.3VA -> /MCU+WIFI+BT/ESP32_D-
- JP2 pad 2: Net-(JP2-Pad2) -> D-
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Routing:
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- added copper zone on F.Cu, net GND
- added copper zone on In1.Cu, net GND
- added copper zone on In2.Cu, net GND
Other:
- board outline added: 126.5 x 76.1 mm
- copper layers 2 -> 4

Commit message: f
Parts:
- removed the C38 at (347.2, 92.3)
- removed the C39 at (377.6, 179.6)
- removed the C40 at (391.2, 182.0)
- removed the D10 at (371.0, 183.3)
- removed the D11 at (370.9, 181.5)
- removed the J9 at (376.9, 188.8)
- removed the JP5 at (367.0, 180.9)
- removed the R50 at (390.2, 178.6)
- removed the R51 at (383.8, 185.2)
- removed the R52 at (374.7, 183.3)
- removed the R53 at (374.6, 181.6)
- removed the R54 at (382.2, 185.2)
- removed SW3: BMS_RESET, SamacSys_Parts:PTS526SK15SMTR2LFS
- removed the U8 at (382.6, 180.5)
- added C19: 100n, Capacitor_SMD:C_0603_1608Metric_Pad1.08x0.95mm_HandSolder, F.Cu at (425.2, 206.1)
- added C43: 220n, Capacitor_SMD:C_0603_1608Metric_Pad1.08x0.95mm_HandSolder, F.Cu at (409.1, 208.1)
- added C45: 22u, Capacitor_SMD:C_0603_1608Metric_Pad1.08x0.95mm_HandSolder, F.Cu at (416.2, 202.6)
- added C56: 100n, Capacitor_SMD:C_0603_1608Metric_Pad1.08x0.95mm_HandSolder, F.Cu at (373.6, 175.7)
- added C57: 4.7n, Capacitor_SMD:C_0603_1608Metric_Pad1.08x0.95mm_HandSolder, F.Cu at (386.6, 172.8)
- added D14: LED_Small, LED_SMD:LED_0603_1608Metric_Pad1.05x0.95mm_HandSolder, F.Cu at (404.8, 209.1)
- added D15: LED_Small, LED_SMD:LED_0603_1608Metric_Pad1.05x0.95mm_HandSolder, F.Cu at (407.5, 205.6)
- added J12: Screw_Terminal_01x03, TerminalBlock:TerminalBlock_Altech_AK300-3_P5.00mm, F.Cu at (370.5, 167.5)
- added NT1: NetTie_2, NetTie:NetTie-2_SMD_Pad0.5mm, F.Cu at (430.4, 205.9)
- added NT2: NetTie_2, NetTie:NetTie-2_SMD_Pad0.5mm, F.Cu at (433.1, 203.5)
- added R58: 100k, Resistor_SMD:R_0603_1608Metric_Pad0.98x0.95mm_HandSolder, F.Cu at (411.8, 205.5)
- added R59: X, Resistor_SMD:R_0603_1608Metric_Pad0.98x0.95mm_HandSolder, F.Cu at (411.9, 202.6)
- added R60: 120, Resistor_SMD:R_0603_1608Metric_Pad0.98x0.95mm_HandSolder, F.Cu at (413.5, 208.0)
- added R61: 50m, Resistor_SMD:R_0805_2012Metric, F.Cu at (407.5, 202.8)
- added R72: 10k, Resistor_SMD:R_0603_1608Metric_Pad0.98x0.95mm_HandSolder, F.Cu at (509.2, 201.7)
- added R73: 10k, Resistor_SMD:R_0603_1608Metric_Pad0.98x0.95mm_HandSolder, F.Cu at (509.2, 199.2)
- added R74: 60, Resistor_SMD:R_0603_1608Metric_Pad0.98x0.95mm_HandSolder, F.Cu at (378.0, 175.7)
- added R75: 300, Resistor_SMD:R_0603_1608Metric_Pad0.98x0.95mm_HandSolder, F.Cu at (369.3, 175.7)
- added R76: 60, Resistor_SMD:R_0603_1608Metric_Pad0.98x0.95mm_HandSolder, F.Cu at (395.0, 161.7)
- added U10: CN3791, Package_SO:SSOP-10_3.9x4.9mm_P1.00mm, F.Cu at (401.4, 204.5)
- added U14: 74LVC1G08, Package_TO_SOT_SMD:SOT-23-5_HandSoldering, B.Cu at (387.3, 169.2)
- added U15: MCP2561-H-SN, Package_SO:SOIC-8_3.9x4.9mm_P1.27mm, B.Cu at (152.3, 121.5)
- added U3: BME280, Package_LGA:Bosch_LGA-8_2.5x2.5mm_P0.65mm_ClockwisePinNumbering, F.Cu at (430.7, 203.4)
- C20: value 1u+ -> z
- C41: value 1u -> 22u
- C42: value 1u -> 100n
- JP1: value Jumper_2_Open -> ADR0; footprint Jumper:SolderJumper-2_P1.3mm_Open_RoundedPad1.0x1.5mm -> Jumper:SolderJumper-3_P1.3mm_Bridged12_RoundedPad1.0x1.5mm_NumberLabels; moved to F.Cu
- JP2: value Jumper_2_Open -> LED_on/off; footprint Jumper:SolderJumper-2_P1.3mm_Open_RoundedPad1.0x1.5mm -> Connector_PinHeader_2.54mm:PinHeader_1x03_P2.54mm_Vertical; moved to F.Cu
- L1: value 6u8 -> x; footprint Z_mycustom_footprint_lib:inductor 6x6mm -> Inductor_SMD:L_Wuerth_MAPI-3012
- R27: renamed from R32; value 10k+ -> y
- R57: value 10k -> 100k
- moved JP1 279.7 mm to (425.9, 203.1), turned to 0 degrees
- moved JP2 247.0 mm to (403.5, 162.8), turned to 0 degrees
- moved L1 43.4 mm to (400.1, 210.3)
- moved C42 43.2 mm to (409.1, 210.6), turned to 0 degrees
- moved R57 42.1 mm to (416.2, 205.1), turned to 0 degrees
- moved C41 35.8 mm to (404.8, 211.6), turned to 0 degrees
- moved U6 18.8 mm to (148.5, 97.4), turned to 90 degrees
- moved D1 9.85 mm to (200.2, 114.1)
- moved J1 3.97 mm to (203.3, 126.0)
- moved FID9 3.15 mm to (435.5, 104.4)
- moved TP2 3.00 mm to (190.8, 113.5)
- moved C15 1.20 mm to (186.9, 114.2)
- moved D6 1.20 mm to (183.9, 111.3)
- moved J5 1.20 mm to (183.6, 116.3)
- moved FID7 0.56 mm to (467.9, 104.4)
- renumbered C4 to C10, C5 to C12, C6 to C13, C10 to C14, C9 to C15, C17 to C16, C18 to C17, C19 to C18, C7 to C2, C16 to C22, C22 to C23, C25 to C24, C23 to C25, C24 to C27, C27 to C28, C28 to C29, C12 to C3, C29 to C30, C32 to C31, C33 to C32, C34 to C33, C35 to C34, C30 to C35, C31 to C36, C36 to C37, C45 to C38, C43 to C39, C14 to C4, C37 to C40, C51 to C46, C46 to C47, C55 to C48, C50 to C49, C8 to C5, C52 to C50, C53 to C51, C47 to C52, C54 to C53, C48 to C54, C49 to C55, C13 to C6, C15 to C7, C2 to C8, C3 to C9, CA4 to CA1, CA6 to CA3, CA1 to CA4, CA3 to CA5, CA5 to CA6, D5 to D1, D14 to D10, D12 to D11, D13 to D12, D15 to D13, D6 to D2, D1 to D3, D2 to D5, D7 to D6, D3 to D7, F3 to F2, F2 to F3, FID8 to FID2, FID2 to FID3, FID6 to FID4, FID4 to FID7, FID9 to FID8, FID5 to FID9, J11 to J10, J10 to J11, J4 to J3, J5 to J4, J3 to J5, J7 to J6, J6 to J7, J12 to J9, JP3 to JP4, JP4 to JP5, L3 to L2, L2 to L3, Q2 to Q1, Q4 to Q2, Q1 to Q3, Q5 to Q4, Q3 to Q5, R16 to R1, R25 to R10, R8 to R12, R5 to R13, R20 to R14, R19 to R15, R17 to R16, R12 to R17, R9 to R18, R6 to R19, R15 to R2, R22 to R20, R13 to R22, R18 to R23, R10 to R24, R7 to R25, R29 to R26, R35 to R28, R26 to R29, R1 to R3, R34 to R30, R33 to R31, R27 to R32, R28 to R33, R30 to R34, R31 to R35, R44 to R36, R41 to R37, R36 to R38, R45 to R39, R3 to R4, R37 to R40, R39 to R41, R46 to R42, R47 to R43, R43 to R44, R40 to R45, R42 to R46, R38 to R47, R59 to R49, R4 to R5, R62 to R50, R58 to R51, R55 to R52, R56 to R53, R60 to R54, R61 to R55, R49 to R56, R2 to R6, R69 to R62, R72 to R63, R63 to R64, R66 to R65, R67 to R66, R68 to R67, R70 to R68, R64 to R69, R14 to R7, R71 to R70, R65 to R71, R23 to R8, R24 to R9, TP2 to TP1, TP1 to TP2, U10 to U11, U11 to U13, U3 to U2, U2 to U4, U4 to U6, U6 to U7, U7 to U8
Connections:
- net Net-(R65-Pad2) renamed /Power Management +BMS/PG_3V3
- net Net-(R71-Pad2) renamed /Power Management +BMS/PG_3V8
- C1 pad 2: GND -> +3V3
- C10 pad 2: GND -> +3V3
- C11 pad 2: GND -> +3V3
- C12 pad 2: GND -> +3V3
- C13 pad 2: GND -> +3V3
- C14 pad 2: GND -> +3V3
- C16 pad 2: GND -> +3V3
- C17 pad 2: GND -> +3V3
- C18 pad 2: GND -> +3V3
- C2 pad 2: GND -> +3V3
- C20 pad 2: GND -> +3V3
- C21 pad 2: GND -> +3V3
- C22 pad 2: GND -> +3V3
- C23 pad 2: GND -> +3V3
- C24 pad 2: GND -> +3V3
- C25 pad 2: GND -> +3V3
- C26 pad 2: GND -> +3V3
- C27 pad 1: /Audio capture/RESET_AUDIO -> /MCU+WIFI+BT/GPIO_38
- C27 pad 2: GND -> +3V3
- C28 pad 2: GND -> +3V3
- C29 pad 2: GND -> +3V3
- C3 pad 2: GND -> +3V3
- C30 pad 2: GND -> +3V3
- C31 pad 2: GND -> +3V3
- C32 pad 2: GND -> +3V3
- C33 pad 2: GND -> +3V3
- C34 pad 2: GND -> +3V3
- C35 pad 2: GND -> +3V3
- C36 pad 2: GND -> +3V3
- C37 pad 2: GND -> +3V3
- C4 pad 2: GND -> +3V3
- C41 pad 1: /Power Management +BMS/VCC -> IN_SYSTEM-
- C41 pad 2: GND -> +3V3
- C42 pad 1: /Power Management +BMS/TMR -> Net-(C42-Pad1)
- C42 pad 2: GND -> IN_SYSTEM-
- C44 pad 2: GND -> +3V3
- C46 pad 2: GND -> +3V3
- C47 pad 2: GND -> +3V3
- C48 pad 2: GND -> +3V3
- C49 pad 2: GND -> +3V3
- C5 pad 2: GND -> +3V3
- C50 pad 2: GND -> +3V3
- C51 pad 2: GND -> +3V3
- C52 pad 2: GND -> +3V3
- C53 pad 2: GND -> +3V3
- C54 pad 2: GND -> +3V3
- C55 pad 2: GND -> +3V3
- C6 pad 2: GND -> +3V3
- C7 pad 2: GND -> +3V3
- C8 pad 2: GND -> +3V3
- C9 pad 2: GND -> +3V3
- CA3 pad 1: GND -> +3V3
- CA4 pad 2: GND -> +3V3
- CA7 pad 1: GND -> +3V3
- CA7 pad 2: GND -> +3V3
- D1 pad 2: GND -> +3V3
- D10 pad 2: GND -> +3V3
- D11 pad 2: GND -> +3V3
- D12 pad 2: GND -> +3V3
- D13 pad 2: GND -> +3V3
- D2 pad 2: GND -> +3V3
- D3 pad 2: +3V8 -> /GSM+GPS/LED_PWR
- D4 pad 2: +3V8 -> /GSM+GPS/LED_PWR
- D5 pad 2: +3V8 -> /GSM+GPS/LED_PWR
- D6 pad 2: GND -> +3V3
- D7 pad 2: +3V8 -> /GSM+GPS/LED_PWR
- H1 pad 1: GND -> +3V3
- H2 pad 1: GND -> +3V3
- H3 pad 1: GND -> +3V3
- H4 pad 1: GND -> +3V3
- H5 pad 1: GND -> +3V3
- H6 pad 1: GND -> +3V3
- IC1 pad 1: +3V3 -> /GSM+GPS/DTR
- IC1 pad 10: +3V3 -> /GSM+GPS/OE_ENABLE
- IC1 pad 11: GND -> +3V3
- J1 pad 5: GND -> +3V3
- J1 pad SH: GND -> +3V3
- J10 pad 1: GND -> +3V3
- J11 pad 1: GND -> +3V3
- J2 pad 2: GND -> +3V3
- J3 pad 2: GND -> +3V3
- J4 pad 2: GND -> +3V3
- J5 pad 4: GND -> +3V3
- J6 pad 1: GND -> +3V3
- J8 pad 1: /MCU+WIFI+BT/DATA2 -> /MCU+WIFI+BT/GPIO_17
- J8 pad 11: GND -> +3V3
- J8 pad 2: /MCU+WIFI+BT/DATA3/CS -> /MCU+WIFI+BT/GPIO_16
- J8 pad 3: /MCU+WIFI+BT/CMD -> /MCU+WIFI+BT/GPIO_15
- J8 pad 5: /MCU+WIFI+BT/SCLK -> /MCU+WIFI+BT/GPIO_07
- J8 pad 6: GND -> +3V3
- J8 pad 7: /MCU+WIFI+BT/DATA0 -> /MCU+WIFI+BT/GPIO_06
- J8 pad 8: /MCU+WIFI+BT/DATA1 -> /MCU+WIFI+BT/GPIO_05
- J8 pad 9: /MCU+WIFI+BT/CARD_DET -> /MCU+WIFI+BT/GPIO_04
- J9 pad 4: GND -> +3V3
- JP1 pad 1: /MCU+WIFI+BT/ESP32_D+ -> +3V3
- JP1 pad 2: D+ -> Net-(JP1-Pad2)
- JP2 pad 1: /MCU+WIFI+BT/ESP32_D- -> +3V8
- JP2 pad 2: D- -> /GSM+GPS/LED_PWR
- JP4 pad 3: GND -> +3V3
- JP5 pad 3: GND -> +3V3
- JP6 pad 3: GND -> +3V3
- L1 pad 1: /Power Management +BMS/SW -> Net-(D16-Pad1)
- L1 pad 2: /Power Management +BMS/CSP -> Net-(L1-Pad2)
- Q1 pad 1: /Audio capture/SDA -> /MCU+WIFI+BT/GPIO_36
- Q1 pad 4: /Audio capture/SCL -> /MCU+WIFI+BT/GPIO_35
- Q2 pad 1: GND -> +3V3
- Q3 pad 4: GND -> +3V3
- Q4 pad 1: GND -> +3V3
- Q4 pad 4: GND -> +3V3
- Q5 pad 1: GND -> +3V3
- Q5 pad 4: GND -> +3V3
- R1 pad 1: GND -> +3V3
- R11 pad 1: GND -> +3V3
- R14 pad 1: GND -> +3V3
- R17 pad 1: GND -> +3V3
- R20 pad 1: GND -> +3V3
- R22 pad 1: GND -> +3V3
- R26 pad 2: GND -> +3V3
- R27 pad 2: +3V3 -> /MCU+WIFI+BT/PG_3V3
- R33 pad 2: GND -> +3V3
- R36 pad 2: GND -> +3V3
- R38 pad 2: GND -> +3V3
- R39 pad 2: GND -> +3V3
- R40 pad 2: GND -> +3V3
- R43 pad 1: GND -> +3V3
- R48 pad 1: /MCU+WIFI+BT/CARD_DET -> /MCU+WIFI+BT/GPIO_04
- R52 pad 2: GND -> +3V3
- R53 pad 2: GND -> +3V3
- R54 pad 2: GND -> +3V3
- R55 pad 2: GND -> +3V3
- R57 pad 1: /Power Management +BMS/NTC -> IN_SYSTEM-
- R57 pad 2: /Power Management +BMS/VCC -> Net-(R57-Pad2)
- R63 pad 2: GND -> +3V3
- R65 pad 2: GND -> +3V3
- SW1 pad 1: GND -> +3V3
- SW2 pad 2: GND -> +3V3
- U1 pad 1: GND -> +3V3
- U1 pad 18: GND -> +3V3
- U1 pad 2: GND -> +3V3
- U1 pad 28: GND -> +3V3
- U1 pad 3: GND -> +3V3
- U1 pad 34: GND -> +3V3
- U1 pad 36: GND -> +3V3
- U1 pad 40: GND -> +3V3
- U1 pad 51: GND -> +3V3
- U1 pad 52: GND -> +3V3
- U1 pad 54: GND -> +3V3
- U1 pad 64: GND -> +3V3
- U1 pad 65: GND -> +3V3
- U1 pad 67: GND -> +3V3
- U1 pad 68: GND -> +3V3
- U11 pad 17: GND -> +3V3
- U11 pad 3: GND -> +3V3
- U11 pad 6: /Audio capture/SCL -> /MCU+WIFI+BT/GPIO_35
- U11 pad 7: /Audio capture/SDA -> /MCU+WIFI+BT/GPIO_36
- U12 pad 2: GND -> +3V3
- U13 pad 2: GND -> +3V3
- U2 pad 1: GND -> +3V3
- U2 pad 11: /MCU+WIFI+BT/GPIO_18 -> /GSM+GPS/RI
- U2 pad 12: /MCU+WIFI+BT/GPIO_08 -> /GSM+GPS/DCD
- U2 pad 13: /MCU+WIFI+BT/ESP32_D- -> USB_OTG_D-
- U2 pad 14: /MCU+WIFI+BT/ESP32_D+ -> USB_OTG_D+
- U2 pad 17: /MCU+WIFI+BT/GPIO_09 -> /GSM+GPS/STAT
- U2 pad 18: /MCU+WIFI+BT/GPIO_10 -> /GSM+GPS/RESET
- U2 pad 19: /MCU+WIFI+BT/GPIO_11 -> /GSM+GPS/TX
- U2 pad 20: /MCU+WIFI+BT/GPIO_12 -> /GSM+GPS/RX
- U2 pad 21: /MCU+WIFI+BT/GPIO_13 -> /GSM+GPS/RTS
- U2 pad 22: /MCU+WIFI+BT/GPIO_14 -> /GSM+GPS/CTS
- U2 pad 30: /MCU+WIFI+BT/GPIO_37 -> /GSM+GPS/DTR
- U2 pad 40: GND -> +3V3
- U2 pad 41: GND -> +3V3
- U4 pad 2: GND -> +3V3
- U4 pad 25: GND -> +3V3
- U5 pad 4: GND -> +3V3
- U6 pad 1: /Audio capture/SCK -> /MCU+WIFI+BT/GPIO_48
- U6 pad 13: GND -> +3V3
- U6 pad 17: /Audio capture/SCL -> /MCU+WIFI+BT/GPIO_35
- U6 pad 18: /Audio capture/SDA -> /MCU+WIFI+BT/GPIO_36
- U6 pad 2: /Audio capture/WS -> /MCU+WIFI+BT/GPIO_47
- U6 pad 23: GND -> +3V3
- U6 pad 3: /Audio capture/SD -> /MCU+WIFI+BT/GPIO_21
- U6 pad 4: /Audio capture/RESET_AUDIO -> /MCU+WIFI+BT/GPIO_38
- U6 pad 6: GND -> +3V3
- U6 pad 9: GND -> +3V3
- U7 pad 2: GND -> +3V3
- U8 pad 2: GND -> +3V3
- U9 pad 2: GND -> +3V3
- Y1 pad 2: GND -> +3V3
Routing:
- net GND: vias 2 -> 0
- net +3V3: vias 0 -> 2
- added copper zone on F.Cu, net +3V3
- added copper zone on In1.Cu, net +3V3
- added copper zone on In2.Cu, net +3V3
- removed copper zone on F.Cu, net GND
- removed copper zone on In1.Cu, net GND
- removed copper zone on In2.Cu, net GND

Commit message: v
Parts:
- removed the C2 at (402.8, 82.1)
- removed the C3 at (398.4, 82.1)
- removed the C4 at (388.8, 84.0)
- removed the C5 at (389.7, 81.5)
- removed the C6 at (417.9, 68.7)
- removed CA7: 1u, Capacitor_SMD:C_0603_1608Metric_Pad1.08x0.95mm_HandSolder
- removed the D5 at (396.1, 69.5)
- removed the D7 at (390.3, 76.5)
- removed FID7: Cell, Z_mycustom_footprint_lib:18650 cell 3d model
- removed the FID8 at (450.2, 104.4)
- removed the J10 at (342.4, 67.9)
- removed JP7: safe, Jumper:SolderJumper-2_P1.3mm_Open_RoundedPad1.0x1.5mm
- removed the R23 at (393.1, 84.0)
- removed the R24 at (409.2, 71.2)
- removed the R25 at (384.4, 84.9)
- removed the R60 at (413.5, 208.0)
- removed the TP1 at (407.3, 79.3)
- removed the U3 at (430.7, 203.4)
- removed the U8 at (334.3, 109.0)
- added C12: DNP, Capacitor_SMD:C_0603_1608Metric_Pad1.08x0.95mm_HandSolder, F.Cu at (316.1, 131.1)
- added C13: DNP, Capacitor_SMD:C_0603_1608Metric_Pad1.08x0.95mm_HandSolder, F.Cu at (326.6, 123.6)
- added C14: DNP, Capacitor_SMD:C_0603_1608Metric_Pad1.08x0.95mm_HandSolder, F.Cu at (308.8, 130.1)
- added C15: DNP, Capacitor_SMD:C_0603_1608Metric_Pad1.08x0.95mm_HandSolder, F.Cu at (321.9, 126.1)
- added C58: 22u, Capacitor_SMD:C_0603_1608Metric_Pad1.08x0.95mm_HandSolder, F.Cu at (356.7, 101.7)
- added C59: 22u, Capacitor_SMD:C_0603_1608Metric_Pad1.08x0.95mm_HandSolder, F.Cu at (346.6, 106.7)
- added C60: 22u, Capacitor_SMD:C_0603_1608Metric_Pad1.08x0.95mm_HandSolder, F.Cu at (359.7, 109.2)
- added C61: 100n, Capacitor_SMD:C_0603_1608Metric_Pad1.08x0.95mm_HandSolder, F.Cu at (361.1, 101.7)
- added C62: 22u, Capacitor_SMD:C_0603_1608Metric_Pad1.08x0.95mm_HandSolder, F.Cu at (352.2, 114.3)
- added C63: 22u, Capacitor_SMD:C_0603_1608Metric_Pad1.08x0.95mm_HandSolder, F.Cu at (356.7, 104.2)
- added C64: 22u, Capacitor_SMD:C_0603_1608Metric_Pad1.08x0.95mm_HandSolder, F.Cu at (351.0, 111.8)
- added C65: 22u, Capacitor_SMD:C_0603_1608Metric_Pad1.08x0.95mm_HandSolder, F.Cu at (361.1, 104.2)
- added C66: 100n, Capacitor_SMD:C_0603_1608Metric_Pad1.08x0.95mm_HandSolder, F.Cu at (359.7, 106.7)
- added C8: DNP, Capacitor_SMD:C_0603_1608Metric_Pad1.08x0.95mm_HandSolder, F.Cu at (313.5, 121.1)
- added D1: LED_Small, LED_SMD:LED_0603_1608Metric_Pad1.05x0.95mm_HandSolder, F.Cu at (298.7, 133.5)
- added D16: LED_Small, LED_SMD:LED_0603_1608Metric_Pad1.05x0.95mm_HandSolder, F.Cu at (292.5, 86.7)
- added D17: D5V0P4UR6SO-7, SamacSys_Parts:SOT95P285X140-6N, F.Cu at (270.2, 106.5)
- added D18: SX33L_R1_00001, Diode_SMD:D_SMA_Handsoldering, F.Cu at (252.9, 102.7)
- added D2: LED_Small, LED_SMD:LED_0603_1608Metric_Pad1.05x0.95mm_HandSolder, F.Cu at (309.2, 120.0)
- added FID4: Cell, Z_mycustom_footprint_lib:18650 cell 3d model, F.Cu at (324.1, 103.6)
- added FID5: Cell, Z_mycustom_footprint_lib:18650 cell 3d model, F.Cu at (324.1, 101.5)
- added J14: batt input, TerminalBlock:TerminalBlock_Altech_AK300-3_P5.00mm, F.Cu at (106.0, 116.0)
- added J8: 292132-3, SamacSys_Parts:SHDR3W65P0X200_1X3_780X580X710P, F.Cu at (138.9, 77.0)
- added J9: 292132-3, SamacSys_Parts:SHDR3W65P0X200_1X3_780X580X710P, F.Cu at (138.9, 68.3)
- added JP3: ADR1, Jumper:SolderJumper-3_P1.3mm_Bridged12_RoundedPad1.0x1.5mm_NumberLabels, B.Cu at (152.0, 90.1)
- added Q10: SSM6N7002, Package_TO_SOT_SMD:SOT-363_SC-70-6_Handsoldering, F.Cu at (286.6, 80.8)
- added Q11: DMP3028LSD, Package_SO:SO-8_3.9x4.9mm_P1.27mm, F.Cu at (279.5, 80.2)
- added Q9: DMP3028LSD, Package_SO:SO-8_3.9x4.9mm_P1.27mm, F.Cu at (269.4, 91.0)
- added R10: 100, Resistor_SMD:R_0603_1608Metric_Pad0.98x0.95mm_HandSolder, F.Cu at (317.6, 126.1)
- added R48: 33k, Resistor_SMD:R_0603_1608Metric_Pad0.98x0.95mm_HandSolder, F.Cu at (148.4, 85.6)
- added R77: 50k+, Resistor_SMD:R_0603_1608Metric_Pad0.98x0.95mm_HandSolder, F.Cu at (290.1, 101.0)
- added R78: 50m, Resistor_SMD:R_0805_2012Metric, F.Cu at (277.1, 102.8)
- added R79: 50k+, Resistor_SMD:R_0603_1608Metric_Pad0.98x0.95mm_HandSolder, F.Cu at (301.2, 86.1)
- added R8: 100, Resistor_SMD:R_0603_1608Metric_Pad0.98x0.95mm_HandSolder, F.Cu at (326.6, 121.1)
- added R80: 50k+, Resistor_SMD:R_0603_1608Metric_Pad0.98x0.95mm_HandSolder, F.Cu at (307.0, 84.2)
- added R81: 50m, Resistor_SMD:R_0805_2012Metric, F.Cu at (302.3, 78.4)
- added R82: 1k, Resistor_SMD:R_0603_1608Metric_Pad0.98x0.95mm_HandSolder, F.Cu at (290.5, 98.4)
- added R83: 100k, Resistor_SMD:R_0603_1608Metric_Pad0.98x0.95mm_HandSolder, F.Cu at (290.4, 95.9)
- added R84: 100k, Resistor_SMD:R_0603_1608Metric_Pad0.98x0.95mm_HandSolder, F.Cu at (291.5, 92.2)
- added R85: 1Meg, Resistor_SMD:R_0603_1608Metric_Pad0.98x0.95mm_HandSolder, F.Cu at (351.0, 109.3)
- added R86: DNP, Resistor_SMD:R_0603_1608Metric_Pad0.98x0.95mm_HandSolder, F.Cu at (355.3, 109.3)
- added R87: 1Meg, Resistor_SMD:R_0603_1608Metric_Pad0.98x0.95mm_HandSolder, F.Cu at (343.5, 114.7)
- added R88: 180k, Resistor_SMD:R_0603_1608Metric_Pad0.98x0.95mm_HandSolder, F.Cu at (351.0, 106.7)
- added R89: 1.32Meg, Resistor_SMD:R_0603_1608Metric_Pad0.98x0.95mm_HandSolder, F.Cu at (346.6, 111.8)
- added R9: 100, Resistor_SMD:R_0603_1608Metric_Pad0.98x0.95mm_HandSolder, F.Cu at (308.8, 127.6)
- added R90: DNP, Resistor_SMD:R_0603_1608Metric_Pad0.98x0.95mm_HandSolder, F.Cu at (346.6, 109.3)
- added R91: 1Meg, Resistor_SMD:R_0603_1608Metric_Pad0.98x0.95mm_HandSolder, F.Cu at (355.3, 111.8)
- added R92: 200k, Resistor_SMD:R_0603_1608Metric_Pad0.98x0.95mm_HandSolder, F.Cu at (339.1, 114.7)
- added R93: 10k, Resistor_SMD:R_0603_1608Metric_Pad0.98x0.95mm_HandSolder, F.Cu at (353.4, 83.8)
- added R94: 100, Resistor_SMD:R_0603_1608Metric_Pad0.98x0.95mm_HandSolder, F.Cu at (353.4, 81.3)
- added R95: 100k, Resistor_SMD:R_0603_1608Metric_Pad0.98x0.95mm_HandSolder, F.Cu at (349.1, 81.3)
- added TH1: 100k, Resistor_SMD:R_1812_4532Metric_Pad1.30x3.40mm_HandSolder, F.Cu at (271.2, 101.7)
- added TH2: 100k, Resistor_SMD:R_1812_4532Metric_Pad1.30x3.40mm_HandSolder, F.Cu at (268.9, 96.7)
- added TP2: TestPoint, TestPoint:TestPoint_Pad_1.5x1.5mm, F.Cu at (332.0, 116.6)
- added U15: APX810S05, Package_TO_SOT_SMD:SOT-23, F.Cu at (302.5, 74.7)
- added U16: TPS63020DSJR, Z_mycustom_footprint_lib:TPS63020, F.Cu at (340.5, 110.0)
- added U17: TPS63020DSJR, Z_mycustom_footprint_lib:TPS63020, F.Cu at (340.5, 103.5)
- added U6: 74LVC1G08, Package_SO:TSOP-5_1.65x3.05mm_P0.95mm, F.Cu at (341.1, 78.6)
- C16: value 10u -> 4p7-10p
- C17, C37: value 10u -> 100n
- C19: value 100n -> 10u
- C20: value z -> 10u
- C23: value 4p7-10p -> z
- C24: value 220p -> 4.7n
- C25: value 4p7-10p -> 100n
- C26: value 220p -> 100n
- C27, C33: value 100n -> 15n
- C28, C30: value 1u -> 15n
- C29: value 1u -> 100n
- C31: value 100n -> 4p7-10p
- C32: value 1u -> 4p7-10p
- C35, C38, C40, C42: value 100n -> 1u
- C41, C45, C53, C54, C55: value 22u -> 100n
- C43: value 220n -> 10u
- C44, F1, F3, R61: moved to B.Cu
- C46, C47: value 22u -> 10u
- C48, C49: value 100n -> 22u
- C50: value 22u -> 1u
- C51: value 22u -> 3.5n; moved to B.Cu
- C52: value 22u -> 220n
- C57: value 4.7n -> 22u
- CA6: value 1u -> 10n?
- D10: value LED_Small -> SX33L_R1_00001; footprint LED_SMD:LED_0603_1608Metric_Pad1.05x0.95mm_HandSolder -> Diode_SMD:D_SMA_Handsoldering
- D11: value MMSZ5245B -> SX33L_R1_00001; footprint Diode_SMD:D_SOD-123 -> Diode_SMD:D_SMA_Handsoldering; moved to B.Cu
- D13: value D5V0P4UR6SO-7 -> MMSZ5245B; footprint SamacSys_Parts:SOT95P285X140-6N -> Diode_SMD:D_SOD-123
- FID10: moved to F.Cu
- FID2: renamed from FID3; moved to B.Cu
- FID6: renamed from FID4; moved to B.Cu
- J11: value backup -> Solar input; footprint TerminalBlock:TerminalBlock_Altech_AK300-2_P5.00mm -> TerminalBlock:TerminalBlock_Altech_AK300-3_P5.00mm
- J12: value Screw_Terminal_01x03 -> 140-502-415-000; footprint TerminalBlock:TerminalBlock_Altech_AK300-3_P5.00mm -> SamacSys_Parts:140502415000; moved to B.Cu
- J6: value 292132-3 -> USB1046-GF-0190-L-B-A; footprint SamacSys_Parts:SHDR3W65P0X200_1X3_780X580X710P -> SamacSys_Parts:USB1046GF0190LBA; moved to B.Cu
- J7: value 292132-3 -> Screw_Terminal_01x03; footprint SamacSys_Parts:SHDR3W65P0X200_1X3_780X580X710P -> TerminalBlock:TerminalBlock_Altech_AK300-3_P5.00mm
- JP1: value ADR0 -> LED_on/off; footprint Jumper:SolderJumper-3_P1.3mm_Bridged12_RoundedPad1.0x1.5mm_NumberLabels -> Connector_PinHeader_2.54mm:PinHeader_1x03_P2.54mm_Vertical
- JP2: value LED_on/off -> ADR0; footprint Connector_PinHeader_2.54mm:PinHeader_1x03_P2.54mm_Vertical -> Jumper:SolderJumper-3_P1.3mm_Bridged12_RoundedPad1.0x1.5mm_NumberLabels
- JP4: value ADR1 -> ADR0; moved to B.Cu
- JP5: value ADR0 -> ADR1
- JP6: value ADR1 -> safe; footprint Jumper:SolderJumper-3_P1.3mm_Bridged12_RoundedPad1.0x1.5mm_NumberLabels -> Jumper:SolderJumper-2_P1.3mm_Open_RoundedPad1.0x1.5mm
- L1: value x -> 15u; footprint Inductor_SMD:L_Wuerth_MAPI-3012 -> Z_mycustom_footprint_lib:L_SMD_3131_(8080_metric)
- Q7, Q8: value DMP2040USD -> DMP3028LSD
- R1, R14, R53: value 100k -> 100
- R12: value 100 -> 100k
- R13, R16: value X -> 100k
- R17: value 100k -> X
- R18: value 100 -> 1k
- R19: value X -> 100
- R26: value 10K -> 1k
- R27: value y -> 1Meg
- R28: value 10k -> 22k
- R29: value 1k -> 47k
- R3: value 100 -> 10k
- R30: value 10k -> 10K
- R31, R5: value 10k -> X
- R32: value 22k -> X
- R33: value 47k -> y
- R34, R35, R59: value X -> 10k
- R36: value ESD supresor -> 10k
- R37: value 100 -> 60
- R38: value 1Meg -> 300
- R39: value 1Meg -> 60
- R40, R41, R71: value 1Meg -> 10k
- R42: value 33k -> 2k
- R43: value 10k -> 1Meg
- R44, R49, R54: value 1k -> 100
- R45: value 2k -> 100
- R46: value 2k -> 1k
- R47: value 1k -> ESD supresor
- R50: value 50m -> 10k; footprint Resistor_SMD:R_0805_2012Metric -> Resistor_SMD:R_0603_1608Metric_Pad0.98x0.95mm_HandSolder
- R51: value 50m -> 2k; footprint Resistor_SMD:R_0805_2012Metric -> Resistor_SMD:R_0603_1608Metric_Pad0.98x0.95mm_HandSolder
- R52, R55: value 100k -> 1Meg
- R56: value 50m -> 1Meg; footprint Resistor_SMD:R_0805_2012Metric -> Resistor_SMD:R_0603_1608Metric_Pad0.98x0.95mm_HandSolder
- R57: value 100k -> ESD supresor
- R58: value 100k -> 33k
- R6, R7: value 100 -> X
- R62: value 1.32Meg -> 50m; footprint Resistor_SMD:R_0603_1608Metric_Pad0.98x0.95mm_HandSolder -> Resistor_SMD:R_0805_2012Metric
- R63: value 200k -> 45; moved to B.Cu
- R64: value 1Meg -> 1k
- R65: value 180k -> 1k
- R66: value 1.18Meg -> 1k
- R67: value 180k -> 100k
- R68: value DNP -> X
- R69: value DNP -> 1Meg
- R70: value 1Meg -> 120
- R72: value 10k -> 280.5587k
- R73: value 10k -> 64k
- R74: value 60 -> 100k
- R75: value 300 -> 100k
- R76: value 60 -> 50k+
- U10: value CN3791 -> MIC5317; footprint Package_SO:SSOP-10_3.9x4.9mm_P1.00mm -> Package_TO_SOT_SMD:SOT-23-5_HandSoldering
- U11: value INA3221 -> MIC5317; footprint Package_DFN_QFN:Texas_RGV_S-PVQFN-N16_EP2.1x2.1mm -> Package_TO_SOT_SMD:SOT-23-5_HandSoldering
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- renumbered C14 to C10, C8 to C2, C9 to C3, C10 to C4, C12 to C5, C13 to C6, C15 to C9, D1 to D5, D2 to D6, D6 to D7, FID2 to FID8, J8 to J10, J9 to J13, J5 to J3, J3 to J4, J4 to J5, R8 to R23, R9 to R24, R10 to R25, R48 to R60, TP2 to TP1, U4 to U2, U2 to U3, U15 to U4, U6 to U8
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Connections:
- C1 pad 2: +3V3 -> GND
- C10 pad 2: +3V3 -> GND
- C11 pad 2: +3V3 -> GND
- C16 pad 1: +3V3 -> /MCU+WIFI+BT/Shield3
- C16 pad 2: +3V3 -> GND
- C17 pad 1: +3V3 -> /MCU+WIFI+BT/VDD_CP
- C17 pad 2: +3V3 -> GND
- C18 pad 1: +3V3 -> /MCU+WIFI+BT/~{RST_CP}
- C18 pad 2: +3V3 -> GND
- C19 pad 2: +3V3 -> GND
- C2 pad 2: +3V3 -> GND
- C20 pad 1: /MCU+WIFI+BT/EN -> +3V3
- C20 pad 2: +3V3 -> GND
- C21 pad 1: /MCU+WIFI+BT/BOOT -> +3V3
- C21 pad 2: +3V3 -> GND
- C22 pad 1: /MCU+WIFI+BT/VDD_CP -> +3V3
- C22 pad 2: +3V3 -> GND
- C23 pad 1: /Audio capture/Shield1 -> /MCU+WIFI+BT/EN
- C23 pad 2: +3V3 -> GND
- C24 pad 2: +3V3 -> GND
- C25 pad 1: /Audio capture/Shield2 -> /MCU+WIFI+BT/BOOT
- C25 pad 2: +3V3 -> GND
- C26 pad 1: Net-(C26-Pad1) -> +3V3
- C26 pad 2: +3V3 -> GND
- C27 pad 1: /MCU+WIFI+BT/GPIO_38 -> Net-(C27-Pad1)
- C27 pad 2: +3V3 -> GND
- C28 pad 1: +3V8 -> Net-(C28-Pad1)
- C28 pad 2: +3V3 -> GND
- C29 pad 1: Net-(C29-Pad1) -> /MCU+WIFI+BT/GPIO_38
- C29 pad 2: +3V3 -> GND
- C3 pad 2: +3V3 -> GND
- C30 pad 1: +3.3VA -> Net-(C30-Pad1)
- C30 pad 2: +3V3 -> GND
- C31 pad 1: +3.3VA -> /Audio capture/Shield1
- C31 pad 2: +3V3 -> GND
- C32 pad 1: +3.3VA -> /Audio capture/Shield2
- C32 pad 2: +3V3 -> GND
- C33 pad 1: +3.3VA -> Net-(C33-Pad1)
- C33 pad 2: +3V3 -> GND
- C34 pad 1: +3.3VA -> +3V8
- C34 pad 2: +3V3 -> GND
- C35 pad 1: 1V8A -> /Audio capture/filtered_3v8
- C35 pad 2: +3V3 -> GND
- C36 pad 1: 1V8A -> +3.3VA
- C36 pad 2: +3V3 -> GND
- C37 pad 1: +3V3 -> 1V8A
- C37 pad 2: +3V3 -> GND
- C38 pad 1: IN_USB_+ -> 1V8A
- C38 pad 2: IN_USB_- -> GND
- C39 pad 1: IN_SOLAR+ -> +3.3VA
- C39 pad 2: IN_SOLAR- -> GND
- C4 pad 2: +3V3 -> GND
- C40 pad 1: IN_SYSTEM- -> +3.3VA
- C40 pad 2: IN_SYSTEM+ -> GND
- C41 pad 1: IN_SYSTEM- -> +3.3VA
- C41 pad 2: +3V3 -> GND
- C42 pad 1: Net-(C42-Pad1) -> +3.3VA
- C42 pad 2: IN_SYSTEM- -> GND
- C43 pad 1: Net-(C43-Pad1) -> +3V3
- C43 pad 2: +3V3 -> GND
- C44 pad 1: +3V3 -> IN_SOLAR+
- C44 pad 2: +3V3 -> IN_SOLAR-
- C45 pad 1: +BATT -> Net-(C45-Pad1)
- C45 pad 2: +3V3 -> VDC
- C46 pad 1: +VDC -> GND
- C46 pad 2: +3V3 -> VDC
- C47 pad 1: +VDC -> VDC
- C47 pad 2: +3V3 -> GND
- C48 pad 1: Net-(C48-Pad1) -> +BATT
- C48 pad 2: +3V3 -> GND
- C49 pad 1: Net-(C49-Pad1) -> +BATT
- C49 pad 2: +3V3 -> GND
- C5 pad 2: +3V3 -> GND
- C50 pad 1: +3V8 -> +BATT
- C50 pad 2: +3V3 -> GND
- C51 pad 1: +3V8 -> Net-(C51-Pad1)
- C51 pad 2: +3V3 -> GND
- C52 pad 1: +3V3 -> Net-(C52-Pad1)
- C52 pad 2: +3V3 -> GND
- C53 pad 1: +3V8 -> +3V3
- C53 pad 2: +3V3 -> GND
- C54 pad 2: +3V3 -> GND
- C55 pad 1: +3V3 -> IN_USB_+
- C55 pad 2: +3V3 -> IN_USB_-
- C56 pad 1: +3V3 -> IN_SYSTEM-
- C56 pad 2: +3V3 -> IN_SYSTEM+
- C57 pad 1: Net-(C57-Pad1) -> IN_SYSTEM+
- C57 pad 2: +3V3 -> GND
- C6 pad 2: +3V3 -> GND
- C7 pad 1: /GSM+GPS/GNSS_RF2 -> /GSM+GPS/GSM_RF1
- C7 pad 2: +3V3 -> GND
- CA1 pad 1: Net-(C24-Pad1) -> Net-(CA1-Pad1)
- CA1 pad 2: Net-(CA1-Pad2) -> Net-(C27-Pad1)
- CA2 pad 2: Net-(CA2-Pad2) -> GND
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Routing:
- added copper zone on B.Cu, net GND
- added copper zone on F.Cu, net GND
Other:
- outline, holes or cut-outs redrawn
