File: Bird_detector_V1/Bird_detector_V1.kicad_pcb (KiCad board)
At the start: 4 copper layers, 126.5 x 76.1 mm, 265 parts, among them IC1 TXB0108PWR, J1 SIM_Card_Shielded, J10 MEM2051, J11 Solar input, J12 140-502-415-000, J13 USB_A, J14 batt input, J2 GSM, J3 USB_A, J4 BT, J5 GNSS, J6 USB1046-GF-0190-L-B-A, J7 Screw_Terminal_01x03, J8 292132-3, J9 292132-3, Q1 SSM6N7002, Q10 SSM6N7002, Q11 DMP3028LSD, Q2 SSM6N7002, Q3 SSM6N7002, Q4 SSM6N7002, Q5 SSM6N7002, Q6 BC847BS, Q7 DMP3028LSD, Q8 DMP3028LSD, Q9 DMP3028LSD, SW1 SW_SPST, SW2 MCU_RESET, U1 SIM808, U10 MIC5317, U11 MIC5317, U12 CN3791, U13 MAX11601, U14 INA3221, U15 APX810S05, U16 TPS63020DSJR, U17 TPS63020DSJR, U2 CP2102N-Axx-xQFN24, U3 ESP32-S3-WROOM-1, U4 MCP2561-H-SN, U5 BME280, U6 74LVC1G08, U7 TLV9161IDBVR, U8 TLV320ADC3100, U9 TLV9161IDBVR, Y1 SiT1602BI-13-33E-12.000000G

Commit message: v
Parts:
- removed C16, C31, C32: 4p7-10p, Capacitor_SMD:C_0603_1608Metric_Pad1.08x0.95mm_HandSolder
- removed FID10, FID4, FID5, FID9: Cell, Z_mycustom_footprint_lib:18650 cell 3d model
- added C67: 1u, Capacitor_SMD:C_0603_1608Metric_Pad1.08x0.95mm_HandSolder, B.Cu at (183.5, 95.9)
- added J15: 2x10, SamacSys_Parts:TSM-110-ZZ-YYY-DH, B.Cu at (190.1, 92.8)
- added J16: PCB CAP, Z_mycustom_footprint_lib:PCB cap start, F.Cu at (139.3, 69.8)
- added J17: PCB CAP, Z_mycustom_footprint_lib:PCB cap start, F.Cu at (184.4, 120.7)
- added JP7: ADR1, Jumper:SolderJumper-3_P1.3mm_Bridged12_RoundedPad1.0x1.5mm_NumberLabels, B.Cu at (179.1, 101.1)
- added JP8: ADR0, Jumper:SolderJumper-3_P1.3mm_Bridged12_RoundedPad1.0x1.5mm_NumberLabels, B.Cu at (178.8, 95.9)
- added JP9: ADR0, Jumper:SolderJumper-3_P1.3mm_Bridged12_RoundedPad1.0x1.5mm_NumberLabels, B.Cu at (180.1, 98.5)
- added U18: TCA9535PWR, Package_SO:TSSOP-24_4.4x7.8mm_P0.65mm, B.Cu at (180.5, 89.9)
- C34, C35, C36, C37, C38, C40, C48, C56, D12, D17, F2, JP2, L2, L3, Q1, Q2, Q3, Q4, Q5, Q7, Q9, R10, R12, R13, R19, R21, R31, R32, R49, R67, R68, R8, R9, TH2, U10, U12, U14, U15, U16, U17, U6, Y1: moved to B.Cu
- FID2: value kicad -> KiCAD
- FID8: value scale -> Scale
- J12: value 140-502-415-000 -> PCB CAP; footprint SamacSys_Parts:140502415000 -> Z_mycustom_footprint_lib:PCB cap start; moved to F.Cu
- J13: footprint Connector_USB:USB_A_Molex_105057_Vertical -> SamacSys_Parts:USB1040GFLB
- J3: footprint Connector_USB:USB_A_Molex_105057_Vertical -> Connector_PinHeader_2.54mm:PinHeader_1x04_P2.54mm_Vertical
- moved C65 249.8 mm to (112.4, 80.7), turned to 90 degrees
- moved C66 244.7 mm to (115.7, 88.0)
- moved C63 242.6 mm to (115.1, 82.4)
- moved C64 241.8 mm to (110.8, 84.0), turned to -90 degrees
- moved R91 240.7 mm to (115.7, 89.7)
- moved C61 238.8 mm to (122.6, 88.3), turned to 180 degrees
- moved L3 237.2 mm to (116.0, 80.1), turned to 180 degrees
- moved C62 236.7 mm to (117.4, 84.3), turned to 180 degrees
- moved R90 235.6 mm to (112.4, 84.1), turned to -90 degrees
- moved R89 234.1 mm to (114.0, 85.6), turned to -90 degrees
- moved C60 232.8 mm to (128.0, 85.6)
- moved R86 232.7 mm to (124.4, 80.6), turned to 180 degrees
- moved C57 231.0 mm to (125.2, 86.6), turned to 90 degrees
- moved JP6 230.9 mm to (118.6, 86.8), turned to 90 degrees
- moved C58 229.4 mm to (128.0, 84.0)
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Connections:
- net /MCU+WIFI+BT/PG_3V3 renamed /Power Management +BMS/SMPSs/PG_3V3
- net /MCU+WIFI+BT/PG_3V8 renamed /Power Management +BMS/SMPSs/PG_3V8
- net /MCU+WIFI+BT/Shield3 renamed /Other data+storage/Shield3
- net Net-(C28-Pad1) renamed /Audio capture/LEFT_IN_AMP
- net Net-(C33-Pad1) renamed /Audio capture/RIGHT_IN_AMP
- net Net-(C52-Pad1) renamed /Power Management +BMS/COM_CAP
- net Net-(C61-Pad1) renamed /Power Management +BMS/SMPSs/EN_3V3
- net Net-(C66-Pad1) renamed /Power Management +BMS/SMPSs/EN_3V8
- net Net-(D11-Pad1) renamed /Power Management +BMS/BMS_SW_OUT
- net Net-(L1-Pad2) renamed /Power Management +BMS/CSP
- net Net-(R46-Pad1) renamed /Audio capture/12MHz_enable
- net Net-(R49-Pad1) renamed /Audio capture/12MHz_raw
- net Net-(R69-Pad2) renamed /Power Management +BMS/MPPT
- net Net-(R70-Pad2) renamed /Power Management +BMS/COM
- net Net-(R85-Pad2) renamed /Power Management +BMS/SMPSs/FB_3V3
- net Net-(R89-Pad2) renamed /Power Management +BMS/SMPSs/FB_3V8
- net USB_OTG_D+ renamed /MCU+WIFI+BT/USB_OTG_D+
- net USB_OTG_D- renamed /MCU+WIFI+BT/USB_OTG_D-
- J12 pad 1: GND -> /Audio capture/Shield1
- Q2 pad 1: /MCU+WIFI+BT/GPIO_36 -> /MCU+WIFI+BT/GPIO_35
- R35 pad 1: /MCU+WIFI+BT/GPIO_36 -> /MCU+WIFI+BT/GPIO_35
- U13 pad 6: /MCU+WIFI+BT/GPIO_36 -> /MCU+WIFI+BT/GPIO_35
- U14 pad 7: /MCU+WIFI+BT/GPIO_36 -> /MCU+WIFI+BT/GPIO_35
- U3 pad 29: /MCU+WIFI+BT/GPIO_36 -> /MCU+WIFI+BT/GPIO_35
- U5 pad 3: /MCU+WIFI+BT/GPIO_36 -> /MCU+WIFI+BT/GPIO_35
- U8 pad 18: /MCU+WIFI+BT/GPIO_36 -> /MCU+WIFI+BT/GPIO_35
Routing:
- net /Other data+storage/Shield3: track 0.00 -> 5.61 mm
- net /Audio capture/Shield1: track 0.00 -> 5.35 mm
- net /Audio capture/Shield2: track 0.00 -> 5.20 mm
- net +3V3: vias 2 -> 0
- added copper zone on F.Cu, net /Audio capture/Shield1
- added copper zone on F.Cu, net /Audio capture/Shield2
- added copper zone on F.Cu, net /Other data+storage/Shield3
Other:
- outline, holes or cut-outs redrawn

Commit message: f
Parts:
- removed C6: 33p, Capacitor_SMD:C_0603_1608Metric_Pad1.08x0.95mm_HandSolder
- removed CA1, CA6: 10n?, Capacitor_SMD:C_0603_1608Metric_Pad1.08x0.95mm_HandSolder
- removed CA2, CA3, CA4, CA5: 1u, Capacitor_SMD:C_0603_1608Metric_Pad1.08x0.95mm_HandSolder
- added C16: 100n, Capacitor_SMD:C_0603_1608Metric_Pad1.08x0.95mm_HandSolder, F.Cu at (267.6, 131.3)
- added C31: 100n, Capacitor_SMD:C_0603_1608Metric_Pad1.08x0.95mm_HandSolder, F.Cu at (271.9, 131.3)
- added C32: DNP, Capacitor_SMD:C_0603_1608Metric_Pad1.08x0.95mm_HandSolder, F.Cu at (266.3, 88.0)
- added C68: 15n, Capacitor_SMD:C_0603_1608Metric_Pad1.08x0.95mm_HandSolder, F.Cu at (252.1, 90.5)
- added C69: 1u, Capacitor_SMD:C_0603_1608Metric_Pad1.08x0.95mm_HandSolder, F.Cu at (256.5, 88.0)
- added C70: 1u, Capacitor_SMD:C_0603_1608Metric_Pad1.08x0.95mm_HandSolder, F.Cu at (247.8, 93.0)
- added C71: 1u, Capacitor_SMD:C_0603_1608Metric_Pad1.08x0.95mm_HandSolder, F.Cu at (252.1, 88.0)
- added C72: 1u, Capacitor_SMD:C_0603_1608Metric_Pad1.08x0.95mm_HandSolder, F.Cu at (247.8, 90.5)
- added C73: 15n, Capacitor_SMD:C_0603_1608Metric_Pad1.08x0.95mm_HandSolder, F.Cu at (247.8, 88.0)
- added C74: 15n, Capacitor_SMD:C_0603_1608Metric_Pad1.08x0.95mm_HandSolder, F.Cu at (258.1, 75.1)
- added C75: 4.7n, Capacitor_SMD:C_0603_1608Metric_Pad1.08x0.95mm_HandSolder, F.Cu at (270.5, 80.5)
- added D19: LED_Small, LED_SMD:LED_0603_1608Metric_Pad1.05x0.95mm_HandSolder, F.Cu at (259.3, 140.2)
- added R96: 10k, Resistor_SMD:R_0603_1608Metric_Pad0.98x0.95mm_HandSolder, F.Cu at (276.3, 131.3)
- added R97: 10k, Resistor_SMD:R_0603_1608Metric_Pad0.98x0.95mm_HandSolder, F.Cu at (280.6, 131.3)
- added R98: 300, Resistor_SMD:R_0603_1608Metric_Pad0.98x0.95mm_HandSolder, F.Cu at (263.7, 140.2)
- added R99: 100k, Resistor_SMD:R_0603_1608Metric_Pad0.98x0.95mm_HandSolder, F.Cu at (270.5, 86.5)
- added TP3: TestPoint, TestPoint:TestPoint_Pad_1.5x1.5mm, F.Cu at (187.3, 112.9)
- added TP4: TestPoint, TestPoint:TestPoint_Pad_1.5x1.5mm, F.Cu at (187.3, 110.4)
- added U19: TLV9161IDBVR, Package_SO:SOIC-8_3.9x4.9mm_P1.27mm, F.Cu at (269.6, 126.8)
- added U20: TLV9161IDBVR, Package_SO:SOIC-8_3.9x4.9mm_P1.27mm, F.Cu at (278.1, 126.8)
- C17, C18, C19, R16, R26, R28, R29: moved to B.Cu
- C23: value z -> 15n
- C27, C28, C30, C33: value 15n -> 100n
- C51: value 3.5n -> 15n
- D6: value z -> 5v1
- R1, R10, R14, R19, R2, R21, R44, R45, R49, R53, R54, R8, R9, R94: value 100 -> 60
- R12, R13: moved to F.Cu
- R15: value 100 -> 60; moved to B.Cu
- R17, R31, R32, R5, R6, R68, R7: value X -> 300
- R30: value 10K -> 10k
- R33: value y -> 60
- R63: value 45 -> 60
- R70: value 120 -> 60
- R76, R77, R79, R80: value 50k+ -> 64k
- R92: value 200k -> 100k
- U13: footprint Package_TO_SOT_SMD:SOT-23-8_Handsoldering -> Package_TO_SOT_SMD:SOT-23-8
- moved R29 115.6 mm to (136.1, 120.7), turned to 180 degrees
- moved R28 111.4 mm to (136.1, 119.1)
- moved R26 110.8 mm to (141.2, 120.4), turned to -90 degrees
- moved C17 110.7 mm to (140.6, 117.2)
- moved C18 107.6 mm to (139.7, 121.8), turned to -90 degrees
- moved R16 101.9 mm to (153.8, 125.2), turned to 180 degrees
- moved R33 100.9 mm to (258.1, 77.6), turned to 0 degrees
- moved C20 96.3 mm to (167.4, 128.1), turned to -90 degrees
- moved R15 88.6 mm to (153.8, 123.7)
- moved C19 80.7 mm to (163.6, 126.1)
- moved C21 80.3 mm to (165.9, 128.1), turned to -90 degrees
- moved Q4 23.7 mm to (186.9, 110.6)
- moved C43 7.08 mm to (210.6, 106.0)
- moved U6 5.71 mm to (150.1, 124.7)
- moved C7 5.24 mm to (175.9, 79.1), turned to -135 degrees
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Connections:
- C51 pad 2: GND -> Net-(C51-Pad2)
- JP3 pad 1: +3.3VA -> GND
- JP3 pad 3: GND -> +3.3VA
- JP4 pad 1: +3.3VA -> GND
- JP4 pad 3: GND -> +3.3VA
- JP7 pad 1: +3V3 -> GND
- JP7 pad 3: GND -> +3V3
- JP8 pad 1: +3V3 -> GND
- JP8 pad 3: GND -> +3V3
- JP9 pad 1: +3V3 -> GND
- JP9 pad 3: GND -> +3V3
- R33 pad 1: /MCU+WIFI+BT/EN -> /Power Management +BMS/COM
- R33 pad 2: /Power Management +BMS/SMPSs/PG_3V3 -> Net-(R33-Pad2)
- R70 pad 1: /Power Management +BMS/COM_CAP -> Net-(R33-Pad2)
- R70 pad 2: /Power Management +BMS/COM -> /Power Management +BMS/COM_CAP
- R76 pad 1: Net-(R76-Pad1) -> /Power Management +BMS/Temp1
- R77 pad 1: Net-(R77-Pad1) -> /Power Management +BMS/Temp2
- R79 pad 2: /Power Management +BMS/Temp1 -> Net-(R79-Pad2)
- R80 pad 2: /Power Management +BMS/Temp2 -> Net-(R80-Pad2)
- R87 pad 2: /Power Management +BMS/SMPSs/PG_3V3 -> /MCU+WIFI+BT/EN
- R92 pad 2: GND -> Net-(R92-Pad2)
- TH1 pad 1: Net-(R76-Pad1) -> /Power Management +BMS/Temp1
- TH1 pad 2: /Power Management +BMS/Temp1 -> Net-(R79-Pad2)
- TH2 pad 1: Net-(R77-Pad1) -> /Power Management +BMS/Temp2
- TH2 pad 2: /Power Management +BMS/Temp2 -> Net-(R80-Pad2)
- U13 pad 1: /Power Management +BMS/Temp1 -> /Power Management +BMS/Temp1_out
- U13 pad 2: /Power Management +BMS/Temp2 -> /Power Management +BMS/Temp2_out
- U13 pad 3: unconnected-(U13-Pad3) -> Net-(TP3-Pad1)
- U13 pad 4: unconnected-(U13-Pad4) -> Net-(TP4-Pad1)
- U16 pad 14: /Power Management +BMS/SMPSs/PG_3V3 -> /MCU+WIFI+BT/EN
- U8 pad 25: (no net) -> GND
Routing:
- net VBUS: track 0.00 -> 56.2 mm
- net /Power Management +BMS/Heater_Input: track 0.00 -> 37.3 mm
- net Net-(F1-Pad1): track 0.00 -> 18.9 mm
- net +3V3: track 0.00 -> 18.5 mm, vias 0 -> 1
- net /MCU+WIFI+BT/USB_OTG_D+: track 0.00 -> 18.4 mm, vias 0 -> 1
- net /MCU+WIFI+BT/USB_OTG_D-: track 0.00 -> 16.9 mm, vias 0 -> 1
- net IN_USB_-: track 0.00 -> 15.0 mm, vias 0 -> 1
- net /MCU+WIFI+BT/VIO: track 0.00 -> 14.4 mm, vias 0 -> 2
- net D+: track 0.00 -> 14.1 mm, vias 0 -> 1
- net +BATT: track 0.00 -> 13.8 mm, vias 0 -> 1
- net D-: track 0.00 -> 12.5 mm, vias 0 -> 1
- net /GSM+GPS/GSM_RF2: track 0.00 -> 10.1 mm
- net /GSM+GPS/GNSS_RF2: track 0.00 -> 9.89 mm
- net /GSM+GPS/GNSS_RF1: track 0.00 -> 9.38 mm
- net /MCU+WIFI+BT/BASE2: track 0.00 -> 9.36 mm, vias 0 -> 2
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