File: Bird_detector_V1/SMPSs.kicad_sch (KiCad schematic)
At the start: 22 parts

Commit message: f
Parts:
- removed C?: 22u, Capacitor_SMD:C_0603_1608Metric_Pad1.08x0.95mm_HandSolder, symbol Device:C_Small
- removed L?: 1-1.5u, symbol Device:L
- removed R? (x2): 100k, Resistor_SMD:R_0603_1608Metric_Pad0.98x0.95mm_HandSolder, symbol Device:R_Small
- added C35: 22u, Capacitor_SMD:C_0603_1608Metric_Pad1.08x0.95mm_HandSolder, symbol Device:C_Small
- added C39, C44: 100n, Capacitor_SMD:C_0603_1608Metric_Pad1.08x0.95mm_HandSolder, symbol Device:C_Small
- added JP5: safe, Jumper:SolderJumper-2_P1.3mm_Open_RoundedPad1.0x1.5mm, symbol Jumper:Jumper_2_Open
- added L2: 1.5u, symbol Device:L
- added R44, R50: DNP, Resistor_SMD:R_0603_1608Metric_Pad0.98x0.95mm_HandSolder, symbol Device:R_Small
- L3: renamed from L?; value 1-1.5u -> 1.5u
- gave numbers to parts that had none: 17
Connections:
- net +3V3: now also R43.1, R44.1
- net +3V8: now also R49.1, R50.1
- net DC: now also C40.1, C35.1; no longer U10.1 (VINA), U10.12 (EN), U9.1 (VINA), U9.12 (EN)
- net GND: now also C40.2, R46.2, R52.2, C35.2, C39.2, C44.2
- net RF_SYNC: now also JP5.1 (A); no longer U9.13 (PS/SYNC)
- net at R52.1: now also R49.2, U10.3 (FB), R50.2
- net at R46.1: now also R43.2, U9.3 (FB), R44.2
- net at U9.8 (L1), U9.9 (L1): now also L2.1
- net at U9.6 (L2), U9.7 (L2): now also L2.2
- new net: C44.1, JP5.2 (B), U10.1 (VINA), U10.12 (EN)
- new net: C39.1, U9.1 (VINA), U9.12 (EN), U9.13 (PS/SYNC)
Other:
- moved on the sheet: C36, C37, C38, C40, C41, C42, C43, R43, R45, R46, R47, R48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

Commit message: R
Parts:
- L2, L3: footprint (none) -> Inductor_SMD:L_Wuerth_MAPI-3012
- renumbered R43 to R44, R44 to R45, R45 to R46, R46 to R47, R47 to R48, R48 to R49, R49 to R50, R50 to R51, R51 to R52, R52 to R53
Changed lines of the file:
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@@
   (symbol (lib_id "Device:R_Small") (at 146.685 212.725 0) (unit 1)
     (in_bom yes) (on_board yes) (fields_autoplaced)
-    (property "Reference" "R52" (id 0) (at 149.225 211.4549 0)
+    (property "Reference" "R53" (id 0) (at 149.225 211.4549 0)
       (effects (font (size 1.27 1.27)) (justify left))
     )
@@
   (symbol (lib_id "Device:R_Small") (at 150.495 103.505 0) (unit 1)
     (in_bom yes) (on_board yes) (fields_autoplaced)
-    (property "Reference" "R46" (id 0) (at 153.035 102.2349 0)
+    (property "Reference" "R47" (id 0) (at 153.035 102.2349 0)
       (effects (font (size 1.27 1.27)) (justify left))
     )
@@
   (symbol (lib_id "power:+3V3") (at 213.995 90.17 0) (unit 1)
     (in_bom yes) (on_board yes) (fields_autoplaced)
-    (property "Reference" "#PWR0115" (id 0) (at 213.995 93.98 0)
+    (property "Reference" "#PWR0118" (id 0) (at 213.995 93.98 0)
       (effects (font (size 1.27 1.27)) hide)
     )
@@
   (symbol (lib_id "power:GND") (at 95.25 120.65 0) (unit 1)
     (in_bom yes) (on_board yes) (fields_autoplaced)
-    (property "Reference" "#PWR0118" (id 0) (at 95.25 127 0)
+    (property "Reference" "#PWR0121" (id 0) (at 95.25 127 0)
       (effects (font (size 1.27 1.27)) hide)
     )
@@
   (symbol (lib_id "Device:R_Small") (at 158.75 203.2 0) (unit 1)
     (in_bom yes) (on_board yes) (fields_autoplaced)
-    (property "Reference" "R50" (id 0) (at 161.29 201.9299 0)
+    (property "Reference" "R51" (id 0) (at 161.29 201.9299 0)
       (effects (font (size 1.27 1.27)) (justify left))
     )
@@
     (pin "2")
   )
-  (symbol (lib_id "Device:L") (at 129.54 78.74 90) (unit 1)
-    (in_bom yes) (on_board yes) (fields_autoplaced)
-    (property "Reference" "L2" (id 0) (at 129.54 72.39 90))
-    (property "Value" "1.5u" (id 1) (at 129.54 74.93 90))
-    (property "Footprint" "" (id 2) (at 129.54 78.74 0)
-      (effects (font (size 1.27 1.27)) hide)
-    )
-    (property "Datasheet" "~" (id 3) (at 129.54 78.74 0)
-      (effects (font (size 1.27 1.27)) hide)
-    )
-    (pin "1")
-    (pin "2")
-  )
   (symbol (lib_id "Device:R_Small") (at 200.66 100.33 0) (unit 1)
     (in_bom yes) (on_board yes) (fields_autoplaced)
-    (property "Reference" "R45" (id 0) (at 203.2 99.0599 0)
+    (property "Reference" "R46" (id 0) (at 203.2 99.0599 0)
       (effects (font (size 1.27 1.27)) (justify left))
     )
@@
   (symbol (lib_id "power:GND") (at 132.08 120.65 0) (unit 1)
     (in_bom yes) (on_board yes) (fields_autoplaced)
-    (property "Reference" "#PWR0119" (id 0) (at 132.08 127 0)
+    (property "Reference" "#PWR0122" (id 0) (at 132.08 127 0)
       (effects (font (size 1.27 1.27)) hide)
     )
@@
   (symbol (lib_id "Device:R_Small") (at 154.305 180.975 0) (unit 1)
     (in_bom yes) (on_board yes) (fields_autoplaced)
-    (property "Reference" "R47" (id 0) (at 156.845 179.7049 0)
+    (property "Reference" "R48" (id 0) (at 156.845 179.7049 0)
       (effects (font (size 1.27 1.27)) (justify left))
     )
@@
   (symbol (lib_id "power:GND") (at 74.93 214.63 0) (unit 1)
     (in_bom yes) (on_board yes) (fields_autoplaced)
-    (property "Reference" "#PWR0121" (id 0) (at 74.93 220.98 0)
+    (property "Reference" "#PWR0124" (id 0) (at 74.93 220.98 0)
       (effects (font (size 1.27 1.27)) hide)
     )
@@
   (symbol (lib_id "Device:R_Small") (at 146.685 203.2 0) (unit 1)
     (in_bom yes) (on_board yes) (fields_autoplaced)
-    (property "Reference" "R49" (id 0) (at 149.225 201.9299 0)
+    (property "Reference" "R50" (id 0) (at 149.225 201.9299 0)
       (effects (font (size 1.27 1.27)) (justify left))
     )
@@
   (symbol (lib_id "Device:R_Small") (at 150.495 93.98 0) (unit 1)
     (in_bom yes) (on_board yes) (fields_autoplaced)
-    (property "Reference" "R43" (id 0) (at 153.035 92.7099 0)
+    (property "Reference" "R44" (id 0) (at 153.035 92.7099 0)
       (effects (font (size 1.27 1.27)) (justify left))
     )
@@
   (symbol (lib_id "power:GND") (at 91.44 229.87 0) (unit 1)
     (in_bom yes) (on_board yes) (fields_autoplaced)
-    (property "Reference" "#PWR0123" (id 0) (at 91.44 236.22 0)
+    (property "Reference" "#PWR0126" (id 0) (at 91.44 236.22 0)
       (effects (font (size 1.27 1.27)) hide)
     )
@@
   (symbol (lib_id "power:GND") (at 150.495 107.315 0) (unit 1)
     (in_bom yes) (on_board yes) (fields_autoplaced)
-    (property "Reference" "#PWR0117" (id 0) (at 150.495 113.665 0)
+    (property "Reference" "#PWR0120" (id 0) (at 150.495 113.665 0)
       (effects (font (size 1.27 1.27)) hide)
     )
@@
   (symbol (lib_id "power:+3V8") (at 186.055 199.39 0) (unit 1)
     (in_bom yes) (on_board yes) (fields_autoplaced)
-    (property "Reference" "#PWR0120" (id 0) (at 186.055 203.2 0)
+    (property "Reference" "#PWR0123" (id 0) (at 186.055 203.2 0)
       (effects (font (size 1.27 1.27)) hide)
     )
@@
     (pin "1")
   )
+  (symbol (lib_id "Device:L") (at 129.54 78.74 90) (unit 1)
+    (in_bom yes) (on_board yes) (fields_autoplaced)
+    (property "Reference" "L2" (id 0) (at 129.54 72.39 90))
+    (property "Value" "1.5u" (id 1) (at 129.54 74.93 90))
+    (property "Footprint" "Inductor_SMD:L_Wuerth_MAPI-3012" (id 2) (at 129.54 78.74 0)
+      (effects (font (size 1.27 1.27)) hide)
+    )
+    (property "Datasheet" "~" (id 3) (at 129.54 78.74 0)
+      (effects (font (size 1.27 1.27)) hide)
+    )
+    (pin "1")
+    (pin "2")
+  )
   (symbol (lib_id "Device:R_Small") (at 154.305 188.595 0) (unit 1)
     (in_bom yes) (on_board yes) (fields_autoplaced)
-    (property "Reference" "R48" (id 0) (at 156.845 187.3249 0)
+    (property "Reference" "R49" (id 0) (at 156.845 187.3249 0)
       (effects (font (size 1.27 1.27)) (justify left))
     )
@@
   (symbol (lib_id "Device:R_Small") (at 161.925 93.98 0) (unit 1)
     (in_bom yes) (on_board yes) (fields_autoplaced)
-    (property "Reference" "R44" (id 0) (at 163.83 92.7099 0)
+    (property "Reference" "R45" (id 0) (at 163.83 92.7099 0)
       (effects (font (size 1.27 1.27)) (justify left))
     )
@@
     (property "Reference" "L3" (id 0) (at 125.73 181.61 90))
     (property "Value" "1.5u" (id 1) (at 125.73 184.15 90))
-    (property "Footprint" "" (id 2) (at 125.73 187.96 0)
+    (property "Footprint" "Inductor_SMD:L_Wuerth_MAPI-3012" (id 2) (at 125.73 187.96 0)
       (effects (font (size 1.27 1.27)) hide)
     )
@@
   (symbol (lib_id "power:GND") (at 128.27 229.87 0) (unit 1)
     (in_bom yes) (on_board yes) (fields_autoplaced)
-    (property "Reference" "#PWR0124" (id 0) (at 128.27 236.22 0)
+    (property "Reference" "#PWR0127" (id 0) (at 128.27 236.22 0)
       (effects (font (size 1.27 1.27)) hide)
     )
@@
   (symbol (lib_id "power:GND") (at 77.47 105.41 0) (unit 1)
     (in_bom yes) (on_board yes) (fields_autoplaced)
-    (property "Reference" "#PWR0116" (id 0) (at 77.47 111.76 0)
+    (property "Reference" "#PWR0119" (id 0) (at 77.47 111.76 0)
       (effects (font (size 1.27 1.27)) hide)
     )
@@
   (symbol (lib_id "Device:R_Small") (at 179.705 209.55 0) (unit 1)
     (in_bom yes) (on_board yes) (fields_autoplaced)
-    (property "Reference" "R51" (id 0) (at 182.245 208.2799 0)
+    (property "Reference" "R52" (id 0) (at 182.245 208.2799 0)
       (effects (font (size 1.27 1.27)) (justify left))
     )
@@
   (symbol (lib_id "power:GND") (at 146.685 216.535 0) (unit 1)
     (in_bom yes) (on_board yes) (fields_autoplaced)
-    (property "Reference" "#PWR0122" (id 0) (at 146.685 222.885 0)
-      (effects (font (size 1.27 1.27)) hide)
-    )
+    (property "Reference" "#PWR0125" (id 0) (at 146.685 222.885 0)
+      (effects (font (size 1.27 1.27)) hide)
+    )

Commit message: v
Parts:
- renumbered C35 to C46, C36 to C47, C37 to C48, C38 to C49, C39 to C50, C40 to C51, C41 to C52, C42 to C53, C43 to C54, C44 to C55, JP5 to JP7, R44 to R63, R45 to R64, R46 to R65, R47 to R66, R48 to R67, R49 to R68, R50 to R69, R51 to R70, R52 to R71, R53 to R72, U9 to U11, U10 to U12
Connections:
- net +3V3: now also C47.1, C48.1, C49.1
- net +3V8: now also C52.1, C53.1, C54.1
- net GND: now also C47.2, C48.2, C49.2, C52.2, C53.2, C54.2
Other:
- moved on the sheet: C47, C48, C49, C52, C53, C54

Commit message: f
Parts:
- renumbered C51 to C46, C46 to C47, C55 to C48, C50 to C49, C52 to C50, C53 to C51, C47 to C52, C54 to C53, C48 to C54, C49 to C55, L3 to L2, L2 to L3, R69 to R62, R72 to R63, R63 to R64, R66 to R65, R67 to R66, R68 to R67, R70 to R68, R64 to R69, R71 to R70, R65 to R71, U11 to U13
Connections:
- net PG_3V3: now reaches R71.2, U13.14 (PG)
- net PG_3V8: now reaches R70.2, U12.14 (PG)
Other:
- moved on the sheet: JP7, R62, R63, R64, R65, R66, R67, R69, R70, R71

Commit message: v
Parts:
- removed R66: 1.18Meg, Resistor_SMD:R_0603_1608Metric_Pad0.98x0.95mm_HandSolder, symbol Device:R_Small
- removed R67: 180k, Resistor_SMD:R_0603_1608Metric_Pad0.98x0.95mm_HandSolder, symbol Device:R_Small
- renumbered C47 to C57, C52 to C58, C54 to C59, C55 to C60, C49 to C61, C46 to C62, C50 to C63, C51 to C64, C53 to C65, C48 to C66, JP7 to JP6, L3 to L2, L2 to L3, R64 to R85, R69 to R86, R71 to R87, R65 to R88, R62 to R89, R68 to R90, R70 to R91, R63 to R92, U13 to U16, U12 to U17

Commit message: v
Connections:
- net FB_3V8: now reaches R89.2, R90.2, R92.1, U17.3 (FB)
- net FB_3V3: now reaches R85.2, R86.2, R88.1, U16.3 (FB)
- net EN_3V8: now reaches C66.1, JP6.2 (B), U17.1 (VINA), U17.12 (EN)
- net EN_3V3: now reaches C61.1, U16.1 (VINA), U16.12 (EN), U16.13 (PS/SYNC)
Changed lines of the file:
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@@
     (effects (font (size 4 4)) (justify right bottom))
+  )
+  (label "FB_3V8" (at 158.75 208.28 0)
+    (effects (font (size 1.27 1.27)) (justify left bottom))
+  )
+  (label "PG_3V3" (at 170.18 110.49 0)
+    (effects (font (size 1.27 1.27)) (justify left bottom))
+  )
+  (label "EN_3V3" (at 99.06 97.79 0)
+    (effects (font (size 1.27 1.27)) (justify left bottom))
+  )
+  (label "PG_3V8" (at 160.02 219.71 0)
+    (effects (font (size 1.27 1.27)) (justify left bottom))
+  )
+  (label "EN_3V8" (at 95.25 207.01 0)
+    (effects (font (size 1.27 1.27)) (justify left bottom))
+  )
+  (label "DC_IN" (at 88.9 199.39 0)
+    (effects (font (size 1.27 1.27)) (justify left bottom))
+  )
+  (label "FB_3V3" (at 162.56 99.06 0)
+    (effects (font (size 1.27 1.27)) (justify left bottom))
   )
   (hierarchical_label "DC" (shape input) (at 66.04 199.39 180)

Commit message: f
Parts:
- added R99: 100k, Resistor_SMD:R_0603_1608Metric_Pad0.98x0.95mm_HandSolder, symbol Device:R_Small
- R92: value 200k -> 100k
Connections:
- net GND: now also R99.2; no longer R92.2
- new net: R92.2, R99.1
Other:
- moved on the sheet: R92
Changed lines of the file:
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@@
+    (stroke (width 0) (type default) (color 0 0 0 0))
+  )
+  (wire (pts (xy 147.32 217.17) (xy 147.32 222.25))
     (stroke (width 0) (type default) (color 0 0 0 0))
   )
@@
     (stroke (width 0) (type default) (color 0 0 0 0))
   )
-  (wire (pts (xy 151.13 106.68) (xy 151.13 107.95))
-    (stroke (width 0) (type default) (color 0 0 0 0))
-  )
   (wire (pts (xy 158.75 208.28) (xy 147.32 208.28))
     (stroke (width 0) (type default) (color 0 0 0 0))
@@
     (stroke (width 0) (type default) (color 0 0 0 0))
   )
-  (wire (pts (xy 147.32 209.55) (xy 147.32 210.82))
+  (wire (pts (xy 147.32 209.55) (xy 147.32 212.09))
     (stroke (width 0) (type default) (color 0 0 0 0))
   )
@@
     (stroke (width 0) (type default) (color 0 0 0 0))
   )
+  (wire (pts (xy 151.13 107.95) (xy 151.13 106.68))
+    (stroke (width 0) (type default) (color 0 0 0 0))
+  )
   (wire (pts (xy 114.3 90.17) (xy 116.84 90.17))
     (stroke (width 0) (type default) (color 0 0 0 0))
@@
     (stroke (width 0) (type default) (color 0 0 0 0))
   )
-  (wire (pts (xy 147.32 215.9) (xy 147.32 217.17))
+  (wire (pts (xy 147.32 227.33) (xy 147.32 229.87))
     (stroke (width 0) (type default) (color 0 0 0 0))
   )
@@
     (effects (font (size 1.27 1.27)) (justify left bottom))
   )
+  (label "DC_IN" (at 87.63 90.17 0)
+    (effects (font (size 1.27 1.27)) (justify left bottom))
+  )
   (label "FB_3V3" (at 162.56 99.06 0)
     (effects (font (size 1.27 1.27)) (justify left bottom))
@@
     (effects (font (size 1.27 1.27)) (justify left))
   )
-  (symbol (lib_id "Device:R_Small") (at 147.32 213.36 0) (unit 1)
-    (in_bom yes) (on_board yes) (fields_autoplaced)
-    (property "Reference" "R92" (id 0) (at 149.86 212.0899 0)
-      (effects (font (size 1.27 1.27)) (justify left))
-    )
-    (property "Value" "200k" (id 1) (at 149.86 214.6299 0)
-      (effects (font (size 1.27 1.27)) (justify left))
-    )
-    (property "Footprint" "Resistor_SMD:R_0603_1608Metric_Pad0.98x0.95mm_HandSolder" (id 2) (at 147.32 213.36 0)
-      (effects (font (size 1.27 1.27)) hide)
-    )
-    (property "Datasheet" "~" (id 3) (at 147.32 213.36 0)
+  (symbol (lib_id "Device:R_Small") (at 147.32 214.63 0) (unit 1)
+    (in_bom yes) (on_board yes) (fields_autoplaced)
+    (property "Reference" "R92" (id 0) (at 149.86 213.3599 0)
+      (effects (font (size 1.27 1.27)) (justify left))
+    )
+    (property "Value" "100k" (id 1) (at 149.86 215.8999 0)
+      (effects (font (size 1.27 1.27)) (justify left))
+    )
+    (property "Footprint" "Resistor_SMD:R_0603_1608Metric_Pad0.98x0.95mm_HandSolder" (id 2) (at 147.32 214.63 0)
+      (effects (font (size 1.27 1.27)) hide)
+    )
+    (property "Datasheet" "~" (id 3) (at 147.32 214.63 0)
       (effects (font (size 1.27 1.27)) hide)
     )
@@
     (pin "2")
   )
+  (symbol (lib_id "power:GND") (at 151.13 107.95 0) (unit 1)
+    (in_bom yes) (on_board yes) (fields_autoplaced)
+    (property "Reference" "#PWR0178" (id 0) (at 151.13 114.3 0)
+      (effects (font (size 1.27 1.27)) hide)
+    )
+    (property "Value" "GND" (id 1) (at 151.13 113.03 0)
+      (effects (font (size 1.27 1.27)) hide)
+    )
+    (property "Footprint" "" (id 2) (at 151.13 107.95 0)
+      (effects (font (size 1.27 1.27)) hide)
+    )
+    (property "Datasheet" "" (id 3) (at 151.13 107.95 0)
+      (effects (font (size 1.27 1.27)) hide)
+    )
+    (pin "1")
+  )
   (symbol (lib_id "Device:R_Small") (at 190.5 100.33 0) (unit 1)
     (in_bom yes) (on_board yes) (fields_autoplaced)
@@
     (pin "1")
     (pin "2")
-  )
-  (symbol (lib_id "power:GND") (at 151.13 107.95 0) (unit 1)
-    (in_bom yes) (on_board yes) (fields_autoplaced)
-    (property "Reference" "#PWR0178" (id 0) (at 151.13 114.3 0)
-      (effects (font (size 1.27 1.27)) hide)
-    )
-    (property "Value" "GND" (id 1) (at 151.13 113.03 0)
-      (effects (font (size 1.27 1.27)) hide)
-    )
-    (property "Footprint" "" (id 2) (at 151.13 107.95 0)
-      (effects (font (size 1.27 1.27)) hide)
-    )
-    (property "Datasheet" "" (id 3) (at 151.13 107.95 0)
-      (effects (font (size 1.27 1.27)) hide)
-    )
-    (pin "1")
   )
   (symbol (lib_id "My_custom_lib:TPS63020DSJR") (at 125.73 199.39 0) (unit 1)
     (in_bom yes) (on_board yes)
-    (property "Reference" "U17" (id 0) (at 133.35 224.79 0)
-      (effects (font (size 1.27 1.27)) (justify left))
-    )
-    (property "Value" "TPS63020DSJR" (id 1) (at 133.35 227.33 0)
+    (property "Reference" "U17" (id 0) (at 135.89 189.23 0)
+      (effects (font (size 1.27 1.27)) (justify left))
+    )
+    (property "Value" "TPS63020DSJR" (id 1) (at 135.89 191.77 0)
       (effects (font (size 1.27 1.27)) (justify left))
     )
@@
     (pin "2")
   )
+  (symbol (lib_id "Device:R_Small") (at 147.32 224.79 0) (unit 1)
+    (in_bom yes) (on_board yes) (fields_autoplaced)
+    (property "Reference" "R99" (id 0) (at 149.86 223.5199 0)
+      (effects (font (size 1.27 1.27)) (justify left))
+    )
+    (property "Value" "100k" (id 1) (at 149.86 226.0599 0)
+      (effects (font (size 1.27 1.27)) (justify left))
+    )
+    (property "Footprint" "Resistor_SMD:R_0603_1608Metric_Pad0.98x0.95mm_HandSolder" (id 2) (at 147.32 224.79 0)
+      (effects (font (size 1.27 1.27)) hide)
+    )
+    (property "Datasheet" "~" (id 3) (at 147.32 224.79 0)
+      (effects (font (size 1.27 1.27)) hide)
+    )
+    (pin "1")
+    (pin "2")
+  )
   (symbol (lib_id "Device:C_Small") (at 213.36 210.82 0) (unit 1)
     (in_bom yes) (on_board yes) (fields_autoplaced)
@@
     (pin "2")
   )
-  (symbol (lib_name "TPS63020DSJR_1") (lib_id "My_custom_lib:TPS63020DSJR") (at 129.54 90.17 0) (unit 1)
+  (symbol (lib_id "My_custom_lib:TPS63020DSJR") (at 129.54 90.17 0) (unit 1)
     (in_bom yes) (on_board yes)
     (property "Reference" "U16" (id 0) (at 137.16 115.57 0)
@@
     (pin "9")
   )
-  (symbol (lib_id "power:GND") (at 147.32 217.17 0) (unit 1)
-    (in_bom yes) (on_board yes) (fields_autoplaced)
-    (property "Reference" "#PWR0186" (id 0) (at 147.32 223.52 0)
-      (effects (font (size 1.27 1.27)) hide)
-    )
-    (property "Value" "GND" (id 1) (at 147.32 222.25 0)
-      (effects (font (size 1.27 1.27)) hide)
-    )
-    (property "Footprint" "" (id 2) (at 147.32 217.17 0)
-      (effects (font (size 1.27 1.27)) hide)
-    )
-    (property "Datasheet" "" (id 3) (at 147.32 217.17 0)
-      (effects (font (size 1.27 1.27)) hide)
-    )
+  (symbol (lib_id "power:GND") (at 147.32 229.87 0) (unit 1)
+    (in_bom yes) (on_board yes) (fields_autoplaced)
+    (property "Reference" "#PWR0186" (id 0) (at 147.32 236.22 0)
+      (effects (font (size 1.27 1.27)) hide)
+    )
+    (property "Value" "GND" (id 1) (at 147.32 234.95 0)
+      (effects (font (size 1.27 1.27)) hide)
+    )
+    (property "Footprint" "" (id 2) (at 147.32 229.87 0)
+      (effects (font (size 1.27 1.27)) hide)
+    )
+    (property "Datasheet" "" (id 3) (at 147.32 229.87 0)
+      (effects (font (size 1.27 1.27)) hide)
+    )

Commit message: h
Parts:
- C57, C58, C59, C60, C62, C63, C64, C65: footprint Capacitor_SMD:C_0603_1608Metric_Pad1.08x0.95mm_HandSolder -> Capacitor_SMD:C_0805_2012Metric_Pad1.18x1.45mm_HandSolder
Changed lines of the file:
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@@
       (effects (font (size 1.27 1.27)) (justify left))
     )
-    (property "Footprint" "Capacitor_SMD:C_0603_1608Metric_Pad1.08x0.95mm_HandSolder" (id 2) (at 223.52 100.33 0)
+    (property "Footprint" "Capacitor_SMD:C_0805_2012Metric_Pad1.18x1.45mm_HandSolder" (id 2) (at 223.52 100.33 0)
       (effects (font (size 1.27 1.27)) hide)
     )
@@
       (effects (font (size 1.27 1.27)) (justify left))
     )
-    (property "Footprint" "Capacitor_SMD:C_0603_1608Metric_Pad1.08x0.95mm_HandSolder" (id 2) (at 215.9 100.33 0)
+    (property "Footprint" "Capacitor_SMD:C_0805_2012Metric_Pad1.18x1.45mm_HandSolder" (id 2) (at 215.9 100.33 0)
       (effects (font (size 1.27 1.27)) hide)
     )
@@
       (effects (font (size 1.27 1.27)) (justify left))
     )
-    (property "Footprint" "Capacitor_SMD:C_0603_1608Metric_Pad1.08x0.95mm_HandSolder" (id 2) (at 77.47 97.79 0)
+    (property "Footprint" "Capacitor_SMD:C_0805_2012Metric_Pad1.18x1.45mm_HandSolder" (id 2) (at 77.47 97.79 0)
       (effects (font (size 1.27 1.27)) hide)
     )
@@
       (effects (font (size 1.27 1.27)) (justify left))
     )
-    (property "Footprint" "Capacitor_SMD:C_0603_1608Metric_Pad1.08x0.95mm_HandSolder" (id 2) (at 205.74 210.82 0)
+    (property "Footprint" "Capacitor_SMD:C_0805_2012Metric_Pad1.18x1.45mm_HandSolder" (id 2) (at 205.74 210.82 0)
       (effects (font (size 1.27 1.27)) hide)
     )
@@
       (effects (font (size 1.27 1.27)) (justify left))
     )
-    (property "Footprint" "Capacitor_SMD:C_0603_1608Metric_Pad1.08x0.95mm_HandSolder" (id 2) (at 213.36 210.82 0)
+    (property "Footprint" "Capacitor_SMD:C_0805_2012Metric_Pad1.18x1.45mm_HandSolder" (id 2) (at 213.36 210.82 0)
       (effects (font (size 1.27 1.27)) hide)
     )
@@
       (effects (font (size 1.27 1.27)) (justify left))
     )
-    (property "Footprint" "Capacitor_SMD:C_0603_1608Metric_Pad1.08x0.95mm_HandSolder" (id 2) (at 220.98 210.82 0)
+    (property "Footprint" "Capacitor_SMD:C_0805_2012Metric_Pad1.18x1.45mm_HandSolder" (id 2) (at 220.98 210.82 0)
       (effects (font (size 1.27 1.27)) hide)
     )
@@
       (effects (font (size 1.27 1.27)) (justify left))
     )
-    (property "Footprint" "Capacitor_SMD:C_0603_1608Metric_Pad1.08x0.95mm_HandSolder" (id 2) (at 74.93 207.01 0)
+    (property "Footprint" "Capacitor_SMD:C_0805_2012Metric_Pad1.18x1.45mm_HandSolder" (id 2) (at 74.93 207.01 0)
       (effects (font (size 1.27 1.27)) hide)
     )
@@
       (effects (font (size 1.27 1.27)) (justify left))
     )
-    (property "Footprint" "Capacitor_SMD:C_0603_1608Metric_Pad1.08x0.95mm_HandSolder" (id 2) (at 231.14 100.33 0)
-      (effects (font (size 1.27 1.27)) hide)
-    )
+    (property "Footprint" "Capacitor_SMD:C_0805_2012Metric_Pad1.18x1.45mm_HandSolder" (id 2) (at 231.14 100.33 0)
+      (effects (font (size 1.27 1.27)) hide)
+    )
