File: Bird_detector_V1/SMPSs.kicad_sch (KiCad schematic)
At the start: 24 parts, among them U16 TPS63020DSJR, U17 TPS63020DSJR

Commit message: b
Other:
- title: (none) -> Bird Detection and Recognition System
Changed lines of the file:
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@@
 (kicad_sch (version 20211123) (generator eeschema)
   (paper "A3")
+  (title_block
+    (title "Bird Detection and Recognition System")
+    (rev "V0.1")
+  )
   (junction (at 130.81 187.96) (diameter 0) (color 0 0 0 0)
   )

Commit message: y
Parts:
- added J12: enable, Connector_PinHeader_2.54mm:PinHeader_1x02_P2.54mm_Vertical, symbol Connector_Generic:Conn_01x02
- R89: value 1.32Meg -> 1.33Meg
Connections:
- net EN_3V3: now also C66.1, JP6.2 (B), U17.12 (EN), J12.2 (Pin_2)
- net GND: now also J12.1 (Pin_1)
- removed net EN_3V8: C66.1, JP6.2 (B), U17.1 (VINA), U17.12 (EN)
- no-connect marks 0 -> 1
Other:
- note added: "3V825"
- note added: "3v277"
- note removed: "3v3"
Changed lines of the file:
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@@
   (junction (at 110.49 227.33) (diameter 0) (color 0 0 0 0)
   )
-  (junction (at 102.87 214.63) (diameter 0) (color 0 0 0 0)
-  )
   (junction (at 147.32 90.17) (diameter 0) (color 0 0 0 0)
   )
@@
   (junction (at 151.13 99.06) (diameter 0) (color 0 0 0 0)
   )
+  (no_connect (at 113.03 214.63))
   (wire (pts (xy 147.32 208.28) (xy 147.32 209.55))
     (stroke (width 0) (type default) (color 0 0 0 0))
@@
     (stroke (width 0) (type default) (color 0 0 0 0))
   )
+  (wire (pts (xy 80.01 168.91) (xy 91.44 168.91))
+    (stroke (width 0) (type default) (color 0 0 0 0))
+  )
   (wire (pts (xy 114.3 92.71) (xy 114.3 90.17))
     (stroke (width 0) (type default) (color 0 0 0 0))
@@
     (stroke (width 0) (type default) (color 0 0 0 0))
   )
+  (wire (pts (xy 80.01 171.45) (xy 80.01 176.53))
+    (stroke (width 0) (type default) (color 0 0 0 0))
+  )
   (wire (pts (xy 114.3 92.71) (xy 116.84 92.71))
     (stroke (width 0) (type default) (color 0 0 0 0))
   )
-  (wire (pts (xy 113.03 214.63) (xy 102.87 214.63))
-    (stroke (width 0) (type default) (color 0 0 0 0))
-  )
   (wire (pts (xy 137.16 78.74) (xy 137.16 82.55))
     (stroke (width 0) (type default) (color 0 0 0 0))
@@
     (stroke (width 0) (type default) (color 0 0 0 0))
   )
-  (text "3v3" (at 163.83 105.41 180)
+  (text "3v277" (at 166.37 105.41 180)
     (effects (font (size 1.27 1.27)) (justify right bottom))
   )
@@
     (effects (font (size 4 4)) (justify right bottom))
   )
+  (text "3V825" (at 157.48 213.36 0)
+    (effects (font (size 1.27 1.27)) (justify left bottom))
+  )
   (text "3V-3V3" (at 144.78 69.85 180)
     (effects (font (size 4 4)) (justify right bottom))
@@
     (effects (font (size 1.27 1.27)) (justify left bottom))
   )
+  (label "EN_3V3" (at 91.44 168.91 0)
+    (effects (font (size 1.27 1.27)) (justify left bottom))
+  )
   (label "PG_3V3" (at 170.18 110.49 0)
+    (effects (font (size 1.27 1.27)) (justify left bottom))
+  )
+  (label "EN_3V8" (at 82.55 168.91 0)
     (effects (font (size 1.27 1.27)) (justify left bottom))
   )
@@
       (effects (font (size 1.27 1.27)) (justify left))
     )
-    (property "Value" "1.32Meg" (id 1) (at 149.86 204.4699 0)
+    (property "Value" "1.33Meg" (id 1) (at 149.86 204.4699 0)
       (effects (font (size 1.27 1.27)) (justify left))
     )
@@
     (pin "9")
   )
+  (symbol (lib_id "power:GND") (at 80.01 176.53 0) (unit 1)
+    (in_bom yes) (on_board yes) (fields_autoplaced)
+    (property "Reference" "#PWR034" (id 0) (at 80.01 182.88 0)
+      (effects (font (size 1.27 1.27)) hide)
+    )
+    (property "Value" "GND" (id 1) (at 80.01 181.61 0)
+      (effects (font (size 1.27 1.27)) hide)
+    )
+    (property "Footprint" "" (id 2) (at 80.01 176.53 0)
+      (effects (font (size 1.27 1.27)) hide)
+    )
+    (property "Datasheet" "" (id 3) (at 80.01 176.53 0)
+      (effects (font (size 1.27 1.27)) hide)
+    )
+    (pin "1")
+  )
   (symbol (lib_id "Device:C_Small") (at 205.74 210.82 0) (unit 1)
     (in_bom yes) (on_board yes) (fields_autoplaced)
@@
     (pin "1")
   )
+  (symbol (lib_id "Connector_Generic:Conn_01x02") (at 74.93 171.45 180) (unit 1)
+    (in_bom no) (on_board yes) (fields_autoplaced)
+    (property "Reference" "J12" (id 0) (at 74.93 162.56 0))
+    (property "Value" "enable" (id 1) (at 74.93 165.1 0))
+    (property "Footprint" "Connector_PinHeader_2.54mm:PinHeader_1x02_P2.54mm_Vertical" (id 2) (at 74.93 171.45 0)
+      (effects (font (size 1.27 1.27)) hide)
+    )
+    (property "Datasheet" "~" (id 3) (at 74.93 171.45 0)
+      (effects (font (size 1.27 1.27)) hide)
+    )
+    (pin "1")
+    (pin "2")
+  )
   (symbol (lib_id "power:GND") (at 231.14 107.95 0) (unit 1)

Commit message: g
Other:
- moved on the sheet: C62, C63, C64, C65, C66, J12, JP6, L3, R89, R90, R91, R92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
