File: Cell_Holder_Board/Cell_Holder_Board.kicad_sch (KiCad schematic)
At the start: 24 parts, among them J1 ntc 10k, SW1 BMS_RESET, U1 MP2615

Commit message: v
Parts:
- added BT1, BT2, BT3: 18650_SMD_top, Z_mycustom_footprint_lib:MYOUNG BH 18650 B1BA002, symbol Device:Battery_Cell
- added BT5, BT6, BT7, BT8: 18650_THT_bottom, Z_mycustom_footprint_lib:MYOUNG MY-18650-01, symbol Device:Battery_Cell
- added FID1, FID2, FID3, FID4: Cell, Z_mycustom_footprint_lib:18650 cell 3d model, symbol Mechanical:Fiducial
- added J2: IN/OUT, TerminalBlock:TerminalBlock_Altech_AK300-3_P5.00mm, symbol Connector:Screw_Terminal_01x03
- added J3: IN/OUT, TerminalBlock:TerminalBlock_Altech_AK300-2_P5.00mm, symbol Connector:Screw_Terminal_01x03
Connections:
- net +BATT: now also BT1.1 (+), BT2.1 (+), BT3.1 (+), BT5.1 (+), BT6.1 (+), BT7.1 (+), BT8.1 (+), J2.2 (Pin_2)
- net GND: now also BT1.2 (-), BT2.2 (-), BT3.2 (-), BT5.2 (-), BT6.2 (-), BT7.2 (-), BT8.2 (-), J2.1 (Pin_1), J3.1 (Pin_1); no longer H1.1, H2.1, H3.1, H4.1, H5.1, H6.1
- net at C1.1, JP1.1 (A), U1.2 (VIN): now also J3.2 (Pin_2)
- new net Heater: J2.3 (Pin_3)
- no-connect marks 1 -> 8

Commit message: f
Parts:
- removed FID1, FID2, FID3, FID4: Cell, Z_mycustom_footprint_lib:18650 cell 3d model, symbol Mechanical:Fiducial
- added NT1: NetTie_2, NetTie:NetTie-2_THT_Pad1.0mm, symbol Device:NetTie_2
Connections:
- net BMS_LED: now also R4.2, R5.2; no longer D1.2 (A), D2.2 (A)
- net GND: now also NT1.1
- net Heater: now also NT1.2
- net at D2.1 (K): now also U1.12 (~{ACOK}); no longer R5.2
- net at U1.11 (~{CHGOK}): now also D1.1 (K); no longer R4.1
- net at R5.1: now also D2.2 (A); no longer U1.12 (~{ACOK})
- new net: D1.2 (A), R4.1
Other:
- note added: "heater: 0.5mm 3755mm long ==> 3.7 ohm @ 3A max"
- moved on the sheet: D1, D2, J3, R4, R5
