File: Cell_Holder_Board_V2/Cell_Holder_Board_V2.kicad_pcb (KiCad board)
At the start: 2 copper layers, 126.5 x 76.1 mm, 16 parts, among them J1 IN/OUT

Commit message: f
Parts:
- added kibuzzard-63734D02: G***, kibuzzard-63734D02, F.Cu at (86.4, 91.2)
- added kibuzzard-63734D02: G***, kibuzzard-63734D02, B.Cu at (86.4, 91.2)
- added kibuzzard-63734D11: G***, kibuzzard-63734D11, F.Cu at (91.8, 86.5)
- added kibuzzard-63734D11: G***, kibuzzard-63734D11, B.Cu at (91.9, 86.5)
- added kibuzzard-63734D26: G***, kibuzzard-63734D26, F.Cu at (80.8, 88.1)
- added kibuzzard-63734D26: G***, kibuzzard-63734D26, B.Cu at (80.8, 88.1)
- added kibuzzard-63736DA7: G***, kibuzzard-63736DA7, B.Cu at (81.0, 113.9)
- added kibuzzard-63736DA7: G***, kibuzzard-63736DA7, B.Cu at (93.0, 109.2)
- added kibuzzard-63736DC2: G***, kibuzzard-63736DC2, B.Cu at (85.5, 113.2)
- added kibuzzard-63736DC2: G***, kibuzzard-63736DC2, B.Cu at (89.0, 108.0)
- added kibuzzard-63736FCA: G***, kibuzzard-63736FCA, B.Cu at (99.1, 113.3)
- added kibuzzard-63736FCA: G***, kibuzzard-63736FCA, B.Cu at (95.6, 107.6)
Routing:
- net /Heater: track 5007.2 -> 15632.6 mm, vias 2 -> 5
- net GND: track 266.3 -> 277.2 mm, vias 0 -> 315
- added copper zone on F.Cu, net +BATT
- added copper zone on B.Cu, net /Heater
- added copper zone on F.Cu, net /Heater
- added copper zone on B.Cu, net GND
