File: Cell_Holder_Board_V2/Cell_Holder_Board_V2.kicad_sch (KiCad schematic)
At the start: 16 parts, among them J1 IN/OUT

Commit message: f
Other:
- note added: "bottom heater: 0.5mm 5000mm ==> 4.9 ohm 3A max delta 60C top heater 0.13mm 1340mm ==> 5.4 ohm 1A max delta 60C Both are in paralel so 2.57 ohm ESR"
Changed lines of the file:
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@@
     (stroke (width 0) (type default) (color 0 0 0 0))
+  )
+  (text "bottom heater: 0.5mm 5000mm ==> 4.9 ohm  3A max delta 60C  \ntop heater 0.13mm 1340mm ==> 5.4 ohm 1A max delta 60C\nBoth are in paralel so 2.57 ohm ESR"
+    (at 187.96 25.4 0)
+    (effects (font (size 1.27 1.27)) (justify left bottom))
   )
   (label "Heater" (at 156.21 31.75 0)
